File: Circuit/robot fő nyák/robot fő nyák.kicad_sch (KiCad schematic)
At the start: 0 parts

Commit message: new circuit_v0.2
Parts:
- added Module1: ComputeModule4, robot fő nyák:Raspberry-Pi-4-Compute-Module, symbol CM4IO:ComputeModule4-CM4
Other:
- added sheet 3v3_psu (3v3_psu.kicad_sch)
- added sheet 4pcs TMC2240 (4pcs TMC2240.kicad_sch)
- added sheet 5V_psu (5v_psu.kicad_sch)
- added sheet bat (bat.kicad_sch)
