File: Circuit/kicad/Robot fő nyák_v3/CM5IO.kicad_sch (KiCad schematic)
At the start: 1 part, among them SW4 SW_DIP_x08

Commit message: kicad update new readme media updates the circuit is 95% finished
Connections:
- net BT_nDis is gone; now on net 5v: SW4.7
- net GND: no longer names the net of SW4.9
- net GND: no longer SW4.10
- net WL_nDis: no longer names the net of SW4.8
- new net TPA_ON: SW4.10
- no-connect marks 0 -> 2
Other:
- sheet CM5_GPIO ( Ethernet, GPIO, SDCARD) ports: added none; removed BT_nDis, WL_nDis
Changed lines of the file:
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@@
+	)
+	(junction
+		(at 270.51 127)
+		(diameter 0)
+		(color 0 0 0 0)
 	)
 	(junction
@@
 	)
 	(junction
-		(at 173.99 46.99)
-		(diameter 0)
-		(color 0 0 0 0)
-	)
-	(junction
 		(at 143.51 39.37)
 		(diameter 0)
 		(color 0 0 0 0)
 	)
+	(no_connect
+		(at 53.34 157.48)
+	)
+	(no_connect
+		(at 53.34 154.94)
+	)
 	(wire
 		(pts
@@
 	(wire
 		(pts
-			(xy 173.99 55.88) (xy 173.99 46.99)
-		)
-		(stroke
-			(width 0)
-			(type default)
-		)
-	)
-	(wire
-		(pts
 			(xy 110.49 92.71) (xy 119.38 92.71)
 		)
@@
 	(wire
 		(pts
-			(xy 173.99 46.99) (xy 173.99 44.45)
-		)
-		(stroke
-			(width 0)
-			(type default)
-		)
-	)
-	(wire
-		(pts
 			(xy 224.79 127) (xy 217.17 127)
 		)
@@
 	(wire
 		(pts
+			(xy 270.51 127) (xy 266.7 127)
+		)
+		(stroke
+			(width 0)
+			(type default)
+		)
+	)
+	(wire
+		(pts
 			(xy 110.49 67.31) (xy 119.38 67.31)
 		)
@@
 	(wire
 		(pts
-			(xy 120.65 158.75) (xy 110.49 158.75)
-		)
-		(stroke
-			(width 0)
-			(type default)
-		)
-	)
-	(wire
-		(pts
 			(xy 171.45 34.29) (xy 182.88 34.29)
 		)
@@
 	(wire
 		(pts
-			(xy 143.51 44.45) (xy 156.21 44.45)
-		)
-		(stroke
-			(width 0)
-			(type default)
-		)
-	)
-	(wire
-		(pts
 			(xy 143.51 39.37) (xy 156.21 39.37)
 		)
@@
 	(wire
 		(pts
+			(xy 273.05 127) (xy 270.51 127)
+		)
+		(stroke
+			(width 0)
+			(type default)
+		)
+	)
+	(wire
+		(pts
 			(xy 224.79 81.28) (xy 217.17 81.28)
 		)
@@
 	(wire
 		(pts
-			(xy 120.65 156.21) (xy 110.49 156.21)
-		)
-		(stroke
-			(width 0)
-			(type default)
-		)
-	)
-	(wire
-		(pts
 			(xy 209.55 33.02) (xy 217.17 33.02)
 		)
@@
 	(wire
 		(pts
+			(xy 274.32 124.46) (xy 270.51 124.46)
+		)
+		(stroke
+			(width 0)
+			(type default)
+		)
+	)
+	(wire
+		(pts
 			(xy 110.49 83.82) (xy 119.38 83.82)
 		)
@@
 	(wire
 		(pts
-			(xy 173.99 44.45) (xy 171.45 44.45)
-		)
-		(stroke
-			(width 0)
-			(type default)
-		)
-	)
-	(wire
-		(pts
 			(xy 217.17 111.76) (xy 224.79 111.76)
 		)
@@
 	(wire
 		(pts
+			(xy 148.59 44.45) (xy 156.21 44.45)
+		)
+		(stroke
+			(width 0)
+			(type default)
+		)
+	)
+	(wire
+		(pts
 			(xy 143.51 41.91) (xy 156.21 41.91)
 		)
@@
 	(wire
 		(pts
+			(xy 270.51 124.46) (xy 270.51 127)
+		)
+		(stroke
+			(width 0)
+			(type default)
+		)
+	)
+	(wire
+		(pts
 			(xy 110.49 69.85) (xy 119.38 69.85)
 		)
@@
 	(wire
 		(pts
-			(xy 171.45 46.99) (xy 173.99 46.99)
-		)
-		(stroke
-			(width 0)
-			(type default)
-		)
-	)
-	(wire
-		(pts
 			(xy 209.55 44.45) (xy 217.17 44.45)
 		)
@@
 		(pts
 			(xy 110.49 100.33) (xy 119.38 100.33)
-		)
-		(stroke
-			(width 0)
-			(type default)
-		)
-	)
-	(wire
-		(pts
-			(xy 143.51 46.99) (xy 156.21 46.99)
 		)
 		(stroke
@@
 		)
 	)
-	(label "BT_nDis"
-		(at 120.65 158.75 180)
+	(label "5v"
+		(at 148.59 44.45 180)
 		(effects
 			(font
@@
 		)
 	)
-	(label "WL_nDis"
-		(at 143.51 46.99 0)
-		(effects
-			(font
-				(size 1.27 1.27)
-			)
-			(justify left bottom)
-		)
-	)
 	(label "Uart_rx"
 		(at 105.41 34.29 180)
@@
 		)
 	)
-	(label "BT_nDis"
-		(at 143.51 44.45 0)
-		(effects
-			(font
-				(size 1.27 1.27)
-			)
-			(justify left bottom)
-		)
-	)
 	(label "12v_1"
 		(at 217.17 137.16 0)
@@
 		)
 	)
-	(label "WL_nDis"
-		(at 120.65 156.21 180)
-		(effects
-			(font
-				(size 1.27 1.27)
-			)
-			(justify right bottom)
-		)
-	)
 	(label "5v"
 		(at 217.17 33.02 180)
@@
 		)
 	)
+	(global_label "5V1"
+		(shape input)
+		(at 274.32 124.46 0)
+		(fields_autoplaced yes)
+		(effects
+			(font
+				(size 1.27 1.27)
+			)
+			(justify left)
+		)
+		(property "Intersheetrefs" "${INTERSHEET_REFS}"
+			(at 280.8128 124.46 0)
+			(effects
+				(font
+					(size 1.27 1.27)
+				)
+				(justify left)
+				(hide yes)
+			)
+		)
+	)
 	(global_label "ESP_3v3"
 		(shape input)
@@
 		)
 	)
-	(global_label "SERVO2"
+	(global_label "SERVO3"
 		(shape input)
 		(at 266.7 101.6 0)
@@
 	(global_label "USB_5V"
 		(shape input)
-		(at 266.7 127 0)
-		(fields_autoplaced yes)
-		(effects
-			(font
-				(size 1.27 1.27)
-			)
-			(justify left)
-		)
-		(property "Intersheetrefs" "${INTERSHEET_REFS}"
-			(at 276.7609 127 0)
+		(at 273.05 127 0)
+		(fields_autoplaced yes)
+		(effects
+			(font
+				(size 1.27 1.27)
+			)
+			(justify left)
+		)
+		(property "Intersheetrefs" "${INTERSHEET_REFS}"
+			(at 283.1109 127 0)
 			(effects
 				(font
@@
 		)
 	)
-	(symbol
-		(lib_id "power:GND")
-		(at 173.99 55.88 0)
-		(unit 1)
-		(exclude_from_sim no)
-		(in_bom yes)
-		(on_board yes)
-		(dnp no)
-		(fields_autoplaced yes)
-		(property "Reference" "#PWR0139"
-			(at 173.99 62.23 0)
-			(effects
-				(font
-					(size 1.27 1.27)
-				)
-				(hide yes)
-			)
-		)
-		(property "Value" "GND"
-			(at 173.99 60.96 0)
-			(effects
-				(font
-					(size 1.27 1.27)
-				)
-			)
-		)
-		(property "Footprint" ""
-			(at 173.99 55.88 0)
-			(effects
-				(font
-					(size 1.27 1.27)
-				)
-				(hide yes)
-			)
-		)
-		(property "Datasheet" ""
-			(at 173.99 55.88 0)
-			(effects
-				(font
-					(size 1.27 1.27)
-				)
-				(hide yes)
-			)
-		)
-		(property "Description" "Power symbol creates a global label with name \"GND\" , ground"
-			(at 173.99 55.88 0)
-			(effects
-				(font
-					(size 1.27 1.27)
-				)
-				(hide yes)
-			)
-		)
-		(pin "1"
-		)
-		(instances
-			(project ""
-				(path "/e63e39d7-6ac0-4ffd-8aa3-1841a4541b55"
-					(reference "#PWR0139")
-					(unit 1)
-				)
+	(global_label "TPA_ON"
+		(shape input)
+		(at 171.45 44.45 0)
+		(fields_autoplaced yes)
+		(effects
+			(font
+				(size 1.27 1.27)
+			)
+			(justify left)
+		)
+		(property "Intersheetrefs" "${INTERSHEET_REFS}"
+			(at 181.4851 44.45 0)
+			(effects
+				(font
+					(size 1.27 1.27)
+				)
+				(justify left)
+				(hide yes)
 			)
 		)
@@
 			(effects
 				(font
-					(size 1.27 1.27)
-				)
-				(justify right)
-			)
-		)
-		(pin "BT_nDis" input
-			(at 110.49 156.21 0)
-			(effects
-				(font
-					(size 1.27 1.27)
-				)
-				(justify right)
-			)
-		)
-		(pin "WL_nDis" input
-			(at 110.49 158.75 0)
-			(effects
-				(font
