File: Circuit/kicad/Robot fő nyák_v3/PCA9685.kicad_sch (KiCad schematic)
At the start: 2 parts, among them U56 ICM-45686

Commit message: kicad update new readme media updates the circuit is 95% finished
Parts:
- renumbered U56 to U
Changed lines of the file:
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@@
 		(instances
 			(project "CM5IO"
+				(path "/e63e39d7-6ac0-4ffd-8aa3-1841a4541b55/a83afe30-5c7e-43cb-a5b2-f6f97a0812b3/86209e6a-92ae-4699-a125-02d46b525fc7/7612cb3a-eef9-4566-8255-3c47e176ac07"
+					(reference "C140")
+					(unit 1)
+				)
 				(path "/e63e39d7-6ac0-4ffd-8aa3-1841a4541b55/a83afe30-5c7e-43cb-a5b2-f6f97a0812b3/86209e6a-92ae-4699-a125-02d46b525fc7/80185d9c-294a-4509-9bcc-8c38b499429e"
 					(reference "C58")
@@
 		(dnp no)
 		(fields_autoplaced yes)
-		(property "Reference" "U56"
+		(property "Reference" "U"
 			(at 71.882 36.322 0)
 			(effects
@@
 		)
 		(pin "2"
+		)
+		(instances
+			(project "CM5IO"
+				(path "/e63e39d7-6ac0-4ffd-8aa3-1841a4541b55/a83afe30-5c7e-43cb-a5b2-f6f97a0812b3/86209e6a-92ae-4699-a125-02d46b525fc7/7612cb3a-eef9-4566-8255-3c47e176ac07"
+					(reference "U66")
+					(unit 1)
+				)
+			)
 		)
 	)
@@
 		(instances
 			(project "CM5IO"
+				(path "/e63e39d7-6ac0-4ffd-8aa3-1841a4541b55/a83afe30-5c7e-43cb-a5b2-f6f97a0812b3/86209e6a-92ae-4699-a125-02d46b525fc7/7612cb3a-eef9-4566-8255-3c47e176ac07"
+					(reference "#PWR0139")
+					(unit 1)
+				)
 				(path "/e63e39d7-6ac0-4ffd-8aa3-1841a4541b55/a83afe30-5c7e-43cb-a5b2-f6f97a0812b3/86209e6a-92ae-4699-a125-02d46b525fc7/80185d9c-294a-4509-9bcc-8c38b499429e"
 					(reference "#PWR0125")
@@
 		(instances
 			(project "CM5IO"
+				(path "/e63e39d7-6ac0-4ffd-8aa3-1841a4541b55/a83afe30-5c7e-43cb-a5b2-f6f97a0812b3/86209e6a-92ae-4699-a125-02d46b525fc7/7612cb3a-eef9-4566-8255-3c47e176ac07"
+					(reference "#PWR0193")
+					(unit 1)
+				)
 				(path "/e63e39d7-6ac0-4ffd-8aa3-1841a4541b55/a83afe30-5c7e-43cb-a5b2-f6f97a0812b3/86209e6a-92ae-4699-a125-02d46b525fc7/80185d9c-294a-4509-9bcc-8c38b499429e"
 					(reference "#PWR0126")
