File: Circuit/kicad/Robot fő nyák_v3/I2C_MUX.kicad_sch (KiCad schematic)
At the start: 2 parts, among them U60 TS5A23157DGSR

Commit message: kicad update new readme media updates the circuit is 95% finished
Parts:
- added C131: 1uf, symbol Device:C
- R104: value 100k -> 47k
Connections:
- net 3V3_in: now also C131.2
- net GND: now also C131.1
Changed lines of the file:
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@@
+	)
+	(junction
+		(at 38.1 63.5)
+		(diameter 0)
+		(color 0 0 0 0)
+	)
+	(junction
+		(at 73.66 53.34)
+		(diameter 0)
+		(color 0 0 0 0)
 	)
 	(junction
@@
 	(wire
 		(pts
-			(xy 36.83 63.5) (xy 40.64 63.5)
+			(xy 36.83 63.5) (xy 38.1 63.5)
 		)
 		(stroke
@@
 		)
 	)
+	(wire
+		(pts
+			(xy 38.1 60.96) (xy 38.1 63.5)
+		)
+		(stroke
+			(width 0)
+			(type default)
+		)
+	)
+	(wire
+		(pts
+			(xy 71.12 53.34) (xy 73.66 53.34)
+		)
+		(stroke
+			(width 0)
+			(type default)
+		)
+	)
+	(wire
+		(pts
+			(xy 38.1 63.5) (xy 40.64 63.5)
+		)
+		(stroke
+			(width 0)
+			(type default)
+		)
+	)
+	(wire
+		(pts
+			(xy 73.66 53.34) (xy 81.28 53.34)
+		)
+		(stroke
+			(width 0)
+			(type default)
+		)
+	)
+	(global_label "I2C_CH"
+		(shape input)
+		(at 38.1 60.96 90)
+		(fields_autoplaced yes)
+		(effects
+			(font
+				(size 1.27 1.27)
+			)
+			(justify left)
+		)
+		(property "Intersheetrefs" "${INTERSHEET_REFS}"
+			(at 38.1 51.3224 90)
+			(effects
+				(font
+					(size 1.27 1.27)
+				)
+				(justify left)
+				(hide yes)
+			)
+		)
+	)
 	(hierarchical_label "I2C_CH"
 		(shape input)
@@
 	(hierarchical_label "3V3_in"
 		(shape input)
-		(at 81.28 53.34 180)
+		(at 71.12 53.34 180)
 		(effects
 			(font
@@
 			)
 			(justify right)
+		)
+	)
+	(symbol
+		(lib_id "power:GND")
+		(at 73.66 45.72 180)
+		(unit 1)
+		(exclude_from_sim no)
+		(in_bom yes)
+		(on_board yes)
+		(dnp no)
+		(fields_autoplaced yes)
+		(property "Reference" "#PWR0180"
+			(at 73.66 39.37 0)
+			(effects
+				(font
+					(size 1.27 1.27)
+				)
+				(hide yes)
+			)
+		)
+		(property "Value" "GND"
+			(at 73.66 40.64 0)
+			(effects
+				(font
+					(size 1.27 1.27)
+				)
+			)
+		)
+		(property "Footprint" ""
+			(at 73.66 45.72 0)
+			(effects
+				(font
+					(size 1.27 1.27)
+				)
+				(hide yes)
+			)
+		)
+		(property "Datasheet" ""
+			(at 73.66 45.72 0)
+			(effects
+				(font
+					(size 1.27 1.27)
+				)
+				(hide yes)
+			)
+		)
+		(property "Description" "Power symbol creates a global label with name \"GND\" , ground"
+			(at 73.66 45.72 0)
+			(effects
+				(font
+					(size 1.27 1.27)
+				)
+				(hide yes)
+			)
+		)
+		(pin "1"
+		)
+		(instances
+			(project "CM5IO"
+				(path "/e63e39d7-6ac0-4ffd-8aa3-1841a4541b55/a83afe30-5c7e-43cb-a5b2-f6f97a0812b3/a92c9c42-f6c0-4e3f-b1e7-7f0cf3827d33"
+					(reference "#PWR0180")
+					(unit 1)
+				)
+			)
 		)
 	)
@@
 	)
 	(symbol
+		(lib_id "Device:C")
+		(at 73.66 49.53 0)
+		(unit 1)
+		(exclude_from_sim no)
+		(in_bom yes)
+		(on_board yes)
+		(dnp no)
+		(fields_autoplaced yes)
+		(property "Reference" "C131"
+			(at 77.47 48.2599 0)
+			(effects
+				(font
+					(size 1.27 1.27)
+				)
+				(justify left)
+			)
+		)
+		(property "Value" "1uf"
+			(at 77.47 50.7999 0)
+			(effects
+				(font
+					(size 1.27 1.27)
+				)
+				(justify left)
+			)
+		)
+		(property "Footprint" ""
+			(at 74.6252 53.34 0)
+			(effects
+				(font
+					(size 1.27 1.27)
+				)
+				(hide yes)
+			)
+		)
+		(property "Datasheet" "~"
+			(at 73.66 49.53 0)
+			(effects
+				(font
+					(size 1.27 1.27)
+				)
+				(hide yes)
+			)
+		)
+		(property "Description" "Unpolarized capacitor"
+			(at 73.66 49.53 0)
+			(effects
+				(font
+					(size 1.27 1.27)
+				)
+				(hide yes)
+			)
+		)
+		(pin "1"
+		)
+		(pin "2"
+		)
+		(instances
+			(project "CM5IO"
+				(path "/e63e39d7-6ac0-4ffd-8aa3-1841a4541b55/a83afe30-5c7e-43cb-a5b2-f6f97a0812b3/a92c9c42-f6c0-4e3f-b1e7-7f0cf3827d33"
+					(reference "C131")
+					(unit 1)
+				)
+			)
+		)
+	)
+	(symbol
 		(lib_id "Device:R")
 		(at 33.02 63.5 90)
@@
 			)
 		)
-		(property "Value" "100k"
+		(property "Value" "47k"
 			(at 33.02 59.69 90)
 			(effects

Commit message: readme updated kicad circuit V1
Parts:
- C138: renamed from C131; footprint (none) -> Capacitor_SMD:C_0805_2012Metric
- R120: renamed from R104; footprint (none) -> Resistor_SMD:R_0805_2012Metric
- U66: renamed from U60; footprint TS5A23157DGSR:SOP50P490X110-10N -> CM5IO:SOP50P490X110-10N
Changed lines of the file:
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@@
 		(dnp no)
 		(fields_autoplaced yes)
-		(property "Reference" "#PWR0180"
+		(property "Reference" "#PWR0188"
 			(at 73.66 39.37 0)
 			(effects
@@
 			(project "CM5IO"
 				(path "/e63e39d7-6ac0-4ffd-8aa3-1841a4541b55/a83afe30-5c7e-43cb-a5b2-f6f97a0812b3/a92c9c42-f6c0-4e3f-b1e7-7f0cf3827d33"
-					(reference "#PWR0180")
+					(reference "#PWR0188")
 					(unit 1)
 				)
@@
 		(dnp no)
 		(fields_autoplaced yes)
-		(property "Reference" "#PWR0152"
+		(property "Reference" "#PWR0187"
 			(at 22.86 63.5 0)
 			(effects
@@
 			(project "CM5IO"
 				(path "/e63e39d7-6ac0-4ffd-8aa3-1841a4541b55/a83afe30-5c7e-43cb-a5b2-f6f97a0812b3/a92c9c42-f6c0-4e3f-b1e7-7f0cf3827d33"
-					(reference "#PWR0152")
+					(reference "#PWR0187")
 					(unit 1)
 				)
@@
 		(dnp no)
 		(fields_autoplaced yes)
-		(property "Reference" "C131"
+		(property "Reference" "C138"
 			(at 77.47 48.2599 0)
 			(effects
@@
 			)
 		)
-		(property "Footprint" ""
+		(property "Footprint" "Capacitor_SMD:C_0805_2012Metric"
 			(at 74.6252 53.34 0)
 			(effects
@@
 			(project "CM5IO"
 				(path "/e63e39d7-6ac0-4ffd-8aa3-1841a4541b55/a83afe30-5c7e-43cb-a5b2-f6f97a0812b3/a92c9c42-f6c0-4e3f-b1e7-7f0cf3827d33"
-					(reference "C131")
+					(reference "C138")
 					(unit 1)
 				)
@@
 		(dnp no)
 		(fields_autoplaced yes)
-		(property "Reference" "R104"
+		(property "Reference" "R120"
 			(at 33.02 57.15 90)
 			(effects
@@
 			)
 		)
-		(property "Footprint" ""
+		(property "Footprint" "Resistor_SMD:R_0805_2012Metric"
 			(at 33.02 65.278 90)
 			(effects
@@
 			(project "CM5IO"
 				(path "/e63e39d7-6ac0-4ffd-8aa3-1841a4541b55/a83afe30-5c7e-43cb-a5b2-f6f97a0812b3/a92c9c42-f6c0-4e3f-b1e7-7f0cf3827d33"
-					(reference "R104")
+					(reference "R120")
 					(unit 1)
 				)
@@
 		(dnp no)
 		(fields_autoplaced yes)
-		(property "Reference" "U60"
+		(property "Reference" "U66"
 			(at 99.06 45.72 0)
 			(effects
@@
 			)
 		)
-		(property "Footprint" "TS5A23157DGSR:SOP50P490X110-10N"
+		(property "Footprint" "CM5IO:SOP50P490X110-10N"
 			(at 99.06 66.04 0)
 			(effects
@@
 			(project ""
 				(path "/e63e39d7-6ac0-4ffd-8aa3-1841a4541b55/a83afe30-5c7e-43cb-a5b2-f6f97a0812b3/a92c9c42-f6c0-4e3f-b1e7-7f0cf3827d33"
-					(reference "U60")
+					(reference "U66")
 					(unit 1)
 				)
@@
 		(dnp no)
 		(fields_autoplaced yes)
-		(property "Reference" "#PWR0146"
+		(property "Reference" "#PWR0189"
 			(at 123.19 78.74 0)
 			(effects
@@
 			(project "CM5IO"
 				(path "/e63e39d7-6ac0-4ffd-8aa3-1841a4541b55/a83afe30-5c7e-43cb-a5b2-f6f97a0812b3/a92c9c42-f6c0-4e3f-b1e7-7f0cf3827d33"
-					(reference "#PWR0146")
+					(reference "#PWR0189")
 					(unit 1)
 				)
