File: Circuit/kicad/Robot fő nyák_v3/_autosave-CM5IO.kicad_pcb (KiCad board)
At the start: 6 copper layers, 473 parts, among them J1 XT60-M, J10 USB_C_Receptacle_USB2.0_16P, J11 THD-02-R, J12 Conn_01x04_Socket, J13 THD-02-R, J2 USB3_A, J3 690-019-298-412, J31 Conn_01x02_Pin, J32 Conn_01x02_Pin, J4 690-019-298-412, J5 MagJack-A70-112-331N126, J6 Bus_M.2_Socket_M, J7 690-008-221-904, J8 USB_C_Receptacle_USB2.0_16P, J9 USB_C_Receptacle_USB2.0_16P, M4 Stepper_Motor_unipolar_6pin, M5 Stepper_Motor_unipolar_6pin, M6 Stepper_Motor_unipolar_6pin, M7 Stepper_Motor_unipolar_6pin, Q1 IRLHM630PbF, Q10 IRLML2502, Q11 IRLML2502, Q12 IRLML2502, Q13 IRLML2502, Q14 IRLML2502, Q15 IRLML2502, Q16 IRLML2502, Q17 IRLML2502, Q18 IRLML2502, Q19 IRLML2502, Q2 SS8050-G, Q20 IRLML2502, Q21 IRLML2502, Q22 IRLML2502, Q23 IRLML2502, Q24 IRLML2502, Q25 IRLML2502, Q26 IRLHM630PbF, Q3 SS8050-G, Q4 IRLML2502, Q5 IRLML2502, Q6 IRLML2502, Q7 IRLML2502, Q8 IRLML2502, Q9 IRLML2502, SW1 Right angle Tact button, SW2 SW_Push, SW3 SW_Push, SW4 SW_Push, U1 AP22653W6, U10 TPD4EUSB30, U11 USB2514B-I/M2, U12 TPD4EUSB30, U13 FSUSB42MUX, U14 TPD4EUSB30, U15 INA226, U16 INA226, U17 INA226, U18 INA226, U19 INA226, U2 RT9742SNGV, U20 INA226, U21 INA226, U22 INA226, U23 INA226, U24 INA226, U25 INA226, U26 INA226, U27 INA226, U28 INA226, U29 INA226, U3 74LVC1G07SE-7, U30 INA226, U31 AP64501SP-13, U32 AP64501SP-13, U33 AP64501SP-13, U34 AP64501SP-13, U35 AP64501SP-13, U37 CH343P, U4 TPD4EUSB30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

Commit message: readme updated kicad circuit V1
Parts:
- moved C7 1009.5 mm to (433.5, 105.3)
- moved D1 1009.5 mm to (434.2, 94.4)
- moved D2 1009.5 mm to (434.2, 97.8)
- moved J12 1009.5 mm to (423.7, 88.9)
- moved R5 1009.5 mm to (414.7, 78.8)
- moved R6 1009.5 mm to (414.7, 81.8)
- moved R7 1009.5 mm to (414.7, 84.7)
- moved TP2 1009.5 mm to (434.1, 56.4)
- moved TP3 1009.5 mm to (434.1, 60.4)
- moved TP7 1009.5 mm to (434.1, 64.5)
- moved TP8 1009.5 mm to (434.1, 68.5)
- moved U5 1009.5 mm to (435.7, 101.8)
- moved BT1 1009.5 mm to (415.5, 102.0)
- moved DSW2 1009.5 mm to (416.6, 92.7)
- moved GPIO1 1009.5 mm to (407.6, 56.6)
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Other:
- board outline added: 130 x 90 mm
