File: Circuit/kicad/Robot fő nyák_v3/spi_mux.kicad_sch (KiCad schematic)
At the start: 6 parts, among them U61 TS5A23157DGSR, U62 TS5A23157DGSR, U63 TS5A23157DGSR, U64 TS5A23157DGSR

Commit message: kicad update new readme media updates the circuit is 95% finished
Parts:
- added C128, C129, C130, C59: 1uf, symbol Device:C
- added CT9: 10uf, symbol Device:C_Polarized_Small
- R103, R105: value 100k -> 47k
Connections:
- net 3V3_in: now also C128.1, C129.1, C130.1, C59.1, CT9.1
- net GND: now also C128.2, C129.2, C130.2, C59.2, CT9.2

Commit message: readme updated kicad circuit V1
Parts:
- C116: renamed from C130; footprint (none) -> Capacitor_SMD:C_0805_2012Metric
- C117: renamed from C129; footprint (none) -> Capacitor_SMD:C_0805_2012Metric
- C118: renamed from C59; footprint (none) -> Capacitor_SMD:C_0805_2012Metric
- C119: renamed from C128; footprint (none) -> Capacitor_SMD:C_0805_2012Metric
- CT8: renamed from CT9; footprint (none) -> Capacitor_Tantalum_SMD:CP_EIA-3528-21_Kemet-B
- R104: renamed from R105; footprint (none) -> Resistor_SMD:R_0805_2012Metric
- R105: renamed from R103; footprint (none) -> Resistor_SMD:R_0805_2012Metric
- U59: renamed from U63; footprint TS5A23157DGSR:SOP50P490X110-10N -> CM5IO:SOP50P490X110-10N
- U60: renamed from U64; footprint TS5A23157DGSR:SOP50P490X110-10N -> CM5IO:SOP50P490X110-10N
- U61, U62: footprint TS5A23157DGSR:SOP50P490X110-10N -> CM5IO:SOP50P490X110-10N
Changed lines of the file:
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@@
 			)
 		)
-		(property "Footprint" "TS5A23157DGSR:SOP50P490X110-10N"
+		(property "Footprint" "CM5IO:SOP50P490X110-10N"
 			(at 237.49 72.39 0)
 			(effects
@@
 		(dnp no)
 		(fields_autoplaced yes)
-		(property "Reference" "C59"
+		(property "Reference" "C118"
 			(at 86.36 153.6699 0)
 			(effects
@@
 			)
 		)
-		(property "Footprint" ""
+		(property "Footprint" "Capacitor_SMD:C_0805_2012Metric"
 			(at 83.5152 158.75 0)
 			(effects
@@
 			(project "CM5IO"
 				(path "/e63e39d7-6ac0-4ffd-8aa3-1841a4541b55/a83afe30-5c7e-43cb-a5b2-f6f97a0812b3/a19d279d-385c-42b4-ac38-2ed1d04b4250"
-					(reference "C59")
+					(reference "C118")
 					(unit 1)
 				)
@@
 			)
 		)
-		(property "Footprint" "TS5A23157DGSR:SOP50P490X110-10N"
+		(property "Footprint" "CM5IO:SOP50P490X110-10N"
 			(at 237.49 110.49 0)
 			(effects
@@
 		(dnp no)
 		(fields_autoplaced yes)
-		(property "Reference" "#PWR0151"
+		(property "Reference" "#PWR0165"
 			(at 161.29 90.17 0)
 			(effects
@@
 			(project "CM5IO"
 				(path "/e63e39d7-6ac0-4ffd-8aa3-1841a4541b55/a83afe30-5c7e-43cb-a5b2-f6f97a0812b3/a19d279d-385c-42b4-ac38-2ed1d04b4250"
-					(reference "#PWR0151")
+					(reference "#PWR0165")
 					(unit 1)
 				)
@@
 		(dnp no)
 		(fields_autoplaced yes)
-		(property "Reference" "CT9"
+		(property "Reference" "CT8"
 			(at 111.76 153.1238 0)
 			(effects
@@
 			)
 		)
-		(property "Footprint" ""
+		(property "Footprint" "Capacitor_Tantalum_SMD:CP_EIA-3528-21_Kemet-B"
 			(at 109.22 154.94 0)
 			(effects
@@
 			(project "CM5IO"
 				(path "/e63e39d7-6ac0-4ffd-8aa3-1841a4541b55/a83afe30-5c7e-43cb-a5b2-f6f97a0812b3/a19d279d-385c-42b4-ac38-2ed1d04b4250"
-					(reference "CT9")
+					(reference "CT8")
 					(unit 1)
 				)
@@
 		(dnp no)
 		(fields_autoplaced yes)
-		(property "Reference" "C130"
+		(property "Reference" "C116"
 			(at 63.5 153.6699 0)
 			(effects
@@
 			)
 		)
-		(property "Footprint" ""
+		(property "Footprint" "Capacitor_SMD:C_0805_2012Metric"
 			(at 60.6552 158.75 0)
 			(effects
@@
 			(project "CM5IO"
 				(path "/e63e39d7-6ac0-4ffd-8aa3-1841a4541b55/a83afe30-5c7e-43cb-a5b2-f6f97a0812b3/a19d279d-385c-42b4-ac38-2ed1d04b4250"
-					(reference "C130")
+					(reference "C116")
 					(unit 1)
 				)
@@
 		(dnp no)
 		(fields_autoplaced yes)
-		(property "Reference" "#PWR0150"
+		(property "Reference" "#PWR0163"
 			(at 128.27 83.82 0)
 			(effects
@@
 			(project "CM5IO"
 				(path "/e63e39d7-6ac0-4ffd-8aa3-1841a4541b55/a83afe30-5c7e-43cb-a5b2-f6f97a0812b3/a19d279d-385c-42b4-ac38-2ed1d04b4250"
-					(reference "#PWR0150")
+					(reference "#PWR0163")
 					(unit 1)
 				)
@@
 		(dnp no)
 		(fields_autoplaced yes)
-		(property "Reference" "#PWR0149"
+		(property "Reference" "#PWR0161"
 			(at 27.94 88.9 0)
 			(effects
@@
 			(project "CM5IO"
 				(path "/e63e39d7-6ac0-4ffd-8aa3-1841a4541b55/a83afe30-5c7e-43cb-a5b2-f6f97a0812b3/a19d279d-385c-42b4-ac38-2ed1d04b4250"
-					(reference "#PWR0149")
+					(reference "#PWR0161")
 					(unit 1)
 				)
@@
 		(dnp no)
 		(fields_autoplaced yes)
-		(property "Reference" "C128"
+		(property "Reference" "C119"
 			(at 99.06 153.6699 0)
 			(effects
@@
 			)
 		)
-		(property "Footprint" ""
+		(property "Footprint" "Capacitor_SMD:C_0805_2012Metric"
 			(at 96.2152 158.75 0)
 			(effects
@@
 			(project "CM5IO"
 				(path "/e63e39d7-6ac0-4ffd-8aa3-1841a4541b55/a83afe30-5c7e-43cb-a5b2-f6f97a0812b3/a19d279d-385c-42b4-ac38-2ed1d04b4250"
-					(reference "C128")
+					(reference "C119")
 					(unit 1)
 				)
@@
 		(dnp no)
 		(fields_autoplaced yes)
-		(property "Reference" "#PWR0153"
+		(property "Reference" "#PWR0164"
 			(at 128.27 121.92 0)
 			(effects
@@
 			(project "CM5IO"
 				(path "/e63e39d7-6ac0-4ffd-8aa3-1841a4541b55/a83afe30-5c7e-43cb-a5b2-f6f97a0812b3/a19d279d-385c-42b4-ac38-2ed1d04b4250"
-					(reference "#PWR0153")
+					(reference "#PWR0164")
 					(unit 1)
 				)
@@
 		(dnp no)
 		(fields_autoplaced yes)
-		(property "Reference" "U64"
+		(property "Reference" "U60"
 			(at 104.14 88.9 0)
 			(effects
@@
 			)
 		)
-		(property "Footprint" "TS5A23157DGSR:SOP50P490X110-10N"
+		(property "Footprint" "CM5IO:SOP50P490X110-10N"
 			(at 104.14 109.22 0)
 			(effects
@@
 			(project "CM5IO"
 				(path "/e63e39d7-6ac0-4ffd-8aa3-1841a4541b55/a83afe30-5c7e-43cb-a5b2-f6f97a0812b3/a19d279d-385c-42b4-ac38-2ed1d04b4250"
-					(reference "U64")
+					(reference "U60")
 					(unit 1)
 				)
@@
 		(dnp no)
 		(fields_autoplaced yes)
-		(property "Reference" "#PWR0148"
+		(property "Reference" "#PWR0167"
 			(at 261.62 123.19 0)
 			(effects
@@
 			(project "CM5IO"
 				(path "/e63e39d7-6ac0-4ffd-8aa3-1841a4541b55/a83afe30-5c7e-43cb-a5b2-f6f97a0812b3/a19d279d-385c-42b4-ac38-2ed1d04b4250"
-					(reference "#PWR0148")
+					(reference "#PWR0167")
 					(unit 1)
 				)
@@
 		(dnp no)
 		(fields_autoplaced yes)
-		(property "Reference" "U63"
+		(property "Reference" "U59"
 			(at 104.14 50.8 0)
 			(effects
@@
 			)
 		)
-		(property "Footprint" "TS5A23157DGSR:SOP50P490X110-10N"
+		(property "Footprint" "CM5IO:SOP50P490X110-10N"
 			(at 104.14 71.12 0)
 			(effects
@@
 			(project "CM5IO"
 				(path "/e63e39d7-6ac0-4ffd-8aa3-1841a4541b55/a83afe30-5c7e-43cb-a5b2-f6f97a0812b3/a19d279d-385c-42b4-ac38-2ed1d04b4250"
-					(reference "U63")
+					(reference "U59")
 					(unit 1)
 				)
@@
 		(dnp no)
 		(fields_autoplaced yes)
-		(property "Reference" "C129"
+		(property "Reference" "C117"
 			(at 74.93 153.6699 0)
 			(effects
@@
 			)
 		)
-		(property "Footprint" ""
+		(property "Footprint" "Capacitor_SMD:C_0805_2012Metric"
 			(at 72.0852 158.75 0)
 			(effects
@@
 			(project "CM5IO"
 				(path "/e63e39d7-6ac0-4ffd-8aa3-1841a4541b55/a83afe30-5c7e-43cb-a5b2-f6f97a0812b3/a19d279d-385c-42b4-ac38-2ed1d04b4250"
-					(reference "C129")
+					(reference "C117")
 					(unit 1)
 				)
@@
 		(dnp no)
 		(fields_autoplaced yes)
-		(property "Reference" "R103"
+		(property "Reference" "R105"
 			(at 171.45 83.82 90)
 			(effects
@@
 			)
 		)
-		(property "Footprint" ""
+		(property "Footprint" "Resistor_SMD:R_0805_2012Metric"
 			(at 171.45 91.948 90)
 			(effects
@@
 			(project ""
 				(path "/e63e39d7-6ac0-4ffd-8aa3-1841a4541b55/a83afe30-5c7e-43cb-a5b2-f6f97a0812b3/a19d279d-385c-42b4-ac38-2ed1d04b4250"
-					(reference "R103")
+					(reference "R105")
 					(unit 1)
 				)
@@
 		(dnp no)
 		(fields_autoplaced yes)
-		(property "Reference" "#PWR0147"
+		(property "Reference" "#PWR0166"
 			(at 261.62 85.09 0)
 			(effects
@@
 			(project "CM5IO"
 				(path "/e63e39d7-6ac0-4ffd-8aa3-1841a4541b55/a83afe30-5c7e-43cb-a5b2-f6f97a0812b3/a19d279d-385c-42b4-ac38-2ed1d04b4250"
-					(reference "#PWR0147")
+					(reference "#PWR0166")
 					(unit 1)
 				)
@@
 		(on_board yes)
 		(dnp no)
-		(property "Reference" "#PWR0179"
+		(property "Reference" "#PWR0162"
 			(at 109.22 167.64 0)
 			(effects
@@
 			(project "CM5IO"
 				(path "/e63e39d7-6ac0-4ffd-8aa3-1841a4541b55/a83afe30-5c7e-43cb-a5b2-f6f97a0812b3/a19d279d-385c-42b4-ac38-2ed1d04b4250"
-					(reference "#PWR0179")
+					(reference "#PWR0162")
 					(unit 1)
 				)
@@
 		(dnp no)
 		(fields_autoplaced yes)
-		(property "Reference" "R105"
+		(property "Reference" "R104"
 			(at 38.1 82.55 90)
 			(effects
@@
 			)
 		)
-		(property "Footprint" ""
+		(property "Footprint" "Resistor_SMD:R_0805_2012Metric"
 			(at 38.1 90.678 90)
 			(effects
@@
 			(project "CM5IO"
 				(path "/e63e39d7-6ac0-4ffd-8aa3-1841a4541b55/a83afe30-5c7e-43cb-a5b2-f6f97a0812b3/a19d279d-385c-42b4-ac38-2ed1d04b4250"
-					(reference "R105")
+					(reference "R104")
 					(unit 1)
 				)
