File: Circuit/kicad/Robot fő nyák_v3/4x tmc5160.kicad_sch (KiCad schematic)
At the start: 28 parts, among them M6 Stepper_Motor_unipolar_6pin, M7 Stepper_Motor_unipolar_6pin, M8 Stepper_Motor_unipolar_6pin, M9 Stepper_Motor_unipolar_6pin, U49 TMC2240_SILENTSTEPSTICK, U50 TMC2240_SILENTSTEPSTICK, U51 TMC2240_SILENTSTEPSTICK, U52 TMC2240_SILENTSTEPSTICK

Commit message: readme updated kicad circuit V1
Parts:
- C97: renamed from C55; value C_Polarized -> 470uf; footprint Capacitor_SMD:C_0805_2012Metric -> Capacitor_SMD:CP_Elec_8x10
- D10, D11, D8, D9: footprint LED_SMD:LED_0603_1608Metric -> Diode_SMD:D_1206_3216Metric
- renumbered C54 to C96, C56 to C98, C57 to C99, M6 to M4, M7 to M5, M8 to M6, M9 to M7, R83 to R84, R84 to R85, R85 to R86, R86 to R87, R87 to R88, R88 to R89, R89 to R90, R90 to R91, R91 to R92, R92 to R93, R93 to R94, R94 to R95, U49 to U48, U50 to U49, U51 to U50, U52 to U51
Changed lines of the file:
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@@
 		(on_board yes)
 		(dnp no)
-		(property "Reference" "R84"
+		(property "Reference" "R85"
 			(at 41.91 41.91 90)
 			(effects
@@
 			(project "CM5IO"
 				(path "/e63e39d7-6ac0-4ffd-8aa3-1841a4541b55/a83afe30-5c7e-43cb-a5b2-f6f97a0812b3/f6ede07b-cbae-470e-ad72-e2de632e13c1"
-					(reference "R84")
+					(reference "R85")
 					(unit 1)
 				)
@@
 		(on_board yes)
 		(dnp no)
-		(property "Reference" "R91"
+		(property "Reference" "R92"
 			(at 240.03 40.64 90)
 			(effects
@@
 			(project "CM5IO"
 				(path "/e63e39d7-6ac0-4ffd-8aa3-1841a4541b55/a83afe30-5c7e-43cb-a5b2-f6f97a0812b3/f6ede07b-cbae-470e-ad72-e2de632e13c1"
-					(reference "R91")
+					(reference "R92")
 					(unit 1)
 				)
@@
 			)
 		)
-		(property "Footprint" "LED_SMD:LED_0603_1608Metric"
+		(property "Footprint" "Diode_SMD:D_1206_3216Metric"
 			(at 99.06 120.65 0)
 			(effects
@@
 		(dnp no)
 		(fields_autoplaced yes)
-		(property "Reference" "M8"
+		(property "Reference" "M6"
 			(at 240.03 62.649 0)
 			(effects
@@
 			(project "CM5IO"
 				(path "/e63e39d7-6ac0-4ffd-8aa3-1841a4541b55/a83afe30-5c7e-43cb-a5b2-f6f97a0812b3/f6ede07b-cbae-470e-ad72-e2de632e13c1"
-					(reference "M8")
+					(reference "M6")
 					(unit 1)
 				)
@@
 		(on_board yes)
 		(dnp no)
-		(property "Reference" "R88"
+		(property "Reference" "R89"
 			(at 120.65 114.3 90)
 			(effects
@@
 			(project "CM5IO"
 				(path "/e63e39d7-6ac0-4ffd-8aa3-1841a4541b55/a83afe30-5c7e-43cb-a5b2-f6f97a0812b3/f6ede07b-cbae-470e-ad72-e2de632e13c1"
-					(reference "R88")
+					(reference "R89")
 					(unit 1)
 				)
@@
 		(on_board yes)
 		(dnp no)
-		(property "Reference" "R89"
+		(property "Reference" "R90"
 			(at 173.99 41.91 90)
 			(effects
@@
 			(project "CM5IO"
 				(path "/e63e39d7-6ac0-4ffd-8aa3-1841a4541b55/a83afe30-5c7e-43cb-a5b2-f6f97a0812b3/f6ede07b-cbae-470e-ad72-e2de632e13c1"
-					(reference "R89")
+					(reference "R90")
 					(unit 1)
 				)
@@
 		(dnp no)
 		(fields_autoplaced yes)
-		(property "Reference" "M7"
+		(property "Reference" "M5"
 			(at 106.68 136.309 0)
 			(effects
@@
 			(project "CM5IO"
 				(path "/e63e39d7-6ac0-4ffd-8aa3-1841a4541b55/a83afe30-5c7e-43cb-a5b2-f6f97a0812b3/f6ede07b-cbae-470e-ad72-e2de632e13c1"
-					(reference "M7")
+					(reference "M5")
 					(unit 1)
 				)
@@
 		(dnp no)
 		(fields_autoplaced yes)
-		(property "Reference" "C55"
+		(property "Reference" "C97"
 			(at 78.74 110.1089 0)
 			(effects
@@
 			)
 		)
-		(property "Value" "C_Polarized"
+		(property "Value" "470uf"
 			(at 78.74 112.6489 0)
 			(effects
@@
 			)
 		)
-		(property "Footprint" "Capacitor_SMD:C_0805_2012Metric"
+		(property "Footprint" "Capacitor_SMD:CP_Elec_8x10"
 			(at 73.9648 106.68 0)
 			(effects
@@
 			(project "CM5IO"
 				(path "/e63e39d7-6ac0-4ffd-8aa3-1841a4541b55/a83afe30-5c7e-43cb-a5b2-f6f97a0812b3/f6ede07b-cbae-470e-ad72-e2de632e13c1"
-					(reference "C55")
+					(reference "C97")
 					(unit 1)
 				)
@@
 			)
 		)
-		(property "Footprint" "LED_SMD:LED_0603_1608Metric"
+		(property "Footprint" "Diode_SMD:D_1206_3216Metric"
 			(at 232.41 120.65 0)
 			(effects
@@
 		(on_board yes)
 		(dnp no)
-		(property "Reference" "R83"
+		(property "Reference" "R84"
 			(at 40.64 115.57 90)
 			(effects
@@
 			(project "CM5IO"
 				(path "/e63e39d7-6ac0-4ffd-8aa3-1841a4541b55/a83afe30-5c7e-43cb-a5b2-f6f97a0812b3/f6ede07b-cbae-470e-ad72-e2de632e13c1"
-					(reference "R83")
+					(reference "R84")
 					(unit 1)
 				)
@@
 		(on_board yes)
 		(dnp no)
-		(property "Reference" "R86"
+		(property "Reference" "R87"
 			(at 106.68 114.3 90)
 			(effects
@@
 			(project "CM5IO"
 				(path "/e63e39d7-6ac0-4ffd-8aa3-1841a4541b55/a83afe30-5c7e-43cb-a5b2-f6f97a0812b3/f6ede07b-cbae-470e-ad72-e2de632e13c1"
-					(reference "R86")
+					(reference "R87")
 					(unit 1)
 				)
@@
 		(on_board yes)
 		(dnp no)
-		(property "Reference" "R94"
+		(property "Reference" "R95"
 			(at 254 114.3 90)
 			(effects
@@
 			(project "CM5IO"
 				(path "/e63e39d7-6ac0-4ffd-8aa3-1841a4541b55/a83afe30-5c7e-43cb-a5b2-f6f97a0812b3/f6ede07b-cbae-470e-ad72-e2de632e13c1"
-					(reference "R94")
+					(reference "R95")
 					(unit 1)
 				)
@@
 		(on_board yes)
 		(dnp no)
-		(property "Reference" "R92"
+		(property "Reference" "R93"
 			(at 240.03 114.3 90)
 			(effects
@@
 			(project "CM5IO"
 				(path "/e63e39d7-6ac0-4ffd-8aa3-1841a4541b55/a83afe30-5c7e-43cb-a5b2-f6f97a0812b3/f6ede07b-cbae-470e-ad72-e2de632e13c1"
-					(reference "R92")
+					(reference "R93")
 					(unit 1)
 				)
@@
 		(dnp no)
 		(fields_autoplaced yes)
-		(property "Reference" "M6"
+		(property "Reference" "M4"
 			(at 106.68 62.649 0)
 			(effects
@@
 			(project "CM5IO"
 				(path "/e63e39d7-6ac0-4ffd-8aa3-1841a4541b55/a83afe30-5c7e-43cb-a5b2-f6f97a0812b3/f6ede07b-cbae-470e-ad72-e2de632e13c1"
-					(reference "M6")
+					(reference "M4")
 					(unit 1)
 				)
@@
 		(on_board yes)
 		(dnp no)
-		(property "Reference" "R87"
+		(property "Reference" "R88"
 			(at 120.65 40.64 90)
 			(effects
@@
 			(project "CM5IO"
 				(path "/e63e39d7-6ac0-4ffd-8aa3-1841a4541b55/a83afe30-5c7e-43cb-a5b2-f6f97a0812b3/f6ede07b-cbae-470e-ad72-e2de632e13c1"
-					(reference "R87")
+					(reference "R88")
 					(unit 1)
 				)
@@
 		(dnp no)
 		(fields_autoplaced yes)
-		(property "Reference" "C56"
+		(property "Reference" "C98"
 			(at 212.09 36.4489 0)
 			(effects
@@
 			(project "CM5IO"
 				(path "/e63e39d7-6ac0-4ffd-8aa3-1841a4541b55/a83afe30-5c7e-43cb-a5b2-f6f97a0812b3/f6ede07b-cbae-470e-ad72-e2de632e13c1"
-					(reference "C56")
+					(reference "C98")
 					(unit 1)
 				)
@@
 		(on_board yes)
 		(dnp no)
-		(property "Reference" "R85"
+		(property "Reference" "R86"
 			(at 106.68 40.64 90)
 			(effects
@@
 			(project "CM5IO"
 				(path "/e63e39d7-6ac0-4ffd-8aa3-1841a4541b55/a83afe30-5c7e-43cb-a5b2-f6f97a0812b3/f6ede07b-cbae-470e-ad72-e2de632e13c1"
-					(reference "R85")
+					(reference "R86")
 					(unit 1)
 				)
@@
 		(on_board yes)
 		(dnp no)
-		(property "Reference" "R93"
+		(property "Reference" "R94"
 			(at 254 40.64 90)
 			(effects
@@
 			(project "CM5IO"
 				(path "/e63e39d7-6ac0-4ffd-8aa3-1841a4541b55/a83afe30-5c7e-43cb-a5b2-f6f97a0812b3/f6ede07b-cbae-470e-ad72-e2de632e13c1"
-					(reference "R93")
+					(reference "R94")
 					(unit 1)
 				)
@@
 		(dnp no)
 		(fields_autoplaced yes)
-		(property "Reference" "U49"
+		(property "Reference" "U48"
 			(at 57.15 36.83 0)
 			(effects
@@
 			(project "CM5IO"
 				(path "/e63e39d7-6ac0-4ffd-8aa3-1841a4541b55/a83afe30-5c7e-43cb-a5b2-f6f97a0812b3/f6ede07b-cbae-470e-ad72-e2de632e13c1"
-					(reference "U49")
+					(reference "U48")
 					(unit 1)
 				)
@@
 		(dnp no)
 		(fields_autoplaced yes)
-		(property "Reference" "U52"
+		(property "Reference" "U51"
 			(at 190.5 110.49 0)
 			(effects
@@
 			(project "CM5IO"
 				(path "/e63e39d7-6ac0-4ffd-8aa3-1841a4541b55/a83afe30-5c7e-43cb-a5b2-f6f97a0812b3/f6ede07b-cbae-470e-ad72-e2de632e13c1"
-					(reference "U52")
+					(reference "U51")
 					(unit 1)
 				)
@@
 		(dnp no)
 		(fields_autoplaced yes)
-		(property "Reference" "C54"
+		(property "Reference" "C96"
 			(at 78.74 36.4489 0)
 			(effects
@@
 			(project "CM5IO"
 				(path "/e63e39d7-6ac0-4ffd-8aa3-1841a4541b55/a83afe30-5c7e-43cb-a5b2-f6f97a0812b3/f6ede07b-cbae-470e-ad72-e2de632e13c1"
-					(reference "C54")
+					(reference "C96")
 					(unit 1)
 				)
@@
 		(dnp no)
 		(fields_autoplaced yes)
-		(property "Reference" "U50"
+		(property "Reference" "U49"
 			(at 57.15 110.49 0)
 			(effects
@@
 			(project "CM5IO"
 				(path "/e63e39d7-6ac0-4ffd-8aa3-1841a4541b55/a83afe30-5c7e-43cb-a5b2-f6f97a0812b3/f6ede07b-cbae-470e-ad72-e2de632e13c1"
-					(reference "U50")
+					(reference "U49")
 					(unit 1)
 				)
@@
 		(on_board yes)
 		(dnp no)
-		(property "Reference" "R90"
+		(property "Reference" "R91"
 			(at 173.99 115.57 90)
 			(effects
@@
 			(project "CM5IO"
 				(path "/e63e39d7-6ac0-4ffd-8aa3-1841a4541b55/a83afe30-5c7e-43cb-a5b2-f6f97a0812b3/f6ede07b-cbae-470e-ad72-e2de632e13c1"
-					(reference "R90")
+					(reference "R91")
 					(unit 1)
 				)
@@
 		(dnp no)
 		(fields_autoplaced yes)
-		(property "Reference" "U51"
+		(property "Reference" "U50"
 			(at 190.5 36.83 0)
 			(effects
@@
 			(project "CM5IO"
 				(path "/e63e39d7-6ac0-4ffd-8aa3-1841a4541b55/a83afe30-5c7e-43cb-a5b2-f6f97a0812b3/f6ede07b-cbae-470e-ad72-e2de632e13c1"
-					(reference "U51")
+					(reference "U50")
 					(unit 1)
 				)
@@
 		(dnp no)
 		(fields_autoplaced yes)
-		(property "Reference" "M9"
+		(property "Reference" "M7"
 			(at 240.03 136.309 0)
 			(effects
@@
 			(project "CM5IO"
 				(path "/e63e39d7-6ac0-4ffd-8aa3-1841a4541b55/a83afe30-5c7e-43cb-a5b2-f6f97a0812b3/f6ede07b-cbae-470e-ad72-e2de632e13c1"
-					(reference "M9")
+					(reference "M7")
 					(unit 1)
 				)
@@
 		(dnp no)
 		(fields_autoplaced yes)
-		(property "Reference" "C57"
+		(property "Reference" "C99"
 			(at 212.09 110.1089 0)
 			(effects
@@
 			(project "CM5IO"
 				(path "/e63e39d7-6ac0-4ffd-8aa3-1841a4541b55/a83afe30-5c7e-43cb-a5b2-f6f97a0812b3/f6ede07b-cbae-470e-ad72-e2de632e13c1"
-					(reference "C57")
+					(reference "C99")
 					(unit 1)
 				)
@@
 			)
 		)
-		(property "Footprint" "LED_SMD:LED_0603_1608Metric"
+		(property "Footprint" "Diode_SMD:D_1206_3216Metric"
 			(at 99.06 46.99 0)
 			(effects
@@
 			)
 		)
-		(property "Footprint" "LED_SMD:LED_0603_1608Metric"
+		(property "Footprint" "Diode_SMD:D_1206_3216Metric"
 			(at 232.41 46.99 0)
 			(effects

Commit message: kicad 2 panel_0.1
Parts:
- C96, C98, C99: footprint Capacitor_SMD:C_0805_2012Metric -> Capacitor_SMD:CP_Elec_8x10
Changed lines of the file:
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@@
 			)
 		)
-		(property "Footprint" "Capacitor_SMD:C_0805_2012Metric"
+		(property "Footprint" "Capacitor_SMD:CP_Elec_8x10"
 			(at 207.3148 33.02 0)
 			(effects
@@
 			)
 		)
-		(property "Footprint" "Capacitor_SMD:C_0805_2012Metric"
+		(property "Footprint" "Capacitor_SMD:CP_Elec_8x10"
 			(at 73.9648 33.02 0)
 			(effects
@@
 			)
 		)
-		(property "Footprint" "Capacitor_SMD:C_0805_2012Metric"
+		(property "Footprint" "Capacitor_SMD:CP_Elec_8x10"
 			(at 207.3148 106.68 0)
 			(effects

Commit message: updated kicad (big_update)
Parts:
- R86, R87, R92, R93: value 320 -> 330
Changed lines of the file:
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@@
 			)
 		)
-		(property "Value" "320"
+		(property "Value" "330"
 			(at 240.03 43.18 90)
 			(effects
@@
 			)
 		)
-		(property "Value" "320"
+		(property "Value" "330"
 			(at 106.68 116.84 90)
 			(effects
@@
 			)
 		)
-		(property "Value" "320"
+		(property "Value" "330"
 			(at 240.03 116.84 90)
 			(effects
@@
 			)
 		)
-		(property "Value" "320"
+		(property "Value" "330"
 			(at 106.68 43.18 90)
 			(effects
