File: Circuit/kicad/Robot fő nyák_v3/ADS8688 .kicad_sch (KiCad schematic)
At the start: 2 parts, among them U56 ICM-45686

Commit message: kicad update new readme media updates the circuit is 95% finished
Parts:
- removed C58: 1uf, Capacitor_SMD:C_0805_2012Metric, symbol Device:C
- removed U56: ICM-45686, CM5IO:IC_ICM-45686, symbol icm:ICM-45686
- added U67: ADS8688, Package_SO:TSSOP-38_4.4x9.7mm_P0.5mm, symbol Analog_ADC:ADS8688
Connections:
- new net: U67.28 (AGND), U67.29 (AGND), U67.31 (AGND), U67.32 (AGND), U67.8 (AGND)
- no-connect marks 7 -> 0

Commit message: readme updated kicad circuit V1
Parts:
- renumbered U67 to U63
Changed lines of the file:
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@@
 		(dnp no)
 		(fields_autoplaced yes)
-		(property "Reference" "U67"
+		(property "Reference" "U63"
 			(at 98.6633 92.71 0)
 			(effects
@@
 			(project ""
 				(path "/e63e39d7-6ac0-4ffd-8aa3-1841a4541b55/a83afe30-5c7e-43cb-a5b2-f6f97a0812b3/86209e6a-92ae-4699-a125-02d46b525fc7/c41f5f78-bb85-4895-95b0-27817ef7b3b3"
-					(reference "U67")
+					(reference "U63")
 					(unit 1)
 				)

Commit message: updated kicad (big_update)
Parts:
- removed U63: ADS8688, Package_SO:TSSOP-38_4.4x9.7mm_P0.5mm, symbol Analog_ADC:ADS8688
- added C39: 68pf, Capacitor_SMD:C_0805_2012Metric, symbol Device:C
- added C42: 100nf, Capacitor_SMD:C_0805_2012Metric, symbol Device:C
- added J17, J18, J21, J22, J23, J24: Conn_01x02_Pin, Connector_PinHeader_2.54mm:PinHeader_2x01_P2.54mm_Vertical, symbol Connector:Conn_01x02_Pin
- added R101, R102, R155, R156, R157, R158: 10k, Resistor_SMD:R_0805_2012Metric, symbol Device:R
- added U47: MCP3208, Package_SO:SOIC-16_3.9x9.9mm_P1.27mm, symbol Analog_ADC:MCP3208
- added U58: MCP1541-TT, Package_TO_SOT_SMD:SOT-23, symbol Reference_Voltage:MCP1541-TT
Connections:
- new net: J17.1 (Pin_1), R156.2
- new net: C39.2, C42.1, U47.15 (Vref), U58.2 (Vout)
- new net: J21.1 (Pin_1), R155.2
- new net: J23.1 (Pin_1), R101.2
- new net: J23.2 (Pin_2), U47.5 (CH4)
- new net: J24.1 (Pin_1), R102.2
- new net: J24.2 (Pin_2), U47.6 (CH5)
- new net: J18.1 (Pin_1), R157.2
- new net: J17.2 (Pin_2), U47.2 (CH1)
- new net: J21.2 (Pin_2), U47.1 (CH0)
- new net: J18.2 (Pin_2), U47.3 (CH2)
- new net: J22.2 (Pin_2), U47.4 (CH3)
- new net: J22.1 (Pin_1), R158.2
- new net 5v: R101.1, R102.1, R155.1, R156.1, R157.1, R158.1, U47.16 (Vdd), U58.1 (Vin)
- new net CS: U47.10 (~{CS}/SHDN)
- new net GND: C39.1, C42.2, U47.14 (AGND), U47.9 (DGND), U58.3 (Vss)
- new net MISO: U47.12 (Dout)
- new net MOSI: U47.11 (Din)
- new net SPI_CLK: U47.13 (CLK)
