File: Circuit/kicad/Robot fő nyák_v3/CM5IO.kicad_pcb (KiCad board)
At the start: 6 copper layers, 473 parts, among them J1 XT60-M, J10 USB_C_Receptacle_USB2.0_16P, J11 THD-02-R, J12 Conn_01x04_Socket, J13 THD-02-R, J2 USB3_A, J3 690-019-298-412, J31 Conn_01x02_Pin, J32 Conn_01x02_Pin, J4 690-019-298-412, J5 MagJack-A70-112-331N126, J6 Bus_M.2_Socket_M, J7 690-008-221-904, J8 USB_C_Receptacle_USB2.0_16P, J9 USB_C_Receptacle_USB2.0_16P, M4 Stepper_Motor_unipolar_6pin, M5 Stepper_Motor_unipolar_6pin, M6 Stepper_Motor_unipolar_6pin, M7 Stepper_Motor_unipolar_6pin, Q1 IRLHM630PbF, Q10 IRLML2502, Q11 IRLML2502, Q12 IRLML2502, Q13 IRLML2502, Q14 IRLML2502, Q15 IRLML2502, Q16 IRLML2502, Q17 IRLML2502, Q18 IRLML2502, Q19 IRLML2502, Q2 SS8050-G, Q20 IRLML2502, Q21 IRLML2502, Q22 IRLML2502, Q23 IRLML2502, Q24 IRLML2502, Q25 IRLML2502, Q26 IRLHM630PbF, Q3 SS8050-G, Q4 IRLML2502, Q5 IRLML2502, Q6 IRLML2502, Q7 IRLML2502, Q8 IRLML2502, Q9 IRLML2502, SW1 Right angle Tact button, SW2 SW_Push, SW3 SW_Push, SW4 SW_Push, U1 AP22653W6, U10 TPD4EUSB30, U11 USB2514B-I/M2, U12 TPD4EUSB30, U13 FSUSB42MUX, U14 TPD4EUSB30, U15 INA226, U16 INA226, U17 INA226, U18 INA226, U19 INA226, U2 RT9742SNGV, U20 INA226, U21 INA226, U22 INA226, U23 INA226, U24 INA226, U25 INA226, U26 INA226, U27 INA226, U28 INA226, U29 INA226, U3 74LVC1G07SE-7, U30 INA226, U31 AP64501SP-13, U32 AP64501SP-13, U33 AP64501SP-13, U34 AP64501SP-13, U35 AP64501SP-13, U37 CH343P, U4 TPD4EUSB30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

Commit message: kicad pcb v1.0
Parts:
- removed the C5 at (-445.1, 282.2)
- removed the C6 at (-445.1, 285.2)
- removed the R75 at (428.4, 64.6)
- removed the R76 at (428.4, 67.5)
- removed the R77 at (428.4, 70.5)
- removed the R78 at (428.4, 73.5)
- removed the R79 at (428.4, 76.4)
- removed the R80 at (428.4, 79.3)
- removed the R81 at (428.4, 82.3)
- removed the R82 at (432.8, 64.6)
- removed the R83 at (432.8, 67.5)
- removed the U2 at (-440.1, 283.1)
- added C88: 1uf, Capacitor_SMD:C_0805_2012Metric, B.Cu at (308.0, 210.0)
- added C89: 1uf, Capacitor_SMD:C_0805_2012Metric, B.Cu at (220.0, 271.0)
- added C90: 1uf, Capacitor_SMD:C_0805_2012Metric, B.Cu at (205.0, 271.0)
- added C92: 1uf, Capacitor_SMD:C_0805_2012Metric, F.Cu at (263.0, 223.0)
- added C93: 1uf, Capacitor_SMD:C_0805_2012Metric, F.Cu at (292.0, 223.0)
- added C94: 1uf, Capacitor_SMD:C_0805_2012Metric, F.Cu at (292.0, 220.0)
- added C95: 1uf, Capacitor_SMD:C_0805_2012Metric, F.Cu at (252.0, 192.0)
- added D11: LED, Diode_SMD:D_1206_3216Metric, F.Cu at (348.0, 242.0)
- added HS1: Heatsink, TestPoint:TestPoint_Pad_1.0x1.0mm, B.Cu at (252.8, 107.3)
- added R100: 100k, Resistor_SMD:R_0805_2012Metric, B.Cu at (260.0, 234.0)
- added R101: 100k, Resistor_SMD:R_0805_2012Metric, B.Cu at (264.0, 237.0)
- added R102: 100k, Resistor_SMD:R_0805_2012Metric, B.Cu at (289.0, 243.0)
- added R103: 100k, Resistor_SMD:R_0805_2012Metric, B.Cu at (274.0, 224.0)
- added R87: 320, Resistor_SMD:R_0805_2012Metric, B.Cu at (313.0, 191.0)
- added R88: 10k, Resistor_SMD:R_0805_2012Metric, B.Cu at (269.0, 221.0)
- added R89: 10k, Resistor_SMD:R_0805_2012Metric, B.Cu at (285.0, 231.0)
- added R90: 10k, Resistor_SMD:R_0805_2012Metric, B.Cu at (272.0, 230.0)
- added R91: 10k, Resistor_SMD:R_0805_2012Metric, B.Cu at (275.0, 215.0)
- added R92: 320, Resistor_SMD:R_0805_2012Metric, B.Cu at (284.0, 243.0)
- added R93: 320, Resistor_SMD:R_0805_2012Metric, B.Cu at (275.0, 218.0)
- added R94: 10k, Resistor_SMD:R_0805_2012Metric, B.Cu at (285.0, 252.0)
- added R95: 10k, Resistor_SMD:R_0805_2012Metric, B.Cu at (274.0, 246.0)
- added R96: 2.2K 1%, Resistor_SMD:R_0805_2012Metric, B.Cu at (285.0, 255.0)
- added R97: 2.2K 1%, Resistor_SMD:R_0805_2012Metric, B.Cu at (280.0, 257.0)
- added R98: 100k, Resistor_SMD:R_0805_2012Metric, B.Cu at (273.0, 267.0)
- added R99: 100k, Resistor_SMD:R_0805_2012Metric, B.Cu at (285.0, 237.0)
- added U36: RT9742SNGV, Package_TO_SOT_SMD:TSOT-23, B.Cu at (218.0, 285.0)
- added U6: AP22653W6, Package_TO_SOT_SMD:SOT-23-6, B.Cu at (219.0, 275.0)
- added U63: ADS8688, Package_SO:TSSOP-38_4.4x9.7mm_P0.5mm, B.Cu at (337.0, 209.0)
- added U66: TS5A23157DGSR, CM5IO:SOP50P490X110-10N, F.Cu at (287.0, 253.0)
- C1, C100, C101, C102, C103, C104, C105, C106, C107, C108, C109, C110, C111, C112, C113, C116, C117, C118, C119, C12, C120, C121, C122, C123, C124, C125, C126, C127, C128, C129, C13, C130, C131, C132, C133, C134, C135, C136, C137, C139, C14, C140, C141, C142, C143, C15, C16, C17, C18, C19, C20, C21, C22, C23, C24, C25, C26, C27, C28, C29, C3, C30, C31, C32, C33, C34, C35, C36, C37, C4, C41, C42, C43, C44, C45, C46, C47, C48, C49, C50, C51, C52, C53, C54, C55, C56, C57, C58, C59, C60, C61, C64, C65, C66, C67, C68, C69, C70, C71, C72, C73, C74, C75, C76, C77, CT2, CT4, CT5, CT6, CT7, CT8, CT9, FB1, L1, L2, L3, L4, L5, Q10, Q11, Q12, Q13, Q14, Q15, Q16, Q17, Q18, Q20, Q21, Q22, Q23, Q24, Q25, Q4, Q5, Q6, Q7, Q8, Q9, R1, R104, R105, R106, R107, R108, R109, R110, R111, R112, R113, R114, R115, R116, R117, R118, R119, R120, R121, R122, R123, R124, R125, R126, R127, R128, R129, R130, R131, R132, R133, R134, R135, R136, R137, R138, R139, R140, R141, R142, R143, R144, R16, R17, R18, R19, R2, R20, R21, R22, R23, R24, R25, R26, R27, R28, R29, R3, R30, R31, R32, R33, R34, R35, R36, R37, R39, R4, R40, R41, R42, R43, R44, R45, R46, R48, R49, R50, R51, R52, R53, R54, R55, R56, R57, R58, R59, R60, R61, R62, R63, R64, R65, R66, R67, R68, R85, SW1, TP10, TP11, TP12, TP13, TP14, TP15, TP16, TP4, TP9, U10, U11, U12, U13, U14, U15, U16, U17, U18, U19, U21, U22, U23, U24, U25, U26, U27, U28, U30, U31, U32, U33, U34, U35, U45, U46, U47, U52, U53, U54, U55, U56, U57, U59, U60, U61, U62, U64, U65, U67, U8, U9, Y1, Y3, Y4: moved to B.Cu
- C2: renamed from C94; value 1uf -> 100uF; footprint Capacitor_SMD:C_0805_2012Metric -> Capacitor_Tantalum_SMD:CP_EIA-7343-31_Kemet-D; moved to B.Cu
- C38: renamed from C88; moved to B.Cu
- C39: renamed from C95; moved to B.Cu
- C40: renamed from C85; moved to B.Cu
- C5: renamed from C86; value 1uf -> 100n; moved to B.Cu
- C6: renamed from C89; value 1uf -> 100n; moved to B.Cu
- C62: renamed from C93; moved to B.Cu
- C63: renamed from C87; moved to B.Cu
- C85: renamed from C92; moved to B.Cu
- C86: renamed from C91; moved to B.Cu
- C87: renamed from C90; moved to B.Cu
- C91: renamed from C2; value 100uF -> 1uf; footprint Capacitor_Tantalum_SMD:CP_EIA-7343-31_Kemet-D -> Capacitor_SMD:C_0805_2012Metric; moved to B.Cu
- D10: renamed from D9; moved to B.Cu
- D7: renamed from D11; moved to B.Cu
- D8: renamed from D10; moved to B.Cu
- D9: renamed from D8; moved to B.Cu
- R75: renamed from R90; moved to B.Cu
- R76: renamed from R87; value 320 -> 100k; moved to B.Cu
- R77: renamed from R94; value 10k -> 100k; moved to B.Cu
- R78: renamed from R95; value 10k -> 100k; moved to B.Cu
- R79: renamed from R91; value 10k -> 100k; moved to B.Cu
- R80: renamed from R86; value 320 -> 100k; moved to B.Cu
- R81: renamed from R93; value 320 -> 100k; moved to B.Cu
- R82: renamed from R84; value 10k -> 100k; moved to B.Cu
- R83: renamed from R92; value 320 -> 100k; moved to B.Cu
- R84: renamed from R88; moved to B.Cu
- R86: renamed from R89; value 10k -> 320; moved to B.Cu
- TP3: footprint TestPoint:TestPoint_Pad_2.0x2.0mm -> TestPoint:TestPoint_Pad_D2.0mm
- TP5, TP6: footprint TestPoint:TestPoint_Pad_D2.0mm -> TestPoint:TestPoint_Pad_D4.0mm
- U2: renamed from U66; value TS5A23157DGSR -> RT9742SNGV; footprint CM5IO:SOP50P490X110-10N -> Package_TO_SOT_SMD:TSOT-23; moved to B.Cu
- moved R7 851.3 mm to (274.7, 261.5), turned to 90 degrees
- moved R13 850.0 mm to (282.2, 261.5), turned to 90 degrees
- moved R10 849.4 mm to (277.2, 261.5), turned to 90 degrees
- moved R6 848.8 mm to (272.2, 261.5), turned to 90 degrees
- moved J13 848.7 mm to (285.5, 264.6)
- moved R12 847.4 mm to (279.7, 261.5), turned to 90 degrees
- moved R5 846.3 mm to (269.8, 261.5), turned to 90 degrees
- moved J5 846.0 mm to (276.7, 279.8)
- moved R11 845.0 mm to (277.2, 257.7), turned to 90 degrees
- moved U4 840.8 mm to (281.9, 266.4), turned to -90 degrees
- moved BT1 840.4 mm to (263.2, 244.3), turned to 90 degrees
- moved DSW2 838.0 mm to (263.2, 266.1)
- moved GPIO1 837.3 mm to (253.3, 222.1)
- moved C7 835.4 mm to (277.2, 266.7), turned to 90 degrees
- moved R9 832.0 mm to (259.2, 237.9), turned to 90 degrees
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Connections:
- C103 pad 1: ESP_5v -> ESP_3v3
- C104 pad 1: ESP_5v -> ESP_3v3
- C105 pad 1: ESP_5v -> ESP_3v3
- C2 pad 1: ESP_5v -> /CM5_HighSpeed/VBUS
- C5 pad 1: /YD-ESP32-S3/I2C_devices/output_pin_2 -> 5V1
- C6 pad 1: /YD-ESP32-S3/I2C_devices/output_pin_5 -> /CM5_HighSpeed/HDMI_5v
- C85 pad 1: /YD-ESP32-S3/I2C_devices/output_pin_8 -> /YD-ESP32-S3/I2C_devices/output_pin_1
- C86 pad 1: /YD-ESP32-S3/I2C_devices/output_pin_7 -> /YD-ESP32-S3/I2C_devices/output_pin_2
- C87 pad 1: /YD-ESP32-S3/I2C_devices/output_pin_6 -> /YD-ESP32-S3/I2C_devices/output_pin_3
- C91 pad 1: /CM5_HighSpeed/VBUS -> /YD-ESP32-S3/I2C_devices/output_pin_7
- CT6 pad 1: ESP_5v -> ESP_3v3
- D10 pad 1: Net-(D9-K) -> Net-(D10-K)
- D10 pad 2: Net-(D9-A) -> Net-(D10-A)
- D4 pad 1: unconnected-(D4-K-Pad1) -> GND
- D8 pad 1: Net-(D10-K) -> Net-(D8-K)
- D8 pad 2: Net-(D10-A) -> Net-(D8-A)
- D9 pad 1: Net-(D8-K) -> Net-(D9-K)
- D9 pad 2: Net-(D8-A) -> Net-(D9-A)
- Q21 pad 3: unconnected-(Q21-D-Pad3) -> ESP_3v3
- Q24 pad 3: unconnected-(Q24-D-Pad3) -> ESP_3v3
- R75 pad 1: /YD-ESP32-S3/4x tmc5161/M2_EN -> ESP_5v
- R75 pad 2: /YD-ESP32-S3/4x tmc5161/TMC_GND -> /YD-ESP32-S3/I2C_devices/I2C_RST
- R76 pad 1: Net-(D9-A) -> GND
- R76 pad 2: ESP_3v3 -> /YD-ESP32-S3/I2C_devices/Sw1
- R77 pad 1: Net-(D10-K) -> GND
- R77 pad 2: ESP_3v3 -> /YD-ESP32-S3/I2C_devices/Sw3
- R78 pad 1: Net-(D11-K) -> GND
- R78 pad 2: ESP_3v3 -> /YD-ESP32-S3/I2C_devices/Sw5
- R79 pad 1: /YD-ESP32-S3/4x tmc5161/M4_EN -> GND
- R79 pad 2: /YD-ESP32-S3/4x tmc5161/TMC_GND -> /YD-ESP32-S3/I2C_devices/Sw7
- R80 pad 1: Net-(D8-A) -> GND
- R80 pad 2: ESP_3v3 -> /YD-ESP32-S3/I2C_devices/Sw2
- R81 pad 1: Net-(D11-A) -> GND
- R81 pad 2: ESP_3v3 -> /YD-ESP32-S3/I2C_devices/Sw4
- R82 pad 1: /YD-ESP32-S3/4x tmc5161/M3_EN -> GND
- R82 pad 2: /YD-ESP32-S3/4x tmc5161/TMC_GND -> /YD-ESP32-S3/I2C_devices/Sw6
- R83 pad 1: Net-(D10-A) -> GND
- R83 pad 2: ESP_3v3 -> /YD-ESP32-S3/I2C_devices/Sw8
- R84 pad 1: Net-(D8-K) -> /YD-ESP32-S3/4x tmc5161/M3_EN
- R84 pad 2: ESP_3v3 -> /YD-ESP32-S3/4x tmc5161/TMC_GND
- R86 pad 1: Net-(D9-K) -> Net-(D8-A)
- TP3 pad 1: Net-(D2-K) -> GND
- U2 pad 1: I2C_CH -> 5V1
- U2 pad 2: INA226_SDA -> /CM5_HighSpeed/HDMI_5v
- U53 pad 9: unconnected-(U53-VDD-Pad9) -> ESP_3v3
- U54 pad 9: unconnected-(U54-VDD-Pad9) -> ESP_3v3
Routing:
- net ESP_3v3: track 0.00 -> 296.4 mm, vias 0 -> 16
- net /12v_1: track 0.00 -> 214.2 mm, vias 0 -> 8
- net SERVO2: track 0.00 -> 107.5 mm, vias 0 -> 2
- net SERVO4: track 0.00 -> 92.7 mm, vias 0 -> 1
- net SERVO3: track 0.00 -> 83.0 mm, vias 0 -> 1
- net SERVO1: track 0.00 -> 65.6 mm, vias 0 -> 1
- net Net-(U35-SW): track 0.00 -> 51.5 mm, vias 0 -> 2
- net Net-(U31-SW): track 0.00 -> 33.4 mm
- net Net-(U32-SW): track 0.00 -> 28.2 mm, vias 0 -> 2
- net /YD-ESP32-S3/I2C_devices/output_pin_3: track 0.00 -> 20.7 mm
- net /YD-ESP32-S3/SPI_2_MOSI: track 0.00 -> 19.9 mm
- net /YD-ESP32-S3/SPI_2_MISO: track 0.00 -> 19.9 mm
- net /YD-ESP32-S3/SPI_2_CLK: track 0.00 -> 19.9 mm
- net Net-(C65-Pad1): track 0.00 -> 9.30 mm
- net /YD-ESP32-S3/I2C_devices/output_pin_7: track 0.00 -> 6.60 mm
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Other:
- board outline added: 155 x 100 mm

Commit message: kicad 2 panel_0.1
Parts:
- removed C38, C39, C40, C62, C63: 1uf, Capacitor_SMD:C_0805_2012Metric
- removed D7: LED, Diode_SMD:D_1206_3216Metric
- removed GPIO2: Conn_02x14_Counter_Clockwise, Connector_PinHeader_2.54mm:PinHeader_2x14_P2.54mm_Vertical
- removed the HS1 at (252.8, 107.3)
- removed R100, R101, R102, R103, R98, R99: 100k, Resistor_SMD:R_0805_2012Metric
- removed R96, R97: 2.2K 1%, Resistor_SMD:R_0805_2012Metric
- removed U36: RT9742SNGV, Package_TO_SOT_SMD:TSOT-23
- removed U6: AP22653W6, Package_TO_SOT_SMD:SOT-23-6
- added HS1: Heatsink, TestPoint:TestPoint_Pad_1.0x1.0mm, F.Cu at (521.1, 126.6)
- added HS1: Heatsink, TestPoint:TestPoint_Pad_1.0x1.0mm, B.Cu at (116.7, 357.4)
- added J14: Conn_02x20_Odd_Even, Connector_PinHeader_2.54mm:PinHeader_2x20_P2.54mm_Vertical, F.Cu at (341.4, 123.6)
- added J15: Conn_02x20_Odd_Even, Connector_PinHeader_2.54mm:PinHeader_2x20_P2.54mm_Vertical, F.Cu at (210.4, 224.1)
- added J16: Conn_01x12, Connector_PinSocket_2.54mm:PinSocket_1x12_P2.54mm_Vertical, F.Cu at (161.4, 212.3)
- C1, C100, C101, C102, C103, C104, C105, C106, C107, C108, C109, C110, C111, C112, C113, C116, C117, C118, C119, C12, C120, C121, C122, C123, C124, C125, C126, C127, C128, C129, C13, C130, C131, C132, C133, C134, C135, C136, C137, C139, C14, C140, C141, C142, C143, C15, C16, C17, C18, C19, C2, C20, C21, C22, C23, C24, C25, C26, C27, C28, C29, C3, C30, C31, C32, C33, C34, C35, C36, C37, C4, C41, C42, C43, C44, C45, C46, C47, C48, C49, C5, C50, C51, C52, C53, C54, C55, C56, C57, C58, C59, C6, C60, C61, C64, C65, C66, C67, C68, C69, C70, C71, C72, C73, C74, C75, C76, C77, C85, C86, C87, C88, C89, C90, C91, CT2, CT4, CT5, CT6, CT7, CT8, CT9, D10, D8, D9, FB1, L1, L2, L3, L4, L5, Q10, Q11, Q12, Q13, Q14, Q15, Q16, Q17, Q18, Q20, Q21, Q22, Q23, Q24, Q25, Q4, Q5, Q6, Q7, Q8, Q9, R1, R104, R105, R106, R107, R108, R109, R110, R111, R112, R113, R114, R115, R116, R117, R118, R119, R120, R121, R122, R123, R124, R125, R126, R127, R128, R129, R130, R131, R132, R133, R134, R135, R136, R137, R138, R139, R140, R141, R142, R143, R144, R16, R17, R18, R19, R2, R20, R21, R22, R23, R24, R25, R26, R27, R28, R29, R3, R30, R31, R32, R33, R34, R35, R36, R37, R39, R4, R40, R41, R42, R43, R44, R45, R46, R48, R49, R50, R51, R52, R53, R54, R55, R56, R57, R58, R59, R60, R61, R62, R63, R64, R65, R66, R67, R68, R75, R76, R77, R78, R79, R80, R81, R82, R83, R84, R85, R86, R87, R88, R89, R90, R91, R92, R93, R94, R95, SW1, TP10, TP11, TP12, TP13, TP14, TP15, TP16, TP4, TP9, U10, U11, U12, U13, U14, U15, U16, U17, U18, U19, U2, U21, U22, U23, U24, U25, U26, U27, U28, U30, U31, U32, U33, U34, U35, U45, U46, U47, U52, U53, U54, U55, U56, U57, U59, U60, U61, U62, U63, U64, U65, U67, U8, U9, Y1, Y3, Y4: moved to F.Cu
- moved R28 354.8 mm to (472.8, 49.6)
- moved TP2 339.7 mm to (520.8, 100.2)
- moved TP7 335.4 mm to (520.8, 108.3)
- moved TP3 334.9 mm to (520.8, 104.2)
- moved CT9 333.4 mm to (533.3, 216.9)
- moved TP8 330.6 mm to (520.8, 112.3)
- moved C135 330.1 mm to (528.0, 200.2)
- moved R22 329.3 mm to (468.4, 49.6)
- moved R119 325.3 mm to (527.9, 227.1)
- moved R118 325.3 mm to (527.9, 224.1)
- moved R16 321.3 mm to (464.0, 49.6)
- moved C121 320.2 mm to (519.1, 203.2)
- moved R112 316.5 mm to (523.5, 221.2)
- moved SW1 314.4 mm to (510.5, 143.0), turned to 0 degrees
- moved Y3 312.3 mm to (543.6, 220.9)
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Connections:
- net /3v3 renamed 3v3
- net /5v renamed 5v
- net /YD-ESP32-S3/H-bridge/EN renamed H_EN
- net /YD-ESP32-S3/I2C_devices/I2C_RST renamed I2C_RST
- net /YD-ESP32-S3/MCP_CS renamed MCP_CS
- net /YD-ESP32-S3/SPI_devices/CS1 renamed /YD-ESP32-S3/CS1
- net /YD-ESP32-S3/SPI_devices/CS2 renamed /YD-ESP32-S3/CS2
- net /YD-ESP32-S3/SPI_devices/CS3 renamed /YD-ESP32-S3/CS3
- net /YD-ESP32-S3/SPI_devices/CS4 renamed /YD-ESP32-S3/CS4
- net /YD-ESP32-S3/SPI_devices/CS5 renamed /YD-ESP32-S3/CS5
- net /YD-ESP32-S3/SPI_devices/CS6 renamed /YD-ESP32-S3/CS6
- net /YD-ESP32-S3/SPI_devices/CS7 renamed /YD-ESP32-S3/CS7
- net /YD-ESP32-S3/SPI_devices/CS8 renamed /YD-ESP32-S3/CS8
- net /YD-ESP32-S3/Shift_registers/B-B_2 renamed B-B_2
- net /YD-ESP32-S3/Shift_registers/B-B_3 renamed B-B_3
- net /YD-ESP32-S3/Shift_registers/B-B_4 renamed B-B_4
- net /YD-ESP32-S3/Shift_registers/B-B_5 renamed B-B_5
- net /YD-ESP32-S3/Shift_registers/B-B_6 renamed B-B_6
- net /YD-ESP32-S3/Shift_registers/B-B_7 renamed B-B_7
- C108 pad 1: ESP_3v3 -> /YD-ESP32-S3/SPI_devices/BMO085/3V3
- C110 pad 1: /YD-ESP32-S3/SPI_devices/BMO085/3v3-input -> ESP_3v3
- C111 pad 1: /YD-ESP32-S3/SPI_devices/BMO085/3v3-input -> ESP_3v3
- CT7 pad 1: /YD-ESP32-S3/SPI_devices/BMO085/3v3-input -> ESP_3v3
- ESP1 pad 17: TOUCH2 -> BMO_INT
- ESP1 pad 18: TOUCH1 -> INA226_ALERT
- U15 pad 3: /INA226/alert out -> INA226_ALERT
- U16 pad 3: /INA226/alert out -> INA226_ALERT
- U17 pad 3: /INA226/alert out -> INA226_ALERT
- U18 pad 3: /INA226/alert out -> INA226_ALERT
- U19 pad 3: /INA226/alert out -> INA226_ALERT
- U20 pad 3: /INA226/alert out -> INA226_ALERT
- U21 pad 3: /INA226/alert out -> INA226_ALERT
- U22 pad 3: /INA226/alert out -> INA226_ALERT
- U23 pad 3: /INA226/alert out -> INA226_ALERT
- U24 pad 3: /INA226/alert out -> INA226_ALERT
- U25 pad 3: /INA226/alert out -> INA226_ALERT
- U26 pad 3: /INA226/alert out -> INA226_ALERT
- U27 pad 3: /INA226/alert out -> INA226_ALERT
- U28 pad 3: /INA226/alert out -> INA226_ALERT
- U29 pad 3: /INA226/alert out -> INA226_ALERT
- U30 pad 3: /INA226/alert out -> INA226_ALERT
- U57 pad 14: unconnected-(U57-H_INTN-Pad14) -> BMO_INT
- U57 pad 28: ESP_3v3 -> /YD-ESP32-S3/SPI_devices/BMO085/3V3
- U57 pad 3: ESP_3v3 -> /YD-ESP32-S3/SPI_devices/BMO085/3V3
- U57 pad 5: ESP_3v3 -> /YD-ESP32-S3/SPI_devices/BMO085/3V3
- U57 pad 6: ESP_3v3 -> /YD-ESP32-S3/SPI_devices/BMO085/3V3
Routing:
- net ESP_3v3: track 296.4 -> 0.00 mm, vias 16 -> 0
- net /12v_1: track 214.2 -> 0.00 mm, vias 8 -> 0
- net SERVO2: track 107.5 -> 0.00 mm, vias 2 -> 0
- net SERVO4: track 92.7 -> 0.00 mm, vias 1 -> 0
- net SERVO3: track 83.0 -> 0.00 mm, vias 1 -> 0
- net SERVO1: track 65.6 -> 0.00 mm, vias 1 -> 0
- net Net-(U35-SW): track 51.5 -> 0.00 mm, vias 2 -> 0
- net Net-(U31-SW): track 33.4 -> 0.00 mm
- net Net-(U32-SW): track 28.2 -> 0.00 mm, vias 2 -> 0
- net /YD-ESP32-S3/I2C_devices/output_pin_3: track 20.7 -> 0.00 mm
- net /YD-ESP32-S3/SPI_2_MOSI: track 19.9 -> 0.00 mm
- net /YD-ESP32-S3/SPI_2_MISO: track 19.9 -> 0.00 mm
- net /YD-ESP32-S3/SPI_2_CLK: track 19.9 -> 0.00 mm
- net Net-(C65-Pad1): track 9.30 -> 0.00 mm
- net /YD-ESP32-S3/I2C_devices/output_pin_7: track 6.60 -> 0.00 mm
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Other:
- board outline removed
- copper layers 6 -> 2

Commit message: kicad update
Parts:
- added Q27: BC850, Package_TO_SOT_SMD:SOT-23, F.Cu at (485.8, 189.8)
- C96, C98, C99: footprint Capacitor_SMD:C_0805_2012Metric -> Capacitor_SMD:CP_Elec_8x10
- moved Module1 275.8 mm to (606.7, 283.9)
- moved J14 258.1 mm to (520.5, 309.5), turned to 180 degrees
- moved L2 245.6 mm to (372.8, 294.9)
- moved L1 245.5 mm to (373.0, 285.2)
- moved L5 245.2 mm to (372.8, 314.7)
- moved L4 244.9 mm to (372.8, 304.8)
- moved U33 244.8 mm to (350.5, 285.0)
- moved GPIO1 244.4 mm to (728.5, 170.5)
- moved L3 243.4 mm to (373.1, 275.3)
- moved J6 241.4 mm to (644.5, 34.4)
- moved U34 240.6 mm to (350.5, 307.5)
- moved U35 240.4 mm to (350.5, 315.0)
- moved U14 239.9 mm to (705.1, 119.5)
- moved R116 239.9 mm to (765.3, 252.4)
- moved R117 239.9 mm to (765.3, 255.4)
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Connections:
- C73 pad 1: /12v_1 -> /12v_2
- C75 pad 1: /12v_1 -> /12v_2
- C77 pad 1: /12v_1 -> /12v_2
- C96 pad 2: /YD-ESP32-S3/4x tmc5161/TMC_GND -> GND
- C97 pad 2: /YD-ESP32-S3/4x tmc5161/TMC_GND -> GND
- C98 pad 2: /YD-ESP32-S3/4x tmc5161/TMC_GND -> GND
- C99 pad 2: /YD-ESP32-S3/4x tmc5161/TMC_GND -> GND
- J15 pad 12: RGB_D_IN -> MCP_CS
- J15 pad 14: GND -> TPA_ON
- L5 pad 2: /12v_1 -> /12v_2
- R67 pad 1: /12v_1 -> /12v_2
- R84 pad 2: /YD-ESP32-S3/4x tmc5161/TMC_GND -> GND
- R85 pad 2: /YD-ESP32-S3/4x tmc5161/TMC_GND -> GND
- R90 pad 2: /YD-ESP32-S3/4x tmc5161/TMC_GND -> GND
- R91 pad 2: /YD-ESP32-S3/4x tmc5161/TMC_GND -> GND
- TP14 pad 1: /12v_1 -> /12v_2
- U14 pad 3: Net-(U14-GND-Pad3) -> GND
- U14 pad 8: Net-(U14-GND-Pad3) -> GND
- U47 pad 20: unconnected-(U47-VCC-Pad20) -> ESP_5v
- U48 pad 1: /YD-ESP32-S3/4x tmc5161/TMC_GND -> GND
- U48 pad 7: /YD-ESP32-S3/4x tmc5161/TMC_GND -> GND
- U49 pad 1: /YD-ESP32-S3/4x tmc5161/TMC_GND -> GND
- U49 pad 7: /YD-ESP32-S3/4x tmc5161/TMC_GND -> GND
- U50 pad 1: /YD-ESP32-S3/4x tmc5161/TMC_GND -> GND
- U50 pad 7: /YD-ESP32-S3/4x tmc5161/TMC_GND -> GND
- U51 pad 1: /YD-ESP32-S3/4x tmc5161/TMC_GND -> GND
- U51 pad 7: /YD-ESP32-S3/4x tmc5161/TMC_GND -> GND
- U53 pad 10: unconnected-(U53-VSS-Pad10) -> GND
- U54 pad 10: unconnected-(U54-VSS-Pad10) -> GND
Routing:
- net GND: vias 0 -> 1
- net 5V1: vias 0 -> 1
Other:
- board outline added: 524.5 x 106.5 mm

Commit message: updated kicad (big_update)
Parts:
- added C39: 1uf, Capacitor_SMD:C_0805_2012Metric, F.Cu at (572.7, 129.2)
- added CT10: 10uf, Capacitor_Tantalum_SMD:CP_EIA-3528-21_Kemet-B, F.Cu at (573.5, 125.5)
- added J17: Conn_01x02_Pin, Connector_PinHeader_2.54mm:PinHeader_2x20_P2.54mm_Vertical, F.Cu at (707.5, -32.7)
- added J18: Conn_01x02_Pin, Connector_PinHeader_2.54mm:PinHeader_2x20_P2.54mm_Vertical, F.Cu at (714.6, -32.7)
- added J19: Conn_01x02_Pin, Connector_PinHeader_2.54mm:PinHeader_2x20_P2.54mm_Vertical, F.Cu at (721.7, -32.7)
- added J20: Conn_01x02_Pin, Connector_PinHeader_2.54mm:PinHeader_2x20_P2.54mm_Vertical, F.Cu at (728.9, -32.7)
- added J21: Conn_01x02_Pin, Connector_PinHeader_2.54mm:PinHeader_2x20_P2.54mm_Vertical, F.Cu at (736.0, -32.7)
- added J22: Conn_01x02_Pin, Connector_PinHeader_2.54mm:PinHeader_2x20_P2.54mm_Vertical, F.Cu at (743.2, -32.7)
- added J23: Conn_01x02_Pin, Connector_PinHeader_2.54mm:PinHeader_2x20_P2.54mm_Vertical, F.Cu at (750.3, -32.7)
- added J24: Conn_01x02_Pin, Connector_PinHeader_2.54mm:PinHeader_2x20_P2.54mm_Vertical, F.Cu at (757.4, -32.7)
- added R100: 47k, Resistor_SMD:R_0805_2012Metric, F.Cu at (707.4, 22.3)
- added R101: 10k, Resistor_SMD:R_0805_2012Metric, F.Cu at (707.4, 25.3)
- added R102: 10k, Resistor_SMD:R_0805_2012Metric, F.Cu at (707.4, 28.2)
- added R103: 10k, Resistor_SMD:R_0805_2012Metric, F.Cu at (711.8, 19.4)
- added R153: 10k, Resistor_SMD:R_0805_2012Metric, F.Cu at (711.8, 22.3)
- added R154: 47k, Resistor_SMD:R_0805_2012Metric, F.Cu at (711.8, 25.3)
- added R155: 10k, Resistor_SMD:R_0805_2012Metric, F.Cu at (711.8, 28.2)
- added R156: 10k, Resistor_SMD:R_0805_2012Metric, F.Cu at (716.2, 19.4)
- added R157: 10k, Resistor_SMD:R_0805_2012Metric, F.Cu at (716.2, 22.3)
- added R158: 10k, Resistor_SMD:R_0805_2012Metric, F.Cu at (716.2, 25.3)
- added R159: 47k, Resistor_SMD:R_0805_2012Metric, F.Cu at (716.2, 28.2)
- added R96: 470k, Resistor_SMD:R_0805_2012Metric, F.Cu at (771.1, -33.5)
- added R97: 47k, Resistor_SMD:R_0805_2012Metric, F.Cu at (557.2, 110.4)
- added R98: 47k, Resistor_SMD:R_0805_2012Metric, F.Cu at (557.2, 113.4)
- added R99: 47k, Resistor_SMD:R_0805_2012Metric, F.Cu at (707.4, 19.4)
- added SW5: SW_SPST, Connector_PinHeader_2.54mm:PinHeader_1x02_P2.54mm_Vertical, F.Cu at (766.6, -32.7)
- added U38: IP2721, Package_SO:TSSOP-16_4.4x5mm_P0.65mm, F.Cu at (548.6, 112.2)
- added U6: BQ24650, Package_DFN_QFN:Texas_RVA_VQFN-16-1EP_3.5x3.5mm_P0.5mm_EP2.14x2.14mm_ThermalVias, F.Cu at (546.8, 118.4)
- C12, C14: value 27pF -> 22pf
- C120, C122: value C -> 22pf
- Q2, Q3: value SS8050-G -> bc akármi
- Q27: value BC850 -> BC817
- R110: value R -> 1M
- R14: value 100K 1% -> 47k
- R86, R87, R92, R93: value 320 -> 330
- R9: footprint Resistor_SMD:R_0805_2012Metric -> Resistor_SMD:R_0603_1608Metric
- moved U52 95.9 mm to (290.5, 197.5)
- moved DC3 95.4 mm to (248.2, 209.2)
- moved DC4 95.4 mm to (248.2, 217.2)
- moved DC5 95.4 mm to (248.2, 225.2)
- moved DC6 95.4 mm to (248.2, 233.2)
- moved Q20 95.4 mm to (252.8, 194.4)
- moved SERVO2 95.4 mm to (248.2, 259.6)
- moved C108 95.4 mm to (676.5, 152.9)
- moved C109 95.4 mm to (676.5, 155.9)
- moved C110 95.4 mm to (676.5, 159.0)
- moved C112 95.4 mm to (676.5, 165.0)
- moved C15 95.4 mm to (649.7, 23.0)
- moved C3 95.4 mm to (632.8, 74.2)
- moved C4 95.4 mm to (632.8, 78.5)
- moved C5 95.4 mm to (590.7, 98.6)
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Connections:
- net Net-(J9-CC1) renamed PD-CHARGE_CC1
- net Net-(J9-CC2) renamed PD-CHARGE_CC2
- C102 pad 2: /YD-ESP32-S3/H-bridge/TB_GND -> GND
- ESP1 pad 10: /Uart_tx -> SPI0_MISO
- ESP1 pad 11: /Uart_rx -> SPI0_CLK
- GPIO1 pad 10: /Uart_rx -> SPI0_CLK
- GPIO1 pad 12: /CM5_GPIO ( Ethernet, GPIO, SDCARD)/GPIO18 -> SPI0_MOSI
- GPIO1 pad 16: /CM5_GPIO ( Ethernet, GPIO, SDCARD)/GPIO23 -> INA226_SCL
- GPIO1 pad 22: /CM5_GPIO ( Ethernet, GPIO, SDCARD)/GPIO25 -> SPI1_MISO
- GPIO1 pad 24: SPI0_CE0 -> INA226_SCL
- GPIO1 pad 26: /CM5_GPIO ( Ethernet, GPIO, SDCARD)/GPIO7 -> INA226_SDA
- GPIO1 pad 38: SPI1_MOSI -> INA226_SDA
- GPIO1 pad 40: SPI1_CLK -> INA226_SCL
- GPIO1 pad 8: /Uart_tx -> SPI0_MISO
- J9 pad A4: unconnected-(J9-VBUS-PadA4) -> PD-CHARGE_VBUS
- J9 pad A9: unconnected-(J9-VBUS-PadA4)_3 -> PD-CHARGE_VBUS
- J9 pad B4: unconnected-(J9-VBUS-PadA4)_1 -> PD-CHARGE_VBUS
- J9 pad B9: unconnected-(J9-VBUS-PadA4)_2 -> PD-CHARGE_VBUS
- Module1 pad 25: SPI1_CLK -> INA226_SCL
- Module1 pad 27: SPI1_MOSI -> INA226_SDA
- Module1 pad 37: /CM5_GPIO ( Ethernet, GPIO, SDCARD)/GPIO7 -> INA226_SDA
- Module1 pad 39: SPI0_CE0 -> INA226_SCL
- Module1 pad 41: /CM5_GPIO ( Ethernet, GPIO, SDCARD)/GPIO25 -> SPI1_MISO
- Module1 pad 47: /CM5_GPIO ( Ethernet, GPIO, SDCARD)/GPIO23 -> INA226_SCL
- Module1 pad 49: /CM5_GPIO ( Ethernet, GPIO, SDCARD)/GPIO18 -> SPI0_MOSI
- Module1 pad 51: /Uart_rx -> SPI0_CLK
- Module1 pad 55: /Uart_tx -> SPI0_MISO
- Q27 pad 1: unconnected-(Q27-B-Pad1) -> /CM5_HighSpeed/PCIE_PWR_EN
- Q27 pad 2: unconnected-(Q27-E-Pad2) -> Net-(Q27-E)
- Q27 pad 3: unconnected-(Q27-C-Pad3) -> /PCIe-M2/12v
- U52 pad 10: /YD-ESP32-S3/H-bridge/TB_GND -> GND
- U52 pad 18: /YD-ESP32-S3/H-bridge/TB_GND -> GND
- U52 pad 3: /YD-ESP32-S3/H-bridge/TB_GND -> GND
- U52 pad 4: /YD-ESP32-S3/H-bridge/TB_GND -> GND
- U52 pad 9: /YD-ESP32-S3/H-bridge/TB_GND -> GND
- U59 pad 2: SPI1_CLK -> INA226_SCL
- U60 pad 2: SPI1_MOSI -> INA226_SDA
- U61 pad 4: SPI0_CE0 -> INA226_SCL
- U63 pad 1: unconnected-(U63-SDI-Pad1) -> /YD-ESP32-S3/SPI_2_MOSI
- U63 pad 10: unconnected-(U63-AUX_IN-Pad10) -> Net-(U63-AUX_IN)
- U63 pad 11: unconnected-(U63-AUX_GND-Pad11) -> GND
- U63 pad 12: unconnected-(U63-AIN_6P-Pad12) -> Net-(J23-Pin_1)
- U63 pad 13: unconnected-(U63-AIN_6GND-Pad13) -> GND
- U63 pad 14: unconnected-(U63-AIN_7P-Pad14) -> Net-(J24-Pin_1)
- U63 pad 15: unconnected-(U63-AIN_7GND-Pad15) -> GND
- U63 pad 16: unconnected-(U63-AIN_0P-Pad16) -> Net-(J17-Pin_1)
- U63 pad 17: unconnected-(U63-AIN_0GND-Pad17) -> GND
- U63 pad 18: unconnected-(U63-AIN_1P-Pad18) -> Net-(J18-Pin_1)
- U63 pad 19: unconnected-(U63-AIN_1GND-Pad19) -> GND
- U63 pad 2: unconnected-(U63-~{RST/PD}-Pad2) -> /YD-ESP32-S3/SPI_devices/ADS8688/AD_RST
- U63 pad 20: unconnected-(U63-AIN_2GND-Pad20) -> GND
- U63 pad 21: unconnected-(U63-AIN_2P-Pad21) -> Net-(J19-Pin_1)
- U63 pad 22: unconnected-(U63-AIN_3GND-Pad22) -> GND
- U63 pad 23: unconnected-(U63-AIN_3P-Pad23) -> Net-(J20-Pin_1)
- U63 pad 24: unconnected-(U63-AIN_4GND-Pad24) -> GND
- U63 pad 25: unconnected-(U63-AIN_4P-Pad25) -> Net-(J21-Pin_1)
- U63 pad 26: unconnected-(U63-AIN_5GND-Pad26) -> GND
- U63 pad 27: unconnected-(U63-AIN_5P-Pad27) -> Net-(J22-Pin_1)
- U63 pad 28: Net-(U63-AGND-Pad28) -> GND
- U63 pad 29: Net-(U63-AGND-Pad28) -> GND
- U63 pad 3: unconnected-(U63-DAISY-Pad3) -> Net-(U63-DAISY)
- U63 pad 30: unconnected-(U63-AVDD-Pad30) -> /YD-ESP32-S3/SPI_devices/ADS8688/5v
- U63 pad 31: Net-(U63-AGND-Pad28) -> GND
- U63 pad 32: Net-(U63-AGND-Pad28) -> GND
- U63 pad 33: unconnected-(U63-DGND-Pad33) -> GND
- U63 pad 34: unconnected-(U63-DVDD-Pad34) -> ESP_3v3
- U63 pad 36: unconnected-(U63-SDO-Pad36) -> /YD-ESP32-S3/SPI_2_MISO
- U63 pad 37: unconnected-(U63-SCLK-Pad37) -> /YD-ESP32-S3/SPI_2_CLK
- U63 pad 38: unconnected-(U63-~{CS}-Pad38) -> /YD-ESP32-S3/CS4
- U63 pad 4: unconnected-(U63-~{REFSEL}-Pad4) -> GND
- U63 pad 6: unconnected-(U63-REFGND-Pad6) -> GND
- U63 pad 7: unconnected-(U63-REFCAP-Pad7) -> Net-(U63-REFCAP)
- U63 pad 8: Net-(U63-AGND-Pad28) -> GND
- U63 pad 9: unconnected-(U63-AVDD-Pad9) -> /YD-ESP32-S3/SPI_devices/ADS8688/5v
