File: Circuit/kicad/Robot fő nyák_v3/USB_AUDIO.kicad_sch (KiCad schematic)
At the start: 40 parts, among them J45 Conn_01x02_Pin, SW1 SW_Push, SW5 SW_Push, SW6 SW_Push, U14 PCM2704C, U65 TPA6203A1DGN, Y3 5MHz

Commit message: readme updated kicad circuit V1
Parts:
- C121: renamed from C73; footprint (none) -> Capacitor_SMD:C_0805_2012Metric
- C123: renamed from C77; footprint (none) -> Capacitor_SMD:C_0805_2012Metric
- C124: renamed from C68; footprint (none) -> Capacitor_SMD:C_0805_2012Metric
- C125: renamed from C69; footprint (none) -> Capacitor_SMD:C_0805_2012Metric
- C126: renamed from C76; footprint (none) -> Capacitor_SMD:C_0805_2012Metric
- C127: renamed from C71; footprint (none) -> Capacitor_SMD:C_0805_2012Metric
- C128: renamed from C70; footprint (none) -> Capacitor_SMD:C_0805_2012Metric
- C129: renamed from C74; footprint (none) -> Capacitor_Tantalum_SMD:CP_EIA-7343-31_Kemet-D
- C130: renamed from C75; footprint (none) -> Capacitor_Tantalum_SMD:CP_EIA-7343-31_Kemet-D
- C131: renamed from C72; footprint (none) -> Capacitor_Tantalum_SMD:CP_EIA-3528-21_Kemet-B
- C132: renamed from C79; footprint (none) -> Capacitor_SMD:C_0805_2012Metric
- C133: renamed from C80; footprint (none) -> Capacitor_SMD:C_0805_2012Metric
- C137: renamed from C78; footprint (none) -> Capacitor_SMD:C_0805_2012Metric
- CT9: renamed from CT3; footprint (none) -> Capacitor_Tantalum_SMD:CP_EIA-3528-21_Kemet-B
- R106: renamed from R107; footprint (none) -> Resistor_SMD:R_0805_2012Metric
- R107: renamed from R108; footprint (none) -> Resistor_SMD:R_0805_2012Metric
- R108: renamed from R109; footprint (none) -> Resistor_SMD:R_0805_2012Metric
- R109: renamed from R110; footprint (none) -> Resistor_SMD:R_0805_2012Metric
- R111: renamed from R112; footprint (none) -> Resistor_SMD:R_0805_2012Metric
- R112: renamed from R111; footprint (none) -> Resistor_SMD:R_0805_2012Metric
- R113, R114, R115, R116, R117, R118, R119: footprint (none) -> Resistor_SMD:R_0805_2012Metric
- SPEAKER1: renamed from J45; footprint (none) -> Connector_JST:JST_PH_B2B-PH-K_1x02_P2.00mm_Vertical
- SW2: renamed from SW1; footprint (none) -> Connector_PinHeader_2.54mm:PinHeader_1x02_P2.54mm_Vertical
- SW3: renamed from SW5; footprint (none) -> Connector_PinHeader_2.54mm:PinHeader_1x02_P2.54mm_Vertical
- SW4: renamed from SW6; footprint (none) -> Connector_PinHeader_2.54mm:PinHeader_1x02_P2.54mm_Vertical
- renumbered C66 to C120, C67 to C122, C91 to C134, C89 to C135, C90 to C136, R106 to R110, U14 to U64

Commit message: updated kicad (big_update)
Parts:
- C120, C122: value C -> 22pf
- R110: value R -> 1M
- U64: value PCM2704C -> PCM2704CDBR
Changed lines of the file:
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@@
 		(fields_autoplaced yes)
 		(property "Reference" "R110"
-			(at 91.4399 49.53 0)
-			(effects
-				(font
-					(size 1.27 1.27)
-				)
-				(justify left)
-			)
-		)
-		(property "Value" "R"
-			(at 93.9799 49.53 0)
-			(effects
-				(font
-					(size 1.27 1.27)
-				)
-				(justify left)
+			(at 92.71 45.72 90)
+			(effects
+				(font
+					(size 1.27 1.27)
+				)
+			)
+		)
+		(property "Value" "1M"
+			(at 92.71 48.26 90)
+			(effects
+				(font
+					(size 1.27 1.27)
+				)
 			)
 		)
@@
 		(fields_autoplaced yes)
 		(property "Reference" "C120"
-			(at 81.28 26.67 90)
-			(effects
-				(font
-					(size 1.27 1.27)
-				)
-			)
-		)
-		(property "Value" "C"
-			(at 83.82 26.67 90)
-			(effects
-				(font
-					(size 1.27 1.27)
-				)
+			(at 92.71 25.3999 0)
+			(effects
+				(font
+					(size 1.27 1.27)
+				)
+				(justify right)
+			)
+		)
+		(property "Value" "22pf"
+			(at 92.71 27.9399 0)
+			(effects
+				(font
+					(size 1.27 1.27)
+				)
+				(justify right)
 			)
 		)
@@
 			)
 		)
-		(property "Value" "PCM2704C"
+		(property "Value" "PCM2704CDBR"
 			(at 92.71 58.42 0)
 			(effects
@@
 			)
 		)
-		(property "Value" "C"
+		(property "Value" "22pf"
 			(at 103.378 26.67 90)
 			(effects
