File: Circuit/kicad/Robot fő nyák_v3/felső panel.kicad_pcb (KiCad board)
At the start: 6 copper layers, 120 x 70.2 mm, 283 parts, among them J10 USB_C_Receptacle_USB2.0_16P, J11 THD-02-R, J12 Conn_01x04_Socket, J13 THD-02-R, J15 Conn_01x60_MountingPin, J17 Conn_01x02_Pin, J18 Conn_01x02_Pin, J19 Conn_01x08_Pin, J2 USB3_A, J20 Conn_01x08_Pin, J21 Conn_01x02_Pin, J22 Conn_01x02_Pin, J23 Conn_01x02_Pin, J24 Conn_01x02_Pin, J28 Conn_01x08_Pin, J3 690-019-298-412, J4 690-019-298-412, J5 MagJack-A70-112-331N126, J6 Bus_M.2_Socket_M, J7 690-008-221-904, J8 USB_C_Receptacle_USB2.0_16P, J9 USB_C_Receptacle_USB2.0_16P, Q2 bc akármi, Q3 bc akármi, SW1 Right angle Tact button, SW2 SW_Push, SW3 SW_Push, SW4 SW_Push, U1 AP22653W6, U10 TPD4EUSB30, U11 USB2514B-I/M2, U12 TPD4EUSB30, U13 FSUSB42MUX, U14 TPD4EUSB30, U2 RT9742SNGV, U3 74LVC1G07SE-7, U32 AP22815AWU, U37 CH343P, U4 TPD4EUSB30, U45 TCA9548APWR, U46 TCA9548APWR, U47 MCP3208, U5 TPD4EUSB30, U54 MCP23S17_SO, U55 ICM-45686, U56 BME280, U57 BNO080, U58 MCP1541-TT, U59 TS5A23157DGSR, U60 TS5A23157DGSR, U61 TS5A23157DGSR, U62 TS5A23157DGSR, U64 PCM2704CDBR, U65 TPA6203A1DGN, U66 TS5A23157DGSR, U7 ASEK-32.768KHZ-L-R-T, U8 FSUSB42MUX, U9 AP22653W6, Y1 24MHz, Y3 5MHz, Y4 32.768MHz

Commit message: new 2 pcb schematics in v4.0 folder, psu sch finish, bad pcb, high speed: bad pcb and sch
Routing:
- net /CM5_HighSpeed/HDMI1_CK_N: track 0.00 -> 11.6 mm
- net /CM5_HighSpeed/HDMI1_CK_P: track 0.00 -> 11.6 mm
Changed lines of the file:
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@@
 		(layer "Edge.Cuts")
+	)
+	(segment
+		(start 78.376863 90.508665)
+		(end 78.376863 89.926484)
+		(width 0.2)
+		(layer "F.Cu")
+		(net 363)
+	)
+	(segment
+		(start 82.35 97.907499)
+		(end 82.075 97.632499)
+		(width 0.2)
+		(layer "F.Cu")
+		(net 363)
+	)
+	(segment
+		(start 82.075 97.632499)
+		(end 82.075 94.206802)
+		(width 0.2)
+		(layer "F.Cu")
+		(net 363)
+	)
+	(segment
+		(start 82.35 99.8575)
+		(end 82.35 97.907499)
+		(width 0.2)
+		(layer "F.Cu")
+		(net 363)
+	)
+	(segment
+		(start 82.075 94.206802)
+		(end 78.376863 90.508665)
+		(width 0.2)
+		(layer "F.Cu")
+		(net 363)
+	)
+	(segment
+		(start 81.35 97.907499)
+		(end 81.625 97.632499)
+		(width 0.2)
+		(layer "F.Cu")
+		(net 365)
+	)
+	(segment
+		(start 81.625 97.632499)
+		(end 81.625 94.393198)
+		(width 0.2)
+		(layer "F.Cu")
+		(net 365)
+	)
+	(segment
+		(start 81.625 94.393198)
+		(end 77.926863 90.695061)
+		(width 0.2)
+		(layer "F.Cu")
+		(net 365)
+	)
+	(segment
+		(start 77.926863 90.695061)
+		(end 77.926863 89.926484)
+		(width 0.2)
+		(layer "F.Cu")
+		(net 365)
+	)
+	(segment
+		(start 81.35 99.8575)
+		(end 81.35 97.907499)
+		(width 0.2)
+		(layer "F.Cu")
+		(net 365)
 	)
 	(group ""
