File: Circuit/kicad/V4/psu_motor-controll/psu.kicad_sch (KiCad schematic)
At the start: 5 parts, among them Q1 bss138, U1 MCP23S17_SO

Commit message: kicad psu pcb finish psu
Connections:
- net M1_DIR: now also U1.2 (GPB1); no longer U1.5 (GPB4)
- net M2_DIR: now also U1.4 (GPB3); no longer U1.6 (GPB5)
- net M2_EN: now also U1.3 (GPB2); no longer U1.2 (GPB1)
- net M3_DIR: now also U1.6 (GPB5); no longer U1.7 (GPB6)
- net M3_EN: now also U1.5 (GPB4); no longer U1.3 (GPB2)
- net M4_EN: now also U1.7 (GPB6); no longer U1.4 (GPB3)
- net B-B_2 renamed DC12V_1
- net B-B_3 renamed DC12V_2
- net B-B_4 renamed DC5V_1
- net B-B_5 renamed DC5V_2
- net B-B_6 renamed DC3.3V_1
- net B-B_7 renamed DC3.3V_2

Commit message: kicad FINISH PSU PCB
Other:
- sheet PCA9531PW renamed PCA9685PW
Changed lines of the file:
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@@
 			(color 0 0 0 0.0000)
 		)
-		(property "Sheetname" "PCA9531PW"
+		(property "Sheetname" "PCA9685PW"
 			(at 234.95 135.128 0)
 			(effects

Commit message: PSU FINISH BOARD NO DRC,ERC,DFM ERRORS
Changed lines of the file:
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@@
 	(wire
 		(pts
-			(xy 71.12 100.33) (xy 92.71 100.33)
+			(xy 71.12 100.33) (xy 91.44 100.33)
 		)
 		(stroke
@@
 	)
 	(label "PCA_RST"
-		(at 92.71 100.33 180)
+		(at 91.44 100.33 180)
 		(effects
 			(font
@@
 			(project "psu"
 				(path "/e63e39d7-6ac0-4ffd-8aa3-1841a4541b55"
-					(page "20")
+					(page "10")
 				)
 			)
@@
 			(project "psu"
 				(path "/e63e39d7-6ac0-4ffd-8aa3-1841a4541b55"
-					(page "10")
-				)
-			)
+					(page "5")
+				)
+			)

Commit message: PSU bugfixes
Parts:
- added R74: 100R, Resistor_SMD:R_0805_2012Metric, symbol Device:R
- added R75: 10k, Resistor_SMD:R_0805_2012Metric, symbol Device:R
Connections:
- net ESP_3v3: no longer Q1.2 (G)
- net GND: now also Q1.3 (S), R75.2
- net WS_2802B_DATA: now also R74.2; no longer Q1.3 (S), R1.1
- new net: Q1.2 (G), R1.1, R74.1, R75.1
Other:
- moved on the sheet: LED1, Q1, R1, R2

Commit message: V4.1.7 PSU  V1.0 debug Card
Changed lines of the file:
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@@
 	)
 	(sheet
-		(at 19.05 19.05)
+		(at 78.74 20.32)
 		(size 48.26 31.75)
 		(exclude_from_sim no)
@@
 		)
 		(property "Sheetname" "power-management"
-			(at 19.05 18.3384 0)
+			(at 78.74 19.6084 0)
 			(effects
 				(font
@@
 		)
 		(property "Sheetfile" "power-management.kicad_sch"
-			(at 19.05 51.3846 0)
+			(at 78.74 52.6546 0)
 			(effects
 				(font
