File: Circuit/kicad/V4/psu_motor-controll/H-bridge.kicad_sch (KiCad schematic)
At the start: 7 parts, among them U2 TB6612FNG

Commit message: kicad psu pcb finish psu
Parts:
- removed C5: 470uf, Capacitor_SMD:CP_Elec_8x10, symbol Device:C_Polarized
- removed C7: 1uf, Capacitor_SMD:C_0805_2012Metric, symbol Device:C
- removed CT1: 10uf, Capacitor_Tantalum_SMD:CP_EIA-3528-21_Kemet-B, symbol Device:C_Polarized_Small
- added C5, C78, C79, C80: 4,7uf, Capacitor_SMD:C_0805_2012Metric, symbol Device:C
Connections:
- net GND: now also C5.2, C78.2, C79.2, C80.2
- net H-bridge: now also C5.1, C78.1, C79.1, C80.1
- net at U2.5 (AO2), U2.6 (AO2): now also H-M1.2 (Pin_2); no longer H-M1.1 (Pin_1)
- net at U2.1 (AO1), U2.2 (AO1): now also H-M1.1 (Pin_1); no longer H-M1.2 (Pin_2)
Other:
- note removed: "//motor A connected between A01 and A02 //motor B connected between B01 and B02 int STBY = 10; //standby //Motor A int PWMA = 3; //Speed control int AIN1 = 9; //Direction int AIN2 = 8; //Direction //Motor B int PWMB = 5; //Speed control int BIN1 = 11; //Direction int BIN2 = 12; //Direction void setup(){ pinMode(STBY, OUTPUT); pinMode(PWMA, OUTPUT); pinMode(AIN1, OUTPUT); pinMode(AIN2, OUTPUT); pi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"
- note removed: "void move(int motor, int speed, int direction){ //Move specific motor at speed and direction //motor: 0 for B 1 for A //speed: 0 is off, and 255 is full speed //direction: 0 clockwise, 1 counter-clockwise digitalWrite(STBY, HIGH); //disable standby boolean inPin1 = LOW; boolean inPin2 = HIGH; if(direction == 1){ inPin1 = HIGH; inPin2 = LOW; } if(motor == 1){ digitalWrite(AIN1, inPin1); digitalWri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"
- moved on the sheet: H-M1

Commit message: updated bom, updated compon
Parts:
- C5, C78, C79, C80: Cikkszám (none) -> 100.427.11; Link (none) -> https://www.hestore.hu/prod_10042711.html
- C6: Cikkszám (none) -> 100.277.53; Link (none) -> https://www.hestore.hu/prod_10027753.html
- H-M1, H-M2: Cikkszám (none) -> 100.385.23; Link (none) -> https://www.hestore.hu/prod_10038523.html
- U2: Cikkszám (none) -> 100.491.22; Link (none) -> https://www.hestore.hu/prod_10049122.html
Changed lines of the file:
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@@
 			)
 		)
-		(property "Datasheet" "~"
+		(property "Datasheet" "https://www.hestore.hu/prod_getfile.php?id=9997"
 			(at 69.85 41.91 0)
 			(effects
@@
 			)
 		)
-		(property "Sim.Device" ""
+		(property "Cikkszám" "100.385.23"
 			(at 69.85 41.91 0)
 			(effects
@@
 			)
 		)
-		(property "Sim.Type" ""
+		(property "Link" "https://www.hestore.hu/prod_10038523.html"
 			(at 69.85 41.91 0)
 			(effects
@@
 			)
 		)
-		(property "Sim.Device" ""
+		(property "Cikkszám" "100.427.11"
 			(at 135.89 48.26 0)
 			(effects
@@
 			)
 		)
-		(property "Sim.Type" ""
+		(property "Link" "https://www.hestore.hu/prod_10042711.html"
 			(at 135.89 48.26 0)
 			(effects
@@
 			)
 		)
-		(property "Sim.Device" ""
+		(property "Cikkszám" "100.427.11"
 			(at 100.33 48.26 0)
 			(effects
@@
 			)
 		)
-		(property "Sim.Type" ""
+		(property "Link" "https://www.hestore.hu/prod_10042711.html"
 			(at 100.33 48.26 0)
 			(effects
@@
 			)
 		)
-		(property "Sim.Device" ""
+		(property "Cikkszám" "100.427.11"
 			(at 124.46 48.26 0)
 			(effects
@@
 			)
 		)
-		(property "Sim.Type" ""
+		(property "Link" "https://www.hestore.hu/prod_10042711.html"
 			(at 124.46 48.26 0)
 			(effects
@@
 			)
 		)
-		(property "Datasheet" "~"
+		(property "Datasheet" "https://www.hestore.hu/prod_getfile.php?id=4317"
 			(at 53.34 101.6 0)
 			(effects
@@
 			)
 		)
-		(property "Sim.Device" ""
+		(property "Cikkszám" "100.277.53"
 			(at 53.34 101.6 0)
 			(effects
@@
 			)
 		)
-		(property "Sim.Type" ""
+		(property "Link" "https://www.hestore.hu/prod_10027753.html"
 			(at 53.34 101.6 0)
 			(effects
@@
 			)
 		)
-		(property "Sim.Device" ""
+		(property "Cikkszám" "100.427.11"
 			(at 111.76 48.26 0)
 			(effects
@@
 			)
 		)
-		(property "Sim.Type" ""
+		(property "Link" "https://www.hestore.hu/prod_10042711.html"
 			(at 111.76 48.26 0)
 			(effects
@@
 			)
 		)
-		(property "Datasheet" "~"
+		(property "Datasheet" "https://www.hestore.hu/prod_getfile.php?id=9997"
 			(at 69.85 57.15 0)
 			(effects
@@
 			)
 		)
-		(property "Sim.Device" ""
+		(property "Cikkszám" "100.385.23"
 			(at 69.85 57.15 0)
 			(effects
@@
 			)
 		)
-		(property "Sim.Type" ""
+		(property "Link" "https://www.hestore.hu/prod_10038523.html"
 			(at 69.85 57.15 0)
 			(effects
@@
 			)
 		)
-		(property "Datasheet" "https://toshiba.semicon-storage.com/us/product/linear/motordriver/detail.TB6612FNG.html"
+		(property "Datasheet" "https://www.hestore.hu/prod_getfile.php?id=20099"
 			(at 55.88 35.56 0)
 			(effects
@@
 			)
 		)
-		(property "Sim.Device" ""
+		(property "Cikkszám" "100.491.22"
 			(at 44.45 50.8 0)
 			(effects
@@
 			)
 		)
-		(property "Sim.Type" ""
+		(property "Link" "https://www.hestore.hu/prod_10049122.html"
 			(at 44.45 50.8 0)
 			(effects
