File: Circuit/kicad/V4/psu_motor-controll/INA226.kicad_sch (KiCad schematic)
At the start: 48 parts, among them U10 INA226, U11 INA226, U12 INA226, U13 INA226, U14 INA226, U15 INA226, U16 INA226, U17 INA226, U18 INA226, U19 INA226, U20 INA226, U21 INA226, U6 INA226, U7 INA226, U8 INA226, U9 INA226

Commit message: kicad v4 psu pcb clean
Parts:
- renumbered C13 to C16, C14 to C17, C15 to C18, C16 to C19, C17 to C20, C18 to C21, C19 to C22, C20 to C23, C21 to C24, C22 to C25, C23 to C26, C24 to C27, C25 to C28, C26 to C29, C27 to C30, C28 to C31, R16 to R19, R17 to R20, R18 to R21, R19 to R22, R20 to R23, R21 to R24, R22 to R25, R23 to R26, R24 to R27, R25 to R28, R26 to R29, R27 to R30, R28 to R31, R29 to R32, R30 to R33, R31 to R34, U11 to U10, U12 to U11, U13 to U12, U14 to U13, U15 to U14, U16 to U15, U17 to U16, U18 to U17, U19 to U18, U20 to U19, U21 to U20, U6 to U5, U7 to U6, U8 to U7, U9 to U8, U10 to U9

Commit message: kicad psu pcb finish psu
Parts:
- removed C20, C21, C22, C23, C24, C25, C26, C27, C28, C29, C30, C31: 1uf, Capacitor_SMD:C_0805_2012Metric, symbol Device:C
Other:
- moved on the sheet: C16, C17, C18, C19

Commit message: PSU bugfixes
Parts:
- R19, R20, R21, R22, R23, R25: value 0.025Ω -> 0.082Ω
- R24, R27, R31, R34: value 0.025Ω -> 0.056Ω
- R26, R32: value 0.025Ω -> 0.150Ω
- R28: value 0.025Ω -> 0.020Ω
- R29, R30, R33: value 0.025Ω -> 0.033Ω
Changed lines of the file:
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@@
 			)
 		)
-		(property "Value" "0.025Ω"
+		(property "Value" "0.056Ω"
 			(at 30.48 146.05 90)
 			(effects
@@
 			)
 		)
-		(property "Value" "0.025Ω"
+		(property "Value" "0.150Ω"
 			(at 72.39 146.05 90)
 			(effects
@@
 			)
 		)
-		(property "Value" "0.025Ω"
+		(property "Value" "0.056Ω"
 			(at 247.65 24.13 90)
 			(effects
@@
 			)
 		)
-		(property "Value" "0.025Ω"
+		(property "Value" "0.082Ω"
 			(at 72.39 22.86 90)
 			(effects
@@
 			)
 		)
-		(property "Value" "0.025Ω"
+		(property "Value" "0.150Ω"
 			(at 72.39 85.09 90)
 			(effects
@@
 			)
 		)
-		(property "Value" "0.025Ω"
+		(property "Value" "0.082Ω"
 			(at 30.48 22.86 90)
 			(effects
@@
 			)
 		)
-		(property "Value" "0.025Ω"
+		(property "Value" "0.056Ω"
 			(at 115.57 85.09 90)
 			(effects
@@
 			)
 		)
-		(property "Value" "0.025Ω"
+		(property "Value" "0.033Ω"
 			(at 200.66 85.09 90)
 			(effects
@@
 			)
 		)
-		(property "Value" "0.025Ω"
+		(property "Value" "0.082Ω"
 			(at 203.2 24.13 90)
 			(effects
@@
 			)
 		)
-		(property "Value" "0.025Ω"
+		(property "Value" "0.082Ω"
 			(at 115.57 22.86 90)
 			(effects
@@
 			)
 		)
-		(property "Value" "0.025Ω"
+		(property "Value" "0.082Ω"
 			(at 157.48 22.86 90)
 			(effects
@@
 			)
 		)
-		(property "Value" "0.025Ω"
+		(property "Value" "0.056Ω"
 			(at 154.94 146.05 90)
 			(effects
@@
 			)
 		)
-		(property "Value" "0.025Ω"
+		(property "Value" "0.020Ω"
 			(at 157.48 85.09 90)
 			(effects
@@
 			)
 		)
-		(property "Value" "0.025Ω"
+		(property "Value" "0.082Ω"
 			(at 30.48 85.09 90)
 			(effects
@@
 			)
 		)
-		(property "Value" "0.025Ω"
+		(property "Value" "0.033Ω"
 			(at 246.38 85.09 90)
 			(effects
@@
 			)
 		)
-		(property "Value" "0.025Ω"
+		(property "Value" "0.033Ω"
 			(at 113.03 146.05 90)
 			(effects

Commit message: updated bom, updated compon
Parts:
- C16, C17, C18, C19: Cikkszám (none) -> 100.277.53; Link (none) -> https://www.hestore.hu/prod_10027753.html
- R19, R20, R21, R22, R23, R25: Cikkszám (none) -> 100.491.24; Link (none) -> https://www.hestore.hu/prod_10049124.html; Url https://hu.farnell.com/vishay/wfma2512r0250fea/res-0r025-3w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 -> (none)
- R24, R27, R31, R34: Cikkszám (none) -> 100.491.07; Link (none) -> https://www.hestore.hu/prod_10049107.html; Url https://hu.farnell.com/vishay/wfma2512r0250fea/res-0r025-3w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 -> (none)
- R26, R32: Cikkszám (none) -> 100.491.08; Link (none) -> https://www.hestore.hu/prod_10049108.html; Url https://hu.farnell.com/vishay/wfma2512r0250fea/res-0r025-3w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 -> (none)
- R28: Cikkszám (none) -> 100.491.05; Link (none) -> https://www.hestore.hu/prod_10049105.html; Url https://hu.farnell.com/vishay/wfma2512r0250fea/res-0r025-3w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 -> (none)
- R29, R30, R33: Cikkszám (none) -> 100.467.55; Link (none) -> https://www.hestore.hu/prod_10046755.html; Url https://hu.farnell.com/vishay/wfma2512r0250fea/res-0r025-3w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 -> (none)
- U10, U11, U12, U13, U14, U15, U16, U17, U18, U19, U20, U5, U6, U7, U8, U9: Cikkszám (none) -> 100.491.20; Link (none) -> https://www.hestore.hu/prod_10049120.html
