File: Circuit/kicad/V4/psu_motor-controll/PCA9531PW.kicad_sch (KiCad schematic)
At the start: 12 parts, among them J2 Conn_01x12, U3 PCA9685PW

Commit message: kicad v4 psu pcb clean
Parts:
- renumbered J2 to J1
Changed lines of the file:
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@@
 		(on_board yes)
 		(dnp no)
-		(property "Reference" "#PWR020"
+		(property "Reference" "#PWR018"
 			(at 182.88 34.29 0)
 			(effects
@@
 			(project "psu"
 				(path "/e63e39d7-6ac0-4ffd-8aa3-1841a4541b55/12f3a577-813a-4f19-bedd-d568a50cedd9"
-					(reference "#PWR020")
+					(reference "#PWR018")
 					(unit 1)
 				)
@@
 		(on_board yes)
 		(dnp no)
-		(property "Reference" "#PWR021"
+		(property "Reference" "#PWR020"
 			(at 182.88 43.18 0)
 			(effects
@@
 			(project "psu"
 				(path "/e63e39d7-6ac0-4ffd-8aa3-1841a4541b55/12f3a577-813a-4f19-bedd-d568a50cedd9"
-					(reference "#PWR021")
+					(reference "#PWR020")
 					(unit 1)
 				)
@@
 		(on_board yes)
 		(dnp no)
-		(property "Reference" "#PWR023"
+		(property "Reference" "#PWR022"
 			(at 182.88 63.5 0)
 			(effects
@@
 			(project "psu"
 				(path "/e63e39d7-6ac0-4ffd-8aa3-1841a4541b55/12f3a577-813a-4f19-bedd-d568a50cedd9"
-					(reference "#PWR023")
+					(reference "#PWR022")
 					(unit 1)
 				)
@@
 		(on_board yes)
 		(dnp no)
-		(property "Reference" "#PWR015"
+		(property "Reference" "#PWR019"
 			(at 107.95 44.45 0)
 			(effects
@@
 			(project "psu"
 				(path "/e63e39d7-6ac0-4ffd-8aa3-1841a4541b55/12f3a577-813a-4f19-bedd-d568a50cedd9"
-					(reference "#PWR015")
+					(reference "#PWR019")
 					(unit 1)
 				)
@@
 		(on_board yes)
 		(dnp no)
-		(property "Reference" "#PWR017"
+		(property "Reference" "#PWR024"
 			(at 118.11 104.14 0)
 			(effects
@@
 			(project "psu"
 				(path "/e63e39d7-6ac0-4ffd-8aa3-1841a4541b55/12f3a577-813a-4f19-bedd-d568a50cedd9"
-					(reference "#PWR017")
+					(reference "#PWR024")
 					(unit 1)
 				)
@@
 		(on_board yes)
 		(dnp no)
-		(property "Reference" "#PWR018"
+		(property "Reference" "#PWR023"
 			(at 125.73 73.66 0)
 			(effects
@@
 			(project "psu"
 				(path "/e63e39d7-6ac0-4ffd-8aa3-1841a4541b55/12f3a577-813a-4f19-bedd-d568a50cedd9"
-					(reference "#PWR018")
+					(reference "#PWR023")
 					(unit 1)
 				)
@@
 		(on_board yes)
 		(dnp no)
-		(property "Reference" "#PWR016"
+		(property "Reference" "#PWR025"
 			(at 101.6 109.22 0)
 			(effects
@@
 			(project "psu"
 				(path "/e63e39d7-6ac0-4ffd-8aa3-1841a4541b55/12f3a577-813a-4f19-bedd-d568a50cedd9"
-					(reference "#PWR016")
+					(reference "#PWR025")
 					(unit 1)
 				)
@@
 		(on_board yes)
 		(dnp no)
-		(property "Reference" "#PWR019"
+		(property "Reference" "#PWR026"
 			(at 140.97 134.62 0)
 			(effects
@@
 			(project "psu"
 				(path "/e63e39d7-6ac0-4ffd-8aa3-1841a4541b55/12f3a577-813a-4f19-bedd-d568a50cedd9"
-					(reference "#PWR019")
+					(reference "#PWR026")
 					(unit 1)
 				)
@@
 		(on_board yes)
 		(dnp no)
-		(property "Reference" "#PWR022"
+		(property "Reference" "#PWR021"
 			(at 182.88 53.34 0)
 			(effects
@@
 			(project "psu"
 				(path "/e63e39d7-6ac0-4ffd-8aa3-1841a4541b55/12f3a577-813a-4f19-bedd-d568a50cedd9"
-					(reference "#PWR022")
+					(reference "#PWR021")
 					(unit 1)
 				)
@@
 		(dnp no)
 		(fields_autoplaced yes)
-		(property "Reference" "J2"
+		(property "Reference" "J1"
 			(at 198.12 105.4099 0)
 			(effects
@@
 			(project "psu"
 				(path "/e63e39d7-6ac0-4ffd-8aa3-1841a4541b55/12f3a577-813a-4f19-bedd-d568a50cedd9"
-					(reference "J2")
-					(unit 1)
-				)
+					(reference "J1")
+					(unit 1)
+				)

Commit message: kicad psu pcb finish psu
Parts:
- removed C12: 1uf, Capacitor_SMD:C_0805_2012Metric, symbol Device:C
Connections:
- net SM1_PWM: now also U3.9 (LED3); no longer U3.6 (LED0)
- net SM2_PWM: now also U3.8 (LED2); no longer U3.7 (LED1)
- net SM3_PWM: now also U3.7 (LED1); no longer U3.8 (LED2)
- net SM4_PWM: now also U3.6 (LED0); no longer U3.9 (LED3)
- net at U3.10 (LED4): now also J1.12 (Pin_12); no longer J1.1 (Pin_1)
- net at U3.11 (LED5): now also J1.11 (Pin_11); no longer J1.2 (Pin_2)
- net at U3.12 (LED6): now also J1.10 (Pin_10); no longer J1.3 (Pin_3)
- net at U3.13 (LED7): now also J1.9 (Pin_9); no longer J1.4 (Pin_4)
- net at U3.15 (LED8): now also J1.8 (Pin_8); no longer J1.5 (Pin_5)
- net at U3.16 (LED9): now also J1.7 (Pin_7); no longer J1.6 (Pin_6)
- net at U3.17 (LED10): now also J1.6 (Pin_6); no longer J1.7 (Pin_7)
- net at U3.18 (LED11): now also J1.5 (Pin_5); no longer J1.8 (Pin_8)
- net at U3.19 (LED12): now also J1.4 (Pin_4); no longer J1.9 (Pin_9)
- net at U3.20 (LED13): now also J1.3 (Pin_3); no longer J1.10 (Pin_10)
- net at U3.21 (LED14): now also J1.2 (Pin_2); no longer J1.11 (Pin_11)
- net at U3.22 (LED15): now also J1.1 (Pin_1); no longer J1.12 (Pin_12)
Changed lines of the file:
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@@
 	(wire
 		(pts
-			(xy 125.73 59.69) (xy 125.73 55.88)
+			(xy 165.1 40.64) (xy 189.23 40.64)
 		)
 		(stroke
@@
 	(wire
 		(pts
-			(xy 165.1 40.64) (xy 189.23 40.64)
+			(xy 107.95 35.56) (xy 120.65 35.56)
 		)
 		(stroke
@@
 		)
 	)
-	(wire
-		(pts
-			(xy 107.95 35.56) (xy 120.65 35.56)
-		)
-		(stroke
-			(width 0)
-			(type default)
-		)
-	)
 	(label "SM4_PWM"
 		(at 165.1 60.96 0)
@@
 	)
 	(label "SM2_PWM"
+		(at 171.45 87.63 180)
+		(effects
+			(font
+				(size 1.27 1.27)
+			)
+			(justify right bottom)
+		)
+	)
+	(label "SM1_PWM"
+		(at 171.45 90.17 180)
+		(effects
+			(font
+				(size 1.27 1.27)
+			)
+			(justify right bottom)
+		)
+	)
+	(label "SM3_PWM"
 		(at 171.45 85.09 180)
-		(effects
-			(font
-				(size 1.27 1.27)
-			)
-			(justify right bottom)
-		)
-	)
-	(label "SM1_PWM"
-		(at 171.45 82.55 180)
-		(effects
-			(font
-				(size 1.27 1.27)
-			)
-			(justify right bottom)
-		)
-	)
-	(label "SM3_PWM"
-		(at 171.45 87.63 180)
 		(effects
 			(font
@@
 	)
 	(label "SM4_PWM"
-		(at 171.45 90.17 180)
+		(at 171.45 82.55 180)
 		(effects
 			(font
@@
 		(shape input)
 		(at 123.19 85.09 180)
-		(effects
-			(font
-				(size 1.27 1.27)
-			)
-			(justify right)
-		)
-	)
-	(hierarchical_label "3v3_in"
-		(shape input)
-		(at 125.73 55.88 180)
 		(effects
 			(font
@@
 	)
 	(symbol
-		(lib_id "Device:C")
-		(at 125.73 63.5 0)
-		(unit 1)
-		(exclude_from_sim no)
-		(in_bom yes)
-		(on_board yes)
-		(dnp no)
-		(fields_autoplaced yes)
-		(property "Reference" "C12"
-			(at 129.54 62.2299 0)
-			(effects
-				(font
-					(size 1.27 1.27)
-				)
-				(justify left)
-			)
-		)
-		(property "Value" "1uf"
-			(at 129.54 64.7699 0)
-			(effects
-				(font
-					(size 1.27 1.27)
-				)
-				(justify left)
-			)
-		)
-		(property "Footprint" "Capacitor_SMD:C_0805_2012Metric"
-			(at 126.6952 67.31 0)
-			(effects
-				(font
-					(size 1.27 1.27)
-				)
-				(hide yes)
-			)
-		)
-		(property "Datasheet" "~"
-			(at 125.73 63.5 0)
-			(effects
-				(font
-					(size 1.27 1.27)
-				)
-				(hide yes)
-			)
-		)
-		(property "Description" "Unpolarized capacitor"
-			(at 125.73 63.5 0)
-			(effects
-				(font
-					(size 1.27 1.27)
-				)
-				(hide yes)
-			)
-		)
-		(property "Sim.Device" ""
-			(at 125.73 63.5 0)
-			(effects
-				(font
-					(size 1.27 1.27)
-				)
-				(hide yes)
-			)
-		)
-		(property "Sim.Type" ""
-			(at 125.73 63.5 0)
-			(effects
-				(font
-					(size 1.27 1.27)
-				)
-				(hide yes)
-			)
-		)
-		(pin "1"
-		)
-		(pin "2"
-		)
-		(instances
-			(project "psu"
-				(path "/e63e39d7-6ac0-4ffd-8aa3-1841a4541b55/12f3a577-813a-4f19-bedd-d568a50cedd9"
-					(reference "C12")
-					(unit 1)
-				)
-			)
-		)
-	)
-	(symbol
 		(lib_id "power:GND")
 		(at 118.11 97.79 0)
@@
 				(path "/e63e39d7-6ac0-4ffd-8aa3-1841a4541b55/12f3a577-813a-4f19-bedd-d568a50cedd9"
 					(reference "#PWR024")
-					(unit 1)
-				)
-			)
-		)
-	)
-	(symbol
-		(lib_id "power:GND")
-		(at 125.73 67.31 0)
-		(unit 1)
-		(exclude_from_sim no)
-		(in_bom yes)
-		(on_board yes)
-		(dnp no)
-		(property "Reference" "#PWR023"
-			(at 125.73 73.66 0)
-			(effects
-				(font
-					(size 1.27 1.27)
-				)
-				(hide yes)
-			)
-		)
-		(property "Value" "GND"
-			(at 125.857 71.7042 0)
-			(effects
-				(font
-					(size 1.27 1.27)
-				)
-			)
-		)
-		(property "Footprint" ""
-			(at 125.73 67.31 0)
-			(effects
-				(font
-					(size 1.27 1.27)
-				)
-				(hide yes)
-			)
-		)
-		(property "Datasheet" ""
-			(at 125.73 67.31 0)
-			(effects
-				(font
-					(size 1.27 1.27)
-				)
-				(hide yes)
-			)
-		)
-		(property "Description" "Power symbol creates a global label with name \"GND\" , ground"
-			(at 125.73 67.31 0)
-			(effects
-				(font
-					(size 1.27 1.27)
-				)
-				(hide yes)
-			)
-		)
-		(pin "1"
-		)
-		(instances
-			(project "psu"
-				(path "/e63e39d7-6ac0-4ffd-8aa3-1841a4541b55/12f3a577-813a-4f19-bedd-d568a50cedd9"
-					(reference "#PWR023")
 					(unit 1)
 				)
@@
 	(symbol
 		(lib_id "Connector_Generic:Conn_01x12")
-		(at 195.58 105.41 0)
+		(at 195.58 107.95 0)
+		(mirror x)
 		(unit 1)
 		(exclude_from_sim no)
@@
 		(on_board yes)
 		(dnp no)
-		(fields_autoplaced yes)
 		(property "Reference" "J1"
-			(at 198.12 105.4099 0)
+			(at 198.12 107.9501 0)
 			(effects
 				(font
@@
 		)
 		(property "Value" "Conn_01x12"
-			(at 198.12 107.9499 0)
+			(at 198.12 105.4101 0)
 			(effects
 				(font
@@
 		)
 		(property "Footprint" "Connector_PinSocket_2.54mm:PinSocket_1x12_P2.54mm_Vertical"
-			(at 195.58 105.41 0)
+			(at 195.58 107.95 0)
 			(effects
 				(font
@@
 		)
 		(property "Datasheet" "~"
-			(at 195.58 105.41 0)
+			(at 195.58 107.95 0)
 			(effects
 				(font
@@
 		)
 		(property "Description" "Generic connector, single row, 01x12, script generated (kicad-library-utils/schlib/autogen/connector/)"
-			(at 195.58 105.41 0)
+			(at 195.58 107.95 0)
 			(effects
 				(font
@@
 		)
 		(property "Sim.Device" ""
-			(at 195.58 105.41 0)
+			(at 195.58 107.95 0)
 			(effects
 				(font
@@
 		)
 		(property "Sim.Type" ""
-			(at 195.58 105.41 0)
-			(effects
-				(font
+			(at 195.58 107.95 0)
+			(effects
+				(font

Commit message: kicad FINISH PSU PCB
Parts:
- added R67, R68, R69, R70: 220, Resistor_SMD:R_0805_2012Metric, symbol Device:R
Connections:
- net SM1_PWM: now also R70.2; no longer U3.9 (LED3)
- net SM2_PWM: now also R69.2; no longer U3.8 (LED2)
- net SM3_PWM: now also R67.2; no longer U3.7 (LED1)
- net SM4_PWM: now also R68.2; no longer U3.6 (LED0)
- new net: R69.1, U3.8 (LED2)
- new net: R68.1, U3.6 (LED0)
- new net: R67.1, U3.7 (LED1)
- new net: R70.1, U3.9 (LED3)

Commit message: PSU FINISH BOARD NO DRC,ERC,DFM ERRORS
Other:
- moved on the sheet: C10, C11, C8, C9, J1, R15, R67, R68, R69, R70, SERVO1, SERVO2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

Commit message: updated bom, updated compon
Parts:
- J1: Cikkszám (none) -> 100.387.12; Link (none) -> https://www.hestore.hu/prod_10038712.html
- R15: Cikkszám (none) -> 100.011.45; Link (none) -> https://www.hestore.hu/prod_10001145.html
- R67, R68, R69, R70: value 220 -> 220R; Cikkszám (none) -> 100.011.62; Link (none) -> https://www.hestore.hu/prod_10001162.html
- SERVO1, SERVO2, SERVO3, SERVO4: Cikkszám (none) -> 100.491.25; Link (none) -> https://www.hestore.hu/prod_10049125.html
- U3: Cikkszám (none) -> 100.377.68; Link (none) -> https://www.hestore.hu/prod_10037768.html
Changed lines of the file:
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@@
 			)
 		)
-		(property "Sim.Device" ""
+		(property "Cikkszám" ""
 			(at 45.72 29.21 0)
 			(effects
@@
 			)
 		)
-		(property "Sim.Type" ""
+		(property "Link" ""
 			(at 45.72 29.21 0)
 			(effects
@@
 			)
 		)
-		(property "Sim.Device" ""
+		(property "Cikkszám" ""
 			(at 58.42 29.21 0)
 			(effects
@@
 			)
 		)
-		(property "Sim.Type" ""
+		(property "Link" ""
 			(at 58.42 29.21 0)
 			(effects
@@
 			)
 		)
-		(property "Sim.Device" ""
+		(property "Cikkszám" "100.491.25"
 			(at 175.26 68.58 0)
 			(effects
@@
 			)
 		)
-		(property "Sim.Type" ""
+		(property "Link" "https://www.hestore.hu/prod_10049125.html"
 			(at 175.26 68.58 0)
 			(effects
@@
 			)
 		)
-		(property "Sim.Device" ""
+		(property "Cikkszám" ""
 			(at 33.02 29.21 0)
 			(effects
@@
 			)
 		)
-		(property "Sim.Type" ""
+		(property "Link" ""
 			(at 33.02 29.21 0)
 			(effects
@@
 			)
 		)
-		(property "Value" "220"
+		(property "Value" "220R"
 			(at 124.46 59.69 90)
 			(effects
@@
 			)
 		)
-		(property "Sim.Device" ""
+		(property "Cikkszám" "100.011.62"
 			(at 124.46 63.5 90)
 			(effects
@@
 			)
 		)
-		(property "Sim.Type" ""
+		(property "Link" "https://www.hestore.hu/prod_10001162.html"
 			(at 124.46 63.5 90)
 			(effects
@@
 			)
 		)
-		(property "Sim.Device" ""
+		(property "Cikkszám" "100.377.68"
 			(at 53.34 72.39 0)
 			(effects
@@
 			)
 		)
-		(property "Sim.Type" ""
+		(property "Link" "https://www.hestore.hu/prod_10037768.html"
 			(at 53.34 72.39 0)
 			(effects
@@
 			)
 		)
-		(property "Sim.Device" ""
+		(property "Cikkszám" "100.011.45"
 			(at 30.48 66.04 0)
 			(effects
@@
 			)
 		)
-		(property "Sim.Type" ""
+		(property "Link" "https://www.hestore.hu/prod_10001145.html"
 			(at 30.48 66.04 0)
 			(effects
@@
 			)
 		)
-		(property "Value" "220"
+		(property "Value" "220R"
 			(at 124.46 50.8 90)
 			(effects
@@
 			)
 		)
-		(property "Sim.Device" ""
+		(property "Cikkszám" "100.011.62"
 			(at 124.46 54.61 90)
 			(effects
@@
 			)
 		)
-		(property "Sim.Type" ""
+		(property "Link" "https://www.hestore.hu/prod_10001162.html"
 			(at 124.46 54.61 90)
 			(effects
@@
 			)
 		)
-		(property "Sim.Device" ""
+		(property "Cikkszám" "100.491.25"
 			(at 175.26 78.74 0)
 			(effects
@@
 			)
 		)
-		(property "Sim.Type" ""
+		(property "Link" "https://www.hestore.hu/prod_10049125.html"
 			(at 175.26 78.74 0)
 			(effects
@@
 			)
 		)
-		(property "Sim.Device" ""
+		(property "Cikkszám" "100.491.25"
 			(at 175.26 59.69 0)
 			(effects
@@
 			)
 		)
-		(property "Sim.Type" ""
+		(property "Link" "https://www.hestore.hu/prod_10049125.html"
 			(at 175.26 59.69 0)
 			(effects
@@
 			)
 		)
-		(property "Value" "220"
+		(property "Value" "220R"
 			(at 124.46 68.58 90)
 			(effects
@@
 			)
 		)
-		(property "Sim.Device" ""
+		(property "Cikkszám" "100.011.62"
 			(at 124.46 72.39 90)
 			(effects
@@
 			)
 		)
-		(property "Sim.Type" ""
+		(property "Link" "https://www.hestore.hu/prod_10001162.html"
 			(at 124.46 72.39 90)
 			(effects
@@
 			)
 		)
-		(property "Sim.Device" ""
+		(property "Cikkszám" ""
 			(at 71.12 29.21 0)
 			(effects
@@
 			)
 		)
-		(property "Sim.Type" ""
+		(property "Link" ""
 			(at 71.12 29.21 0)
 			(effects
@@
 			)
 		)
-		(property "Value" "220"
+		(property "Value" "220R"
 			(at 124.46 41.91 90)
 			(effects
@@
 			)
 		)
-		(property "Sim.Device" ""
+		(property "Cikkszám" "100.011.62"
 			(at 124.46 45.72 90)
 			(effects
@@
 			)
 		)
-		(property "Sim.Type" ""
+		(property "Link" "https://www.hestore.hu/prod_10001162.html"
 			(at 124.46 45.72 90)
 			(effects
@@
 			)
 		)
-		(property "Sim.Device" ""
+		(property "Cikkszám" "100.491.25"
 			(at 175.26 88.9 0)
 			(effects
@@
 			)
 		)
-		(property "Sim.Type" ""
+		(property "Link" "https://www.hestore.hu/prod_10049125.html"
 			(at 175.26 88.9 0)
 			(effects
@@
 			)
 		)
-		(property "Datasheet" "~"
+		(property "Datasheet" "https://www.hestore.hu/prod_getfile.php?id=10186"
 			(at 107.95 80.01 0)
 			(effects
@@
 			)
 		)
-		(property "Sim.Device" ""
+		(property "Cikkszám" "100.387.12"
 			(at 107.95 80.01 0)
 			(effects
@@
 			)
 		)
-		(property "Sim.Type" ""
+		(property "Link" "https://www.hestore.hu/prod_10038712.html"
 			(at 107.95 80.01 0)
 			(effects
