File: Circuit/kicad/V4/psu_motor-controll/fpp-kábel.kicad_sch (KiCad schematic)
At the start: 1 part, among them J5 Conn_01x60_MountingPin

Commit message: kicad psu pcb finish psu
Parts:
- added TP6, TP7: TestPoint, TestPoint:TestPoint_Pad_D1.0mm, symbol Connector:TestPoint
Connections:
- net GND: no longer J5.20 (Pin_20)
- net I2C_SCL_sensors: now also TP6.1
- net I2C_SDA_sensors: now also TP7.1
- net M1_CS: now also J5.20 (Pin_20); no longer J5.28 (Pin_28)
- net M1_step: now also J5.19 (Pin_19); no longer J5.16 (Pin_16)
- net M2_CS: now also J5.18 (Pin_18); no longer J5.27 (Pin_27)
- net M2_step: now also J5.17 (Pin_17); no longer J5.15 (Pin_15)
- net M3_CS: now also J5.16 (Pin_16); no longer J5.26 (Pin_26)
- net M3_step: now also J5.15 (Pin_15); no longer J5.14 (Pin_14)
- net M4_CS: now also J5.14 (Pin_14); no longer J5.25 (Pin_25)
- net MOSI: now also J5.4 (Pin_4); no longer J5.6 (Pin_6)
- net PWMA: no longer J5.18 (Pin_18)
- net PWMB: no longer J5.17 (Pin_17)
- net SPI_CLK: now also J5.6 (Pin_6); no longer J5.4 (Pin_4)
- net WS_2802B_DATA: no longer J5.19 (Pin_19)

Commit message: psu pcb update
Connections:
- net AIN1: now also J5.25 (Pin_25); no longer J5.24 (Pin_24)
- net AIN2: now also J5.24 (Pin_24); no longer J5.23 (Pin_23)
- net H_EN: now also J5.23 (Pin_23); no longer J5.31 (Pin_31)
Changed lines of the file:
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@@
+		)
+	)
+	(global_label "AIN1"
+		(shape input)
+		(at 31.75 114.3 0)
+		(fields_autoplaced yes)
+		(effects
+			(font
+				(size 1.27 1.27)
+			)
+			(justify left)
+		)
+		(property "Intersheetrefs" "${INTERSHEET_REFS}"
+			(at 39.0637 114.3 0)
+			(effects
+				(font
+					(size 1.27 1.27)
+				)
+				(justify left)
+				(hide yes)
+			)
 		)
 	)
@@
 		)
 	)
+	(global_label "H_EN"
+		(shape input)
+		(at 31.75 119.38 0)
+		(fields_autoplaced yes)
+		(effects
+			(font
+				(size 1.27 1.27)
+			)
+			(justify left)
+		)
+		(property "Intersheetrefs" "${INTERSHEET_REFS}"
+			(at 39.6079 119.38 0)
+			(effects
+				(font
+					(size 1.27 1.27)
+				)
+				(justify left)
+				(hide yes)
+			)
+		)
+	)
 	(global_label "MOSI"
 		(shape input)
@@
 		)
 	)
+	(global_label "AIN2"
+		(shape input)
+		(at 31.75 116.84 0)
+		(fields_autoplaced yes)
+		(effects
+			(font
+				(size 1.27 1.27)
+			)
+			(justify left)
+		)
+		(property "Intersheetrefs" "${INTERSHEET_REFS}"
+			(at 39.0637 116.84 0)
+			(effects
+				(font
+					(size 1.27 1.27)
+				)
+				(justify left)
+				(hide yes)
+			)
+		)
+	)
 	(global_label "M2_step"
 		(shape input)
@@
 		)
 	)
-	(global_label "H_EN"
-		(shape input)
-		(at 31.75 99.06 0)
-		(fields_autoplaced yes)
-		(effects
-			(font
-				(size 1.27 1.27)
-			)
-			(justify left)
-		)
-		(property "Intersheetrefs" "${INTERSHEET_REFS}"
-			(at 39.6079 99.06 0)
-			(effects
-				(font
-					(size 1.27 1.27)
-				)
-				(justify left)
-				(hide yes)
-			)
-		)
-	)
 	(global_label "RPI_5V"
 		(shape input)
@@
 		)
 	)
-	(global_label "AIN2"
-		(shape input)
-		(at 31.75 119.38 0)
-		(fields_autoplaced yes)
-		(effects
-			(font
-				(size 1.27 1.27)
-			)
-			(justify left)
-		)
-		(property "Intersheetrefs" "${INTERSHEET_REFS}"
-			(at 39.0637 119.38 0)
-			(effects
-				(font
-					(size 1.27 1.27)
-				)
-				(justify left)
-				(hide yes)
-			)
-		)
-	)
 	(global_label "ESP_5v"
 		(shape input)
@@
 			(effects
 				(font
-					(size 1.27 1.27)
-				)
-				(justify left)
-				(hide yes)
-			)
-		)
-	)
-	(global_label "AIN1"
-		(shape input)
-		(at 31.75 116.84 0)
-		(fields_autoplaced yes)
-		(effects
-			(font
-				(size 1.27 1.27)
-			)
-			(justify left)
-		)
-		(property "Intersheetrefs" "${INTERSHEET_REFS}"
-			(at 39.0637 116.84 0)
-			(effects
-				(font

Commit message: kicad FINISH PSU PCB
Connections:
- net H_EN is gone; now on net AIN2: J5.23 (Pin_23)
- net AIN1: now also J5.24 (Pin_24); no longer J5.25 (Pin_25)
- net AIN2: no longer J5.24 (Pin_24)
- net GND: now also J5.27 (Pin_27), J5.28 (Pin_28)
- net PWMA: now also J5.26 (Pin_26)
- net PWMB: now also J5.25 (Pin_25)
- net WS_2802B_DATA: now also J5.31 (Pin_31)

Commit message: PSU bugfixes
Parts:
- added C12, C20, C7: ha kell pár pf, Capacitor_SMD:C_0805_2012Metric, symbol Device:C
- added R71, R72, R73: 330, Resistor_SMD:R_0805_2012Metric, symbol Device:R
- renumbered TP6 to SCL1, TP7 to SDA1
Connections:
- net GND: now also C12.2, C20.2, C7.2
- net MISO: now also C20.1, R73.2; no longer J5.2 (Pin_2)
- net MOSI: now also C12.1, R72.2; no longer J5.4 (Pin_4)
- net SPI_CLK: now also C7.1, R71.2; no longer J5.6 (Pin_6)
- new net: J5.4 (Pin_4), R72.1
- new net: J5.2 (Pin_2), R73.1
- new net: J5.6 (Pin_6), R71.1
Other:
- moved on the sheet: SCL1, SDA1

Commit message: updated bom, updated compon
Parts:
- C12, C20, C7: value ha kell pár pf -> 1nf; Cikkszám (none) -> 100.277.92; Link (none) -> https://www.hestore.hu/prod_10027792.html
- J5: Cikkszám (none) -> ?; Link (none) -> https://www.tme.eu/en/details/fh28k-60s-05sh-98/connectors-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
- R71, R72, R73: Cikkszám (none) -> 100.011.70; Link (none) -> https://www.hestore.hu/prod_10001170.html
- SCL1, SDA1: now left out of the parts list
Changed lines of the file:
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@@
 			)
 		)
-		(property "Value" "ha kell pár pf"
+		(property "Value" "1nf"
 			(at 118.11 144.7799 0)
 			(effects
@@
 			)
 		)
-		(property "Sim.Device" ""
+		(property "Cikkszám" "100.277.92"
 			(at 114.3 143.51 0)
 			(effects
@@
 			)
 		)
-		(property "Sim.Type" ""
+		(property "Link" "https://www.hestore.hu/prod_10027792.html"
 			(at 114.3 143.51 0)
 			(effects
@@
 			)
 		)
-		(property "Datasheet" "~"
+		(property "Datasheet" "https://www.hestore.hu/prod_getfile.php?id=3657"
 			(at 68.58 167.64 0)
 			(effects
@@
 			)
 		)
-		(property "Sim.Device" ""
+		(property "Cikkszám" "100.011.70"
 			(at 68.58 167.64 90)
 			(effects
@@
 			)
 		)
-		(property "Sim.Type" ""
+		(property "Link" "https://www.hestore.hu/prod_10001170.html"
 			(at 68.58 167.64 90)
 			(effects
@@
 			)
 		)
-		(property "Value" "ha kell pár pf"
+		(property "Value" "1nf"
 			(at 168.91 144.7799 0)
 			(effects
@@
 			)
 		)
-		(property "Sim.Device" ""
+		(property "Cikkszám" "100.277.92"
 			(at 165.1 143.51 0)
 			(effects
@@
 			)
 		)
-		(property "Sim.Type" ""
+		(property "Link" "https://www.hestore.hu/prod_10027792.html"
 			(at 165.1 143.51 0)
 			(effects
@@
 		(unit 1)
 		(exclude_from_sim no)
-		(in_bom yes)
+		(in_bom no)
 		(on_board yes)
 		(dnp no)
@@
 			)
 		)
+		(property "Cikkszám" ""
+			(at 68.58 124.46 0)
+			(effects
+				(font
+					(size 1.27 1.27)
+				)
+				(hide yes)
+			)
+		)
+		(property "Link" ""
+			(at 68.58 124.46 0)
+			(effects
+				(font
+					(size 1.27 1.27)
+				)
+				(hide yes)
+			)
+		)
 		(pin "1"
 		)
@@
 		(unit 1)
 		(exclude_from_sim no)
-		(in_bom yes)
+		(in_bom no)
 		(on_board yes)
 		(dnp no)
@@
 		)
 		(property "Description" "test point"
+			(at 68.58 135.89 0)
+			(effects
+				(font
+					(size 1.27 1.27)
+				)
+				(hide yes)
+			)
+		)
+		(property "Cikkszám" ""
+			(at 68.58 135.89 0)
+			(effects
+				(font
+					(size 1.27 1.27)
+				)
+				(hide yes)
+			)
+		)
+		(property "Link" ""
 			(at 68.58 135.89 0)
 			(effects
@@
 			)
 		)
-		(property "Datasheet" "~"
+		(property "Datasheet" "https://www.hestore.hu/prod_getfile.php?id=3657"
 			(at 68.58 177.8 0)
 			(effects
@@
 			)
 		)
-		(property "Sim.Device" ""
+		(property "Cikkszám" "100.011.70"
 			(at 68.58 177.8 90)
 			(effects
@@
 			)
 		)
-		(property "Sim.Type" ""
+		(property "Link" "https://www.hestore.hu/prod_10001170.html"
 			(at 68.58 177.8 90)
 			(effects
@@
 			)
 		)
-		(property "Datasheet" "~"
+		(property "Datasheet" "https://www.hestore.hu/prod_getfile.php?id=3657"
 			(at 68.58 157.48 0)
 			(effects
@@
 			)
 		)
-		(property "Sim.Device" ""
+		(property "Cikkszám" "100.011.70"
 			(at 68.58 157.48 90)
 			(effects
@@
 			)
 		)
-		(property "Sim.Type" ""
+		(property "Link" "https://www.hestore.hu/prod_10001170.html"
 			(at 68.58 157.48 90)
 			(effects
@@
 			)
 		)
-		(property "Value" "ha kell pár pf"
+		(property "Value" "1nf"
 			(at 143.51 144.7799 0)
 			(effects
@@
 			)
 		)
-		(property "Sim.Device" ""
+		(property "Cikkszám" "100.277.92"
 			(at 139.7 143.51 0)
 			(effects
@@
 			)
 		)
-		(property "Sim.Type" ""
+		(property "Link" "https://www.hestore.hu/prod_10027792.html"
 			(at 139.7 143.51 0)
 			(effects
@@
 			)
 		)
-		(property "Sim.Device" ""
+		(property "Cikkszám" "?"
 			(at 19.05 101.6 0)
 			(effects
@@
 			)
 		)
-		(property "Sim.Type" ""
+		(property "Link" "https://www.tme.eu/en/details/fh28k-60s-05sh-98/connectors-ffc-fpc-0-5mm/hirose/fh28k-60s-0-5sh-98/"
 			(at 19.05 101.6 0)
 			(effects

Commit message: kicad
Parts:
- removed J5: Conn_01x60_MountingPin, Connector_FFC-FPC:Amphenol_F32Q-1A7x1-11060_1x60-1MP_P0.5mm_Horizontal, symbol Connector_Generic_MountingPin:Conn_01x60_MountingPin
- added FFC_NC1, FFC_NC2, FFC_NC3, FFC_NC4, FFC_NC5: TestPoint, TestPoint:TestPoint_Pad_D1.0mm, symbol Connector:TestPoint
- added J5: Conn_01x40_MountingPin, Connector_FFC-FPC:Amphenol_F32Q-1A7x1-11040_1x40-1MP_P0.5mm_Horizontal, symbol Connector_Generic_MountingPin:Conn_01x40_MountingPin
- added J6: Conn_02x04_Counter_Clockwise, Connector_Molex:Molex_Micro-Fit_3.0_43045-0812_2x04_P3.00mm_Vertical, symbol Connector_Generic:Conn_02x04_Counter_Clockwise
Connections:
- net 3V3_M.2: now also J6.4 (Pin_4)
- net AIN1: now also J5.25 (Pin_25)
- net AIN2: now also J5.24 (Pin_24)
- net BIN1: now also J5.23 (Pin_23)
- net BIN2: now also J5.22 (Pin_22)
- net ESP_3v3: now also J6.8 (Pin_8)
- net ESP_5v: now also J6.7 (Pin_7)
- net GND: now also J5.1 (Pin_1), J5.10 (Pin_10), J5.13 (Pin_13), J5.28 (Pin_28), J5.3 (Pin_3), J5.34 (Pin_34), J5.40 (Pin_40), J5.5 (Pin_5), J5.7 (Pin_7), J5.MP (MountPin), J6.1 (Pin_1), J6.2 (Pin_2), J6.3 (Pin_3)
- net I2C_SCL_sensors: now also J5.9 (Pin_9)
- net I2C_SDA_sensors: now also J5.8 (Pin_8)
- net INA226_ALERT: now also J5.33 (Pin_33)
- net INA226_SCL: now also J5.12 (Pin_12)
- net INA226_SDA: now also J5.11 (Pin_11)
- net M1_CS: now also J5.21 (Pin_21)
- net M1_step: now also J5.20 (Pin_20)
- net M2_CS: now also J5.19 (Pin_19)
- net M2_step: now also J5.18 (Pin_18)
- net M3_CS: now also J5.17 (Pin_17)
- net M3_step: now also J5.16 (Pin_16)
- net M4_CS: now also J5.15 (Pin_15)
- net M4_step: now also J5.14 (Pin_14)
- net MCP_CS: now also J5.29 (Pin_29)
- net MCP_RST: now also J5.30 (Pin_30)
- net PWMA: now also J5.27 (Pin_27)
- net PWMB: now also J5.26 (Pin_26)
- net RPI_5V: now also J6.6 (Pin_6)
- net TPA_ON: now also J5.32 (Pin_32)
- net USB_5V: now also J6.5 (Pin_5)
- net WS_2802B_DATA: now also J5.31 (Pin_31)
- net at R72.1: now also J5.4 (Pin_4)
- net at R73.1: now also J5.2 (Pin_2)
- net at R71.1: now also J5.6 (Pin_6)
- new net: FFC_NC2.1, J5.37 (Pin_37)
- new net: FFC_NC1.1, J5.38 (Pin_38)
- new net: FFC_NC5.1, J5.39 (Pin_39)
- new net: FFC_NC3.1, J5.36 (Pin_36)
- new net: FFC_NC4.1, J5.35 (Pin_35)
Other:
- moved on the sheet: SCL1, SDA1
