File: Circuit/kicad/V4/psu_motor-controll/4x tmc5160.kicad_sch (KiCad schematic)
At the start: 28 parts, among them M1 Stepper_Motor_unipolar_6pin, M2 Stepper_Motor_unipolar_6pin, M3 Stepper_Motor_unipolar_6pin, M4 Stepper_Motor_unipolar_6pin

Commit message: kicad v4 psu pcb clean
Parts:
- renumbered D4 to D3, D3 to D4
Changed lines of the file:
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@@
 		(dnp no)
 		(fields_autoplaced yes)
-		(property "Reference" "#PWR06"
+		(property "Reference" "#PWR07"
 			(at 81.28 78.74 0)
 			(effects
@@
 			(project ""
 				(path "/e63e39d7-6ac0-4ffd-8aa3-1841a4541b55/d1e0c7e2-68f3-4828-b2d5-d40ec13307ce"
-					(reference "#PWR06")
+					(reference "#PWR07")
 					(unit 1)
 				)
@@
 		(dnp no)
 		(fields_autoplaced yes)
-		(property "Reference" "#PWR013"
+		(property "Reference" "#PWR014"
 			(at 214.63 152.4 0)
 			(effects
@@
 			(project "psu"
 				(path "/e63e39d7-6ac0-4ffd-8aa3-1841a4541b55/d1e0c7e2-68f3-4828-b2d5-d40ec13307ce"
-					(reference "#PWR013")
+					(reference "#PWR014")
 					(unit 1)
 				)
@@
 		(dnp no)
 		(fields_autoplaced yes)
-		(property "Reference" "#PWR02"
+		(property "Reference" "#PWR03"
 			(at 74.93 26.67 0)
 			(effects
@@
 			(project "psu"
 				(path "/e63e39d7-6ac0-4ffd-8aa3-1841a4541b55/d1e0c7e2-68f3-4828-b2d5-d40ec13307ce"
-					(reference "#PWR02")
+					(reference "#PWR03")
 					(unit 1)
 				)
@@
 		(dnp no)
 		(fields_autoplaced yes)
-		(property "Reference" "#PWR08"
+		(property "Reference" "#PWR09"
 			(at 74.93 100.33 0)
 			(effects
@@
 			(project "psu"
 				(path "/e63e39d7-6ac0-4ffd-8aa3-1841a4541b55/d1e0c7e2-68f3-4828-b2d5-d40ec13307ce"
-					(reference "#PWR08")
+					(reference "#PWR09")
 					(unit 1)
 				)
@@
 		(dnp no)
 		(fields_autoplaced yes)
-		(property "Reference" "#PWR03"
+		(property "Reference" "#PWR04"
 			(at 208.28 26.67 0)
 			(effects
@@
 			(project "psu"
 				(path "/e63e39d7-6ac0-4ffd-8aa3-1841a4541b55/d1e0c7e2-68f3-4828-b2d5-d40ec13307ce"
-					(reference "#PWR03")
+					(reference "#PWR04")
 					(unit 1)
 				)
@@
 		(dnp no)
 		(fields_autoplaced yes)
-		(property "Reference" "D4"
+		(property "Reference" "D3"
 			(at 97.4725 114.3 0)
 			(effects
@@
 			(project "psu"
 				(path "/e63e39d7-6ac0-4ffd-8aa3-1841a4541b55/d1e0c7e2-68f3-4828-b2d5-d40ec13307ce"
-					(reference "D4")
+					(reference "D3")
 					(unit 1)
 				)
@@
 		(dnp no)
 		(fields_autoplaced yes)
-		(property "Reference" "#PWR012"
+		(property "Reference" "#PWR013"
 			(at 81.28 152.4 0)
 			(effects
@@
 			(project "psu"
 				(path "/e63e39d7-6ac0-4ffd-8aa3-1841a4541b55/d1e0c7e2-68f3-4828-b2d5-d40ec13307ce"
-					(reference "#PWR012")
+					(reference "#PWR013")
 					(unit 1)
 				)
@@
 		(dnp no)
 		(fields_autoplaced yes)
-		(property "Reference" "#PWR09"
+		(property "Reference" "#PWR010"
 			(at 208.28 100.33 0)
 			(effects
@@
 			(project "psu"
 				(path "/e63e39d7-6ac0-4ffd-8aa3-1841a4541b55/d1e0c7e2-68f3-4828-b2d5-d40ec13307ce"
-					(reference "#PWR09")
+					(reference "#PWR010")
 					(unit 1)
 				)
@@
 		(dnp no)
 		(fields_autoplaced yes)
-		(property "Reference" "#PWR05"
+		(property "Reference" "#PWR06"
 			(at 167.64 31.75 0)
 			(effects
@@
 			(project "psu"
 				(path "/e63e39d7-6ac0-4ffd-8aa3-1841a4541b55/d1e0c7e2-68f3-4828-b2d5-d40ec13307ce"
-					(reference "#PWR05")
+					(reference "#PWR06")
 					(unit 1)
 				)
@@
 		(dnp no)
 		(fields_autoplaced yes)
-		(property "Reference" "#PWR07"
+		(property "Reference" "#PWR08"
 			(at 214.63 78.74 0)
 			(effects
@@
 			(project "psu"
 				(path "/e63e39d7-6ac0-4ffd-8aa3-1841a4541b55/d1e0c7e2-68f3-4828-b2d5-d40ec13307ce"
-					(reference "#PWR07")
+					(reference "#PWR08")
 					(unit 1)
 				)
@@
 		(dnp no)
 		(fields_autoplaced yes)
-		(property "Reference" "#PWR04"
+		(property "Reference" "#PWR05"
 			(at 35.56 31.75 0)
 			(effects
@@
 			(project "psu"
 				(path "/e63e39d7-6ac0-4ffd-8aa3-1841a4541b55/d1e0c7e2-68f3-4828-b2d5-d40ec13307ce"
-					(reference "#PWR04")
+					(reference "#PWR05")
 					(unit 1)
 				)
@@
 		(dnp no)
 		(fields_autoplaced yes)
-		(property "Reference" "#PWR011"
+		(property "Reference" "#PWR012"
 			(at 167.64 105.41 0)
 			(effects
@@
 			(project "psu"
 				(path "/e63e39d7-6ac0-4ffd-8aa3-1841a4541b55/d1e0c7e2-68f3-4828-b2d5-d40ec13307ce"
-					(reference "#PWR011")
+					(reference "#PWR012")
 					(unit 1)
 				)
@@
 		(dnp no)
 		(fields_autoplaced yes)
-		(property "Reference" "D3"
+		(property "Reference" "D4"
 			(at 230.8225 114.3 0)
 			(effects
@@
 			(project "psu"
 				(path "/e63e39d7-6ac0-4ffd-8aa3-1841a4541b55/d1e0c7e2-68f3-4828-b2d5-d40ec13307ce"
-					(reference "D3")
+					(reference "D4")
 					(unit 1)
 				)
@@
 		(dnp no)
 		(fields_autoplaced yes)
-		(property "Reference" "#PWR010"
+		(property "Reference" "#PWR011"
 			(at 34.29 105.41 0)
 			(effects
@@
 			(project "psu"
 				(path "/e63e39d7-6ac0-4ffd-8aa3-1841a4541b55/d1e0c7e2-68f3-4828-b2d5-d40ec13307ce"
-					(reference "#PWR010")
-					(unit 1)
-				)
+					(reference "#PWR011")
+					(unit 1)
+				)

Commit message: updated bom, updated compon
Parts:
- C1, C2, C3, C4: Cikkszám (none) -> 100.392.15; Link (none) -> https://www.hestore.hu/prod_10039215.html
- D1, D2, D3, D4: Cikkszám (none) -> 100.365.90; Link (none) -> https://www.hestore.hu/prod_10036590.html
- M1, M2, M3, M4: Cikkszám (none) -> 100.491.16; Link (none) -> https://www.hestore.hu/prod_10049116.html
- R10, R11, R12, R3, R4, R5, R6, R9: Cikkszám (none) -> 100.011.45; Link (none) -> https://www.hestore.hu/prod_10001145.html
- R13, R14, R7, R8: Cikkszám (none) -> 100.011.70; Link (none) -> https://www.hestore.hu/prod_10001170.html
- TMC1, TMC2, TMC3, TMC4: value ~ -> 2*8pin socket; Cikkszám (none) -> 100.280.57; Link (none) -> https://www.hestore.hu/prod_10028057.html

Commit message: FINISH PSU V1.4.9 to production 1
Parts:
- TMC1, TMC2, TMC3, TMC4: footprint psu:TMC2209 -> panel:TMC2209
Connections:
- net TMC_MISO: now also TMC1.12 (MISO), TMC2.12 (MISO), TMC3.12 (MISO), TMC4.12 (MISO); no longer TMC1.11 (MISO), TMC2.11 (MISO), TMC3.11 (MISO), TMC4.11 (MISO)
