File: Circuit/kicad/V4/psu_motor-controll/Battery-circuit.kicad_sch (KiCad schematic)
At the start: 12 parts, among them J6 Charge, Q2 IRFR7546TRPBF, Q3 IRFR7546TRPBF

Commit message: kicad v4 psu pcb clean
Parts:
- renumbered C75 to C13, C76 to C14, C77 to C15, D10 to D5, J3 to J2, J6 to J3, R64 to R16, R65 to R17, R66 to R18
Changed lines of the file:
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@@
 		(on_board yes)
 		(dnp no)
-		(property "Reference" "J3"
+		(property "Reference" "J2"
 			(at 90.17 102.87 0)
 			(effects
@@
 			(project "psu"
 				(path "/e63e39d7-6ac0-4ffd-8aa3-1841a4541b55/4c1824a3-ede3-44a9-9cc4-1658cb86e3ae/681cd5e3-d1a9-4f5a-899b-9dce52990abf"
-					(reference "J3")
+					(reference "J2")
 					(unit 1)
 				)
@@
 		(dnp no)
 		(fields_autoplaced yes)
-		(property "Reference" "#PWR0116"
+		(property "Reference" "#PWR031"
 			(at 177.8 118.11 0)
 			(effects
@@
 			(project "psu"
 				(path "/e63e39d7-6ac0-4ffd-8aa3-1841a4541b55/4c1824a3-ede3-44a9-9cc4-1658cb86e3ae/681cd5e3-d1a9-4f5a-899b-9dce52990abf"
-					(reference "#PWR0116")
+					(reference "#PWR031")
 					(unit 1)
 				)
@@
 		(dnp no)
 		(fields_autoplaced yes)
-		(property "Reference" "J6"
+		(property "Reference" "J3"
 			(at 109.855 97.79 0)
 			(effects
@@
 			(project ""
 				(path "/e63e39d7-6ac0-4ffd-8aa3-1841a4541b55/4c1824a3-ede3-44a9-9cc4-1658cb86e3ae/681cd5e3-d1a9-4f5a-899b-9dce52990abf"
-					(reference "J6")
+					(reference "J3")
 					(unit 1)
 				)
@@
 		(dnp no)
 		(fields_autoplaced yes)
-		(property "Reference" "R66"
+		(property "Reference" "R18"
 			(at 135.89 107.95 90)
 			(effects
@@
 			(project ""
 				(path "/e63e39d7-6ac0-4ffd-8aa3-1841a4541b55/4c1824a3-ede3-44a9-9cc4-1658cb86e3ae/681cd5e3-d1a9-4f5a-899b-9dce52990abf"
-					(reference "R66")
+					(reference "R18")
 					(unit 1)
 				)
@@
 		(on_board yes)
 		(dnp no)
-		(property "Reference" "R65"
+		(property "Reference" "R17"
 			(at 151.892 99.314 0)
 			(effects
@@
 			(project "psu"
 				(path "/e63e39d7-6ac0-4ffd-8aa3-1841a4541b55/4c1824a3-ede3-44a9-9cc4-1658cb86e3ae/681cd5e3-d1a9-4f5a-899b-9dce52990abf"
-					(reference "R65")
+					(reference "R17")
 					(unit 1)
 				)
@@
 		(dnp no)
 		(fields_autoplaced yes)
-		(property "Reference" "C75"
+		(property "Reference" "C13"
 			(at 187.96 83.8199 0)
 			(effects
@@
 			(project "psu"
 				(path "/e63e39d7-6ac0-4ffd-8aa3-1841a4541b55/4c1824a3-ede3-44a9-9cc4-1658cb86e3ae/681cd5e3-d1a9-4f5a-899b-9dce52990abf"
-					(reference "C75")
+					(reference "C13")
 					(unit 1)
 				)
@@
 		(dnp no)
 		(fields_autoplaced yes)
-		(property "Reference" "R64"
+		(property "Reference" "R16"
 			(at 142.24 83.8199 0)
 			(effects
@@
 			(project ""
 				(path "/e63e39d7-6ac0-4ffd-8aa3-1841a4541b55/4c1824a3-ede3-44a9-9cc4-1658cb86e3ae/681cd5e3-d1a9-4f5a-899b-9dce52990abf"
-					(reference "R64")
+					(reference "R16")
 					(unit 1)
 				)
@@
 		(dnp no)
 		(fields_autoplaced yes)
-		(property "Reference" "#PWR01"
+		(property "Reference" "#PWR027"
 			(at 191.77 109.22 0)
 			(effects
@@
 			(project "psu"
 				(path "/e63e39d7-6ac0-4ffd-8aa3-1841a4541b55/4c1824a3-ede3-44a9-9cc4-1658cb86e3ae/681cd5e3-d1a9-4f5a-899b-9dce52990abf"
-					(reference "#PWR01")
+					(reference "#PWR027")
 					(unit 1)
 				)
@@
 		(dnp no)
 		(fields_autoplaced yes)
-		(property "Reference" "C76"
+		(property "Reference" "C14"
 			(at 195.58 91.4399 0)
 			(effects
@@
 			(project "psu"
 				(path "/e63e39d7-6ac0-4ffd-8aa3-1841a4541b55/4c1824a3-ede3-44a9-9cc4-1658cb86e3ae/681cd5e3-d1a9-4f5a-899b-9dce52990abf"
-					(reference "C76")
+					(reference "C14")
 					(unit 1)
 				)
@@
 		(dnp no)
 		(fields_autoplaced yes)
-		(property "Reference" "D10"
+		(property "Reference" "D5"
 			(at 121.92 96.5199 90)
 			(effects
@@
 			(project ""
 				(path "/e63e39d7-6ac0-4ffd-8aa3-1841a4541b55/4c1824a3-ede3-44a9-9cc4-1658cb86e3ae/681cd5e3-d1a9-4f5a-899b-9dce52990abf"
-					(reference "D10")
+					(reference "D5")
 					(unit 1)
 				)
@@
 		(dnp no)
 		(fields_autoplaced yes)
-		(property "Reference" "#PWR0115"
+		(property "Reference" "#PWR030"
 			(at 146.05 114.3 0)
 			(effects
@@
 			(project "psu"
 				(path "/e63e39d7-6ac0-4ffd-8aa3-1841a4541b55/4c1824a3-ede3-44a9-9cc4-1658cb86e3ae/681cd5e3-d1a9-4f5a-899b-9dce52990abf"
-					(reference "#PWR0115")
+					(reference "#PWR030")
 					(unit 1)
 				)
@@
 		(dnp no)
 		(fields_autoplaced yes)
-		(property "Reference" "C77"
+		(property "Reference" "C15"
 			(at 138.43 96.5199 0)
 			(effects
@@
 			(project ""
 				(path "/e63e39d7-6ac0-4ffd-8aa3-1841a4541b55/4c1824a3-ede3-44a9-9cc4-1658cb86e3ae/681cd5e3-d1a9-4f5a-899b-9dce52990abf"
-					(reference "C77")
+					(reference "C15")
 					(unit 1)
 				)
@@
 		(dnp no)
 		(fields_autoplaced yes)
-		(property "Reference" "#PWR0114"
+		(property "Reference" "#PWR029"
 			(at 106.68 118.11 0)
 			(effects
@@
 			(project ""
 				(path "/e63e39d7-6ac0-4ffd-8aa3-1841a4541b55/4c1824a3-ede3-44a9-9cc4-1658cb86e3ae/681cd5e3-d1a9-4f5a-899b-9dce52990abf"
-					(reference "#PWR0114")
+					(reference "#PWR029")
 					(unit 1)
 				)
@@
 		(dnp no)
 		(fields_autoplaced yes)
-		(property "Reference" "#PWR088"
+		(property "Reference" "#PWR028"
 			(at 127 110.49 0)
 			(effects
@@
 			(project "psu"
 				(path "/e63e39d7-6ac0-4ffd-8aa3-1841a4541b55/4c1824a3-ede3-44a9-9cc4-1658cb86e3ae/681cd5e3-d1a9-4f5a-899b-9dce52990abf"
-					(reference "#PWR088")
-					(unit 1)
-				)
+					(reference "#PWR028")
+					(unit 1)
+				)

Commit message: kicad psu pcb finish psu
Parts:
- added F1: 5A fuse, Resistor_SMD:R_1206_3216Metric_Pad1.30x1.75mm_HandSolder, symbol Device:Fuse_Small
- D5: footprint Diode_SMD:D_SOD-923 -> Diode_SMD:Nexperia_CFP3_SOD-123W
Connections:
- net BAT_OUT: now also F1.2; no longer C13.2, C14.1, Q3.1 (D), U4.4 (VOut)
- new net: C13.2, C14.1, F1.1, Q3.1 (D), U4.4 (VOut)
Changed lines of the file:
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@@
 	(wire
 		(pts
-			(xy 191.77 88.9) (xy 200.66 88.9)
+			(xy 191.77 88.9) (xy 208.28 88.9)
 		)
 		(stroke
@@
 		(pts
 			(xy 179.07 88.9) (xy 184.15 88.9)
+		)
+		(stroke
+			(width 0)
+			(type default)
+		)
+	)
+	(wire
+		(pts
+			(xy 213.36 88.9) (xy 234.95 88.9)
 		)
 		(stroke
@@
 	(hierarchical_label "BAT_OUT"
 		(shape input)
-		(at 200.66 88.9 0)
+		(at 234.95 88.9 0)
 		(effects
 			(font
@@
 			)
 			(justify right)
+		)
+	)
+	(symbol
+		(lib_id "Device:Fuse_Small")
+		(at 210.82 88.9 0)
+		(unit 1)
+		(exclude_from_sim no)
+		(in_bom yes)
+		(on_board yes)
+		(dnp no)
+		(fields_autoplaced yes)
+		(property "Reference" "F1"
+			(at 210.82 83.82 0)
+			(effects
+				(font
+					(size 1.27 1.27)
+				)
+			)
+		)
+		(property "Value" "5A fuse"
+			(at 210.82 86.36 0)
+			(effects
+				(font
+					(size 1.27 1.27)
+				)
+			)
+		)
+		(property "Footprint" "Resistor_SMD:R_1206_3216Metric_Pad1.30x1.75mm_HandSolder"
+			(at 210.82 88.9 0)
+			(effects
+				(font
+					(size 1.27 1.27)
+				)
+				(hide yes)
+			)
+		)
+		(property "Datasheet" "~"
+			(at 210.82 88.9 0)
+			(effects
+				(font
+					(size 1.27 1.27)
+				)
+				(hide yes)
+			)
+		)
+		(property "Description" "Fuse, small symbol"
+			(at 210.82 88.9 0)
+			(effects
+				(font
+					(size 1.27 1.27)
+				)
+				(hide yes)
+			)
+		)
+		(property "Url" "https://hu.farnell.com/vishay/wfma2512r0250fea/res-0r025-3w-2512-metal-plate/dp/3102734?srsltid=AfmBOoo6H5Un0cHiqeag9ovCQvXpnbJqYON7v56Iowkpb5I1FAlzBtap"
+			(at 210.82 88.9 0)
+			(effects
+				(font
+					(size 1.27 1.27)
+				)
+				(hide yes)
+			)
+		)
+		(property "Sim.Device" ""
+			(at 210.82 88.9 90)
+			(effects
+				(font
+					(size 1.27 1.27)
+				)
+				(hide yes)
+			)
+		)
+		(property "Sim.Type" ""
+			(at 210.82 88.9 90)
+			(effects
+				(font
+					(size 1.27 1.27)
+				)
+				(hide yes)
+			)
+		)
+		(pin "1"
+		)
+		(pin "2"
+		)
+		(instances
+			(project "psu"
+				(path "/e63e39d7-6ac0-4ffd-8aa3-1841a4541b55/4c1824a3-ede3-44a9-9cc4-1658cb86e3ae/681cd5e3-d1a9-4f5a-899b-9dce52990abf"
+					(reference "F1")
+					(unit 1)
+				)
+			)
 		)
 	)
@@
 			)
 		)
-		(property "Footprint" "Diode_SMD:D_SOD-923"
+		(property "Footprint" "Diode_SMD:Nexperia_CFP3_SOD-123W"
 			(at 119.38 97.79 0)
 			(effects

Commit message: PSU FINISH BOARD NO DRC,ERC,DFM ERRORS
Other:
- moved on the sheet: C13, C14, C15, D5, F1, J2, J3, Q2, Q3, R16, R17, R18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

Commit message: PSU bugfixes
Parts:
- D5: value SMCJ45A -> SMCJ20A
- U4: value ~ -> KTS1900QGXAA-TA
Connections:
- net BAT_OUT: now also C13.2, C14.1, Q3.1 (D), U4.4 (VOut); no longer F1.2
- net SW_N: now also F1.2; no longer J2.P (POS), J3.1 (Pin_1)
- new net: F1.1, J2.P (POS), J3.1 (Pin_1)
Other:
- moved on the sheet: F1, J2, J3
Changed lines of the file:
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@@
 	)
 	(junction
-		(at 52.07 55.88)
+		(at 35.56 72.39)
 		(diameter 0)
 		(color 0 0 0 0)
@@
 	)
 	(junction
-		(at 44.45 72.39)
+		(at 86.36 50.8)
 		(diameter 0)
 		(color 0 0 0 0)
 	)
 	(junction
-		(at 86.36 50.8)
+		(at 43.18 55.88)
 		(diameter 0)
 		(color 0 0 0 0)
@@
 	(wire
 		(pts
-			(xy 44.45 73.66) (xy 44.45 72.39)
-		)
-		(stroke
-			(width 0)
-			(type default)
-		)
-	)
-	(wire
-		(pts
-			(xy 129.54 50.8) (xy 146.05 50.8)
+			(xy 129.54 50.8) (xy 172.72 50.8)
 		)
 		(stroke
@@
 	(wire
 		(pts
+			(xy 27.94 72.39) (xy 35.56 72.39)
+		)
+		(stroke
+			(width 0)
+			(type default)
+		)
+	)
+	(wire
+		(pts
 			(xy 62.23 80.01) (xy 69.85 80.01)
 		)
@@
 	(wire
 		(pts
-			(xy 52.07 64.77) (xy 52.07 55.88)
-		)
-		(stroke
-			(width 0)
-			(type default)
-		)
-	)
-	(wire
-		(pts
 			(xy 77.47 50.8) (xy 77.47 55.88)
 		)
@@
 	(wire
 		(pts
-			(xy 52.07 55.88) (xy 36.83 55.88)
-		)
-		(stroke
-			(width 0)
-			(type default)
-		)
-	)
-	(wire
-		(pts
 			(xy 69.85 76.2) (xy 69.85 80.01)
 		)
@@
 	(wire
 		(pts
+			(xy 49.53 55.88) (xy 57.15 55.88)
+		)
+		(stroke
+			(width 0)
+			(type default)
+		)
+	)
+	(wire
+		(pts
+			(xy 43.18 55.88) (xy 27.94 55.88)
+		)
+		(stroke
+			(width 0)
+			(type default)
+		)
+	)
+	(wire
+		(pts
 			(xy 69.85 80.01) (xy 86.36 80.01)
 		)
@@
 	(wire
 		(pts
-			(xy 52.07 55.88) (xy 57.15 55.88)
+			(xy 43.18 67.31) (xy 43.18 72.39)
+		)
+		(stroke
+			(width 0)
+			(type default)
+		)
+	)
+	(wire
+		(pts
+			(xy 43.18 64.77) (xy 43.18 55.88)
 		)
 		(stroke
@@
 	(wire
 		(pts
-			(xy 151.13 50.8) (xy 172.72 50.8)
-		)
-		(stroke
-			(width 0)
-			(type default)
-		)
-	)
-	(wire
-		(pts
 			(xy 77.47 43.18) (xy 121.92 43.18)
 		)
@@
 	(wire
 		(pts
-			(xy 52.07 67.31) (xy 52.07 72.39)
-		)
-		(stroke
-			(width 0)
-			(type default)
-		)
-	)
-	(wire
-		(pts
 			(xy 72.39 55.88) (xy 77.47 55.88)
 		)
@@
 	(wire
 		(pts
+			(xy 27.94 58.42) (xy 27.94 72.39)
+		)
+		(stroke
+			(width 0)
+			(type default)
+		)
+	)
+	(wire
+		(pts
 			(xy 64.77 63.5) (xy 72.39 63.5)
 		)
@@
 	(wire
 		(pts
-			(xy 36.83 58.42) (xy 36.83 72.39)
-		)
-		(stroke
-			(width 0)
-			(type default)
-		)
-	)
-	(wire
-		(pts
-			(xy 44.45 72.39) (xy 52.07 72.39)
+			(xy 35.56 72.39) (xy 43.18 72.39)
 		)
 		(stroke
@@
 	(wire
 		(pts
+			(xy 35.56 73.66) (xy 35.56 72.39)
+		)
+		(stroke
+			(width 0)
+			(type default)
+		)
+	)
+	(wire
+		(pts
+			(xy 43.18 55.88) (xy 44.45 55.88)
+		)
+		(stroke
+			(width 0)
+			(type default)
+		)
+	)
+	(wire
+		(pts
 			(xy 77.47 50.8) (xy 86.36 50.8)
-		)
-		(stroke
-			(width 0)
-			(type default)
-		)
-	)
-	(wire
-		(pts
-			(xy 36.83 72.39) (xy 44.45 72.39)
 		)
 		(stroke
@@
 	(symbol
 		(lib_id "Device:Fuse_Small")
-		(at 148.59 50.8 0)
+		(at 46.99 55.88 0)
 		(unit 1)
 		(exclude_from_sim no)
@@
 		(fields_autoplaced yes)
 		(property "Reference" "F1"
-			(at 148.59 45.72 0)
+			(at 46.99 50.8 0)
 			(effects
 				(font
@@
 		)
 		(property "Value" "5A fuse"
-			(at 148.59 48.26 0)
+			(at 46.99 53.34 0)
 			(effects
 				(font
@@
 		)
 		(property "Footprint" "Resistor_SMD:R_1206_3216Metric_Pad1.30x1.75mm_HandSolder"
-			(at 148.59 50.8 0)
+			(at 46.99 55.88 0)
 			(effects
 				(font
@@
 		)
 		(property "Datasheet" "~"
-			(at 148.59 50.8 0)
+			(at 46.99 55.88 0)
 			(effects
 				(font
@@
 		)
 		(property "Description" "Fuse, small symbol"
-			(at 148.59 50.8 0)
+			(at 46.99 55.88 0)
 			(effects
 				(font
@@
 		)
 		(property "Url" "https://hu.farnell.com/vishay/wfma2512r0250fea/res-0r025-3w-2512-metal-plate/dp/3102734?srsltid=AfmBOoo6H5Un0cHiqeag9ovCQvXpnbJqYON7v56Iowkpb5I1FAlzBtap"
-			(at 148.59 50.8 0)
+			(at 46.99 55.88 0)
 			(effects
 				(font
@@
 		)
 		(property "Sim.Device" ""
-			(at 148.59 50.8 90)
+			(at 46.99 55.88 90)
 			(effects
 				(font
@@
 		)
 		(property "Sim.Type" ""
-			(at 148.59 50.8 90)
+			(at 46.99 55.88 90)
 			(effects
 				(font
@@
 	(symbol
 		(lib_id "CM5:XT60")
-		(at 22.86 57.15 0)
+		(at 13.97 57.15 0)
 		(mirror y)
 		(unit 1)
@@
 		(dnp no)
 		(property "Reference" "J2"
-			(at 27.94 64.77 0)
+			(at 19.05 64.77 0)
 			(effects
 				(font
@@
 		)
 		(property "Value" "~"
-			(at 27.94 62.23 0)
+			(at 19.05 62.23 0)
 			(effects
 				(font
@@
 		)
 		(property "Footprint" "psu:AMASS_XT60-M"
-			(at 22.86 57.15 0)
+			(at 13.97 57.15 0)
 			(effects
 				(font
@@
 		)
 		(property "Datasheet" ""
-			(at 22.86 57.15 0)
+			(at 13.97 57.15 0)
 			(effects
 				(font
@@
 		)
 		(property "Description" ""
-			(at 22.86 57.15 0)
+			(at 13.97 57.15 0)
 			(effects
 				(font
@@
 	(symbol
 		(lib_id "Connector:Conn_01x02_Pin")
-		(at 46.99 64.77 0)
+		(at 38.1 64.77 0)
 		(unit 1)
 		(exclude_from_sim no)
@@
 		(fields_autoplaced yes)
 		(property "Reference" "J3"
-			(at 47.625 59.69 0)
+			(at 38.735 59.69 0)
 			(effects
 				(font
@@
 		)
 		(property "Value" "Charge"
-			(at 47.625 62.23 0)
+			(at 38.735 62.23 0)
 			(effects
 				(font
@@
 		)
 		(property "Footprint" "Connector_JST:JST_PH_B2B-PH-K_1x02_P2.00mm_Vertical"
-			(at 46.99 64.77 0)
+			(at 38.1 64.77 0)
 			(effects
 				(font
@@
 		)
 		(property "Datasheet" "~"
-			(at 46.99 64.77 0)
+			(at 38.1 64.77 0)
 			(effects
 				(font
@@
 		)
 		(property "Description" "Generic connector, single row, 01x02, script generated"
-			(at 46.99 64.77 0)
+			(at 38.1 64.77 0)
 			(effects
 				(font
@@
 		)
 		(instances
-			(project ""
+			(project "psu"
 				(path "/e63e39d7-6ac0-4ffd-8aa3-1841a4541b55/4c1824a3-ede3-44a9-9cc4-1658cb86e3ae/681cd5e3-d1a9-4f5a-899b-9dce52990abf"
 					(reference "J3")
@@
 			)
 		)
-		(property "Value" "SMCJ45A"
+		(property "Value" "SMCJ20A"
 			(at 59.69 60.9599 90)
 			(effects
@@
 		(on_board yes)
 		(dnp no)
-		(fields_autoplaced yes)
 		(property "Reference" "U4"
 			(at 97.79 85.09 0)
@@
 			)
 		)
-		(property "Value" "~"
-			(at 97.79 86.36 0)
+		(property "Value" "KTS1900QGXAA-TA"
+			(at 97.79 87.884 0)
 			(effects
 				(font
@@
 			)
 		)
-		(property "Datasheet" ""
+		(property "Datasheet" "https://hu.mouser.com/datasheet/3/2612/1/KTS1900-04e.pdf"
 			(at 97.79 77.47 0)
 			(effects
@@
 	(symbol
 		(lib_id "power:GND")
-		(at 44.45 73.66 0)
+		(at 35.56 73.66 0)
 		(unit 1)
 		(exclude_from_sim no)
@@
 		(fields_autoplaced yes)
 		(property "Reference" "#PWR029"
-			(at 44.45 80.01 0)
+			(at 35.56 80.01 0)
 			(effects
 				(font
@@
 		)
 		(property "Value" "GND"
-			(at 44.45 78.74 0)
+			(at 35.56 78.74 0)
 			(effects
 				(font
@@
 		)
 		(property "Footprint" ""
-			(at 44.45 73.66 0)
+			(at 35.56 73.66 0)
 			(effects
 				(font
@@
 		)
 		(property "Datasheet" ""
-			(at 44.45 73.66 0)
+			(at 35.56 73.66 0)
 			(effects
 				(font
@@
 		)
 		(property "Description" "Power symbol creates a global label with name \"GND\" , ground"
-			(at 44.45 73.66 0)
+			(at 35.56 73.66 0)
 			(effects
 				(font
@@
 		)
 		(instances
-			(project ""
+			(project "psu"
 				(path "/e63e39d7-6ac0-4ffd-8aa3-1841a4541b55/4c1824a3-ede3-44a9-9cc4-1658cb86e3ae/681cd5e3-d1a9-4f5a-899b-9dce52990abf"
 					(reference "#PWR029")
