File: Circuit/kicad/V4/psu_motor-controll/Battery-circuit.kicad_sch (KiCad schematic)
At the start: 13 parts, among them J3 Charge, Q2 IRFR7546TRPBF, Q3 IRFR7546TRPBF, U4 KTS1900QGXAA-TA

Commit message: updated bom, updated compon
Parts:
- C13: Cikkszám (none) -> 100.011.24; Link (none) -> https://www.hestore.hu/prod_10001124.html
- C14, C15: value 4.7uf -> 4,7uf; Cikkszám (none) -> 100.427.11; Link (none) -> https://www.hestore.hu/prod_10042711.html
- D5: Cikkszám (none) -> 100.489.14; Link (none) -> https://www.hestore.hu/prod_10048914.html
- F1: Cikkszám (none) -> C1F-5; Link (none) -> https://www.tme.eu/hu/details/c1f-5/biztositekok-smd-1206-g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; Url https://hu.farnell.com/vishay/wfma2512r0250fea/res-0r025-3w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 -> (none)
- J2: value ~ -> xt-60; Cikkszám (none) -> 100.354.92; Link (none) -> https://www.hestore.hu/prod_10035492.html
- J3: Cikkszám (none) -> 100.385.23; Link (none) -> https://www.hestore.hu/prod_10038523.html
- Q2, Q3: Cikkszám (none) -> 100.484.30; Link (none) -> https://www.hestore.hu/prod_10048430.html
- R16: value 100r -> 100R; Cikkszám (none) -> 100.011.42; Link (none) -> https://www.hestore.hu/prod_10001142.html
- R17: value 10r -> 10R; Cikkszám (none) -> 100.011.44; Link (none) -> https://www.hestore.hu/prod_10001144.html
- R18: Cikkszám (none) -> 100.011.43; Link (none) -> https://www.hestore.hu/prod_10001143.html
- U4: Cikkszám (none) -> 389-KTS1900QGXAA-TA; Link (none) -> https://hu.mouser.com/ProductDetail/Kinetic-Technologies/KT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
Changed lines of the file:
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@@
 			)
 		)
-		(property "Url" "https://hu.farnell.com/vishay/wfma2512r0250fea/res-0r025-3w-2512-metal-plate/dp/3102734?srsltid=AfmBOoo6H5Un0cHiqeag9ovCQvXpnbJqYON7v56Iowkpb5I1FAlzBtap"
+		(property "Cikkszám" "C1F-5"
 			(at 46.99 55.88 0)
 			(effects
@@
 			)
 		)
-		(property "Sim.Device" ""
-			(at 46.99 55.88 90)
-			(effects
-				(font
-					(size 1.27 1.27)
-				)
-				(hide yes)
-			)
-		)
-		(property "Sim.Type" ""
-			(at 46.99 55.88 90)
+		(property "Link" "https://www.tme.eu/hu/details/c1f-5/biztositekok-smd-1206-gyors/bel-fuse/0685f5000-01/"
+			(at 46.99 55.88 0)
 			(effects
 				(font
@@
 			)
 		)
-		(property "Value" "~"
+		(property "Value" "xt-60"
 			(at 19.05 62.23 0)
 			(effects
@@
 		)
 		(property "Description" ""
+			(at 13.97 57.15 0)
+			(effects
+				(font
+					(size 1.27 1.27)
+				)
+				(hide yes)
+			)
+		)
+		(property "Cikkszám" "100.354.92"
+			(at 13.97 57.15 0)
+			(effects
+				(font
+					(size 1.27 1.27)
+				)
+				(hide yes)
+			)
+		)
+		(property "Link" "https://www.hestore.hu/prod_10035492.html"
 			(at 13.97 57.15 0)
 			(effects
@@
 			)
 		)
-		(property "Datasheet" "https://ngspice.sourceforge.io/docs/ngspice-html-manual/manual.xhtml#cha_MOSFETs"
+		(property "Datasheet" "https://www.hestore.hu/prod_getfile.php?id=19307"
 			(at 99.06 53.34 0)
 			(effects
@@
 			)
 		)
-		(property "Sim.Device" "NMOS"
-			(at 94.615 53.34 0)
-			(effects
-				(font
-					(size 1.27 1.27)
-				)
-				(hide yes)
-			)
-		)
-		(property "Sim.Type" "VDMOS"
-			(at 92.71 53.34 0)
-			(effects
-				(font
-					(size 1.27 1.27)
-				)
-				(hide yes)
-			)
-		)
-		(property "Sim.Pins" "1=D 2=G 3=S"
-			(at 96.52 53.34 0)
+		(property "Cikkszám" "100.484.30"
+			(at 111.76 53.34 90)
+			(effects
+				(font
+					(size 1.27 1.27)
+				)
+				(hide yes)
+			)
+		)
+		(property "Link" "https://www.hestore.hu/prod_10048430.html"
+			(at 111.76 53.34 90)
 			(effects
 				(font
@@
 			)
 		)
-		(property "Datasheet" "~"
+		(property "Datasheet" "https://www.hestore.hu/prod_getfile.php?id=9997"
 			(at 38.1 64.77 0)
 			(effects
@@
 		)
 		(property "Description" "Generic connector, single row, 01x02, script generated"
+			(at 38.1 64.77 0)
+			(effects
+				(font
+					(size 1.27 1.27)
+				)
+				(hide yes)
+			)
+		)
+		(property "Cikkszám" "100.385.23"
+			(at 38.1 64.77 0)
+			(effects
+				(font
+					(size 1.27 1.27)
+				)
+				(hide yes)
+			)
+		)
+		(property "Link" "https://www.hestore.hu/prod_10038523.html"
 			(at 38.1 64.77 0)
 			(effects
@@
 			)
 		)
-		(property "Datasheet" "~"
+		(property "Datasheet" "https://www.hestore.hu/prod_getfile.php?id=3654"
 			(at 73.66 76.2 0)
 			(effects
@@
 		(property "Description" "Resistor"
 			(at 73.66 76.2 0)
+			(effects
+				(font
+					(size 1.27 1.27)
+				)
+				(hide yes)
+			)
+		)
+		(property "Cikkszám" "100.011.43"
+			(at 73.66 76.2 90)
+			(effects
+				(font
+					(size 1.27 1.27)
+				)
+				(hide yes)
+			)
+		)
+		(property "Link" "https://www.hestore.hu/prod_10001143.html"
+			(at 73.66 76.2 90)
 			(effects
 				(font
@@
 			)
 		)
-		(property "Datasheet" "https://ngspice.sourceforge.io/docs/ngspice-html-manual/manual.xhtml#cha_MOSFETs"
+		(property "Datasheet" "https://www.hestore.hu/prod_getfile.php?id=19307"
 			(at 107.95 53.34 0)
 			(effects
@@
 			)
 		)
-		(property "Sim.Device" "NMOS"
-			(at 112.395 53.34 0)
-			(effects
-				(font
-					(size 1.27 1.27)
-				)
-				(hide yes)
-			)
-		)
-		(property "Sim.Type" "VDMOS"
-			(at 114.3 53.34 0)
-			(effects
-				(font
-					(size 1.27 1.27)
-				)
-				(hide yes)
-			)
-		)
-		(property "Sim.Pins" "1=D 2=G 3=S"
-			(at 110.49 53.34 0)
+		(property "Cikkszám" "100.484.30"
+			(at 95.25 53.34 90)
+			(effects
+				(font
+					(size 1.27 1.27)
+				)
+				(hide yes)
+			)
+		)
+		(property "Link" "https://www.hestore.hu/prod_10048430.html"
+			(at 95.25 53.34 90)
 			(effects
 				(font
@@
 			)
 		)
-		(property "Value" "10r"
+		(property "Value" "10R"
 			(at 90.17 63.5 0)
 			(effects
@@
 		)
 		(property "Description" "Resistor"
+			(at 95.25 62.23 0)
+			(effects
+				(font
+					(size 1.27 1.27)
+				)
+				(hide yes)
+			)
+		)
+		(property "Cikkszám" "100.011.44"
+			(at 95.25 62.23 0)
+			(effects
+				(font
+					(size 1.27 1.27)
+				)
+				(hide yes)
+			)
+		)
+		(property "Link" "https://www.hestore.hu/prod_10001144.html"
 			(at 95.25 62.23 0)
 			(effects
@@
 			)
 		)
-		(property "Datasheet" "~"
+		(property "Datasheet" "https://www.hestore.hu/prod_getfile.php?id=3645"
 			(at 121.92 46.99 0)
 			(effects
@@
 		)
 		(property "Description" "Unpolarized capacitor"
+			(at 121.92 46.99 0)
+			(effects
+				(font
+					(size 1.27 1.27)
+				)
+				(hide yes)
+			)
+		)
+		(property "Cikkszám" "100.011.24"
+			(at 121.92 46.99 0)
+			(effects
+				(font
+					(size 1.27 1.27)
+				)
+				(hide yes)
+			)
+		)
+		(property "Link" "https://www.hestore.hu/prod_10001124.html"
 			(at 121.92 46.99 0)
 			(effects
@@
 			)
 		)
-		(property "Value" "100r"
+		(property "Value" "100R"
 			(at 80.01 48.2599 0)
 			(effects
@@
 			)
 		)
-		(property "Datasheet" "~"
+		(property "Datasheet" "https://www.hestore.hu/prod_getfile.php?id=3653"
 			(at 77.47 46.99 0)
 			(effects
@@
 		)
 		(property "Description" "Resistor"
+			(at 77.47 46.99 0)
+			(effects
+				(font
+					(size 1.27 1.27)
+				)
+				(hide yes)
+			)
+		)
+		(property "Cikkszám" "100.011.42"
+			(at 77.47 46.99 0)
+			(effects
+				(font
+					(size 1.27 1.27)
+				)
+				(hide yes)
+			)
+		)
+		(property "Link" "https://www.hestore.hu/prod_10001142.html"
 			(at 77.47 46.99 0)
 			(effects
@@
 			)
 		)
-		(property "Value" "4.7uf"
+		(property "Value" "4,7uf"
 			(at 133.35 55.8799 0)
 			(effects
@@
 		)
 		(property "Description" "Unpolarized capacitor"
+			(at 129.54 54.61 0)
+			(effects
+				(font
+					(size 1.27 1.27)
+				)
+				(hide yes)
+			)
+		)
+		(property "Cikkszám" "100.427.11"
+			(at 129.54 54.61 0)
+			(effects
+				(font
+					(size 1.27 1.27)
+				)
+				(hide yes)
+			)
+		)
+		(property "Link" "https://www.hestore.hu/prod_10042711.html"
 			(at 129.54 54.61 0)
 			(effects
@@
 			)
 		)
-		(property "Datasheet" "https://www.onsemi.com/pub/Collateral/ESD9B-D.PDF"
+		(property "Datasheet" "https://www.hestore.hu/prod_getfile.php?id=19854"
 			(at 57.15 59.69 0)
 			(effects
@@
 		(property "Description" "ESD protection diode, 5.0Vrwm, SOD-923"
 			(at 57.15 59.69 0)
+			(effects
+				(font
+					(size 1.27 1.27)
+				)
+				(hide yes)
+			)
+		)
+		(property "Cikkszám" "100.489.14"
+			(at 57.15 59.69 90)
+			(effects
+				(font
+					(size 1.27 1.27)
+				)
+				(hide yes)
+			)
+		)
+		(property "Link" "https://www.hestore.hu/prod_10048914.html"
+			(at 57.15 59.69 90)
 			(effects
 				(font
@@
 			)
 		)
-		(property "Value" "4.7uf"
+		(property "Value" "4,7uf"
 			(at 76.2 60.9599 0)
 			(effects
@@
 			)
 		)
+		(property "Cikkszám" "100.427.11"
+			(at 72.39 59.69 0)
+			(effects
+				(font
+					(size 1.27 1.27)
+				)
+				(hide yes)
+			)
+		)
+		(property "Link" "https://www.hestore.hu/prod_10042711.html"
+			(at 72.39 59.69 0)
+			(effects
+				(font
+					(size 1.27 1.27)
+				)
+				(hide yes)
+			)
+		)
 		(pin "1"
 		)
@@
 			)
 		)
-		(property "Datasheet" "https://hu.mouser.com/datasheet/3/2612/1/KTS1900-04e.pdf"
+		(property "Datasheet" "https://www.hestore.hu/prod_getfile.php?id=9498"
 			(at 97.79 77.47 0)
 			(effects
@@
 			(at 97.79 77.47 0)
 			(effects
+				(font
+					(size 1.27 1.27)
+				)
+				(hide yes)
+			)
+		)
+		(property "Cikkszám" "389-KTS1900QGXAA-TA"
+			(at 97.79 77.47 0)
+			(effects
+				(font
+					(size 1.27 1.27)
+				)
+				(hide yes)
+			)
+		)
+		(property "Link" "https://hu.mouser.com/ProductDetail/Kinetic-Technologies/KTS1900QGXAA-TA?qs=jcD%2FCkGBYeO843PJRZf5hw%3D%3D"
+			(at 97.79 77.47 0)
+			(effects

Commit message: FINISH PSU V1.4.9 to production 1
Parts:
- D5: footprint Diode_SMD:Nexperia_CFP3_SOD-123W -> panel:P37_SOD-123FL
- F1: footprint Resistor_SMD:R_1206_3216Metric_Pad1.30x1.75mm_HandSolder -> Diode_SMD:D_2512_6332Metric
- J2: footprint psu:AMASS_XT60-M -> panel:AMASS_XT60-M
- Q2, Q3: footprint psu:nmos_dpak -> panel:nmos_dpak
Changed lines of the file:
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@@
 			)
 		)
-		(property "Footprint" "Resistor_SMD:R_1206_3216Metric_Pad1.30x1.75mm_HandSolder"
+		(property "Footprint" "Diode_SMD:D_2512_6332Metric"
 			(at 46.99 55.88 0)
 			(effects
@@
 			)
 		)
-		(property "Footprint" "psu:AMASS_XT60-M"
+		(property "Footprint" "panel:AMASS_XT60-M"
 			(at 13.97 57.15 0)
 			(effects
@@
 			)
 		)
-		(property "Footprint" "psu:nmos_dpak"
+		(property "Footprint" "panel:nmos_dpak"
 			(at 114.3 48.26 0)
 			(effects
@@
 			)
 		)
-		(property "Footprint" "psu:nmos_dpak"
+		(property "Footprint" "panel:nmos_dpak"
 			(at 92.71 48.26 0)
 			(effects
@@
 			)
 		)
-		(property "Footprint" "Diode_SMD:Nexperia_CFP3_SOD-123W"
+		(property "Footprint" "panel:P37_SOD-123FL"
 			(at 57.15 59.69 0)
 			(effects
