File: Circuit/kicad/V4/psu_motor-controll/PSUs.kicad_sch (KiCad schematic)
At the start: 98 parts, among them U23 LTC3119EFE_PBF, U26 LTC3119EFE_PBF

Commit message: kicad v4 psu pcb clean
Parts:
- renumbered C29 to C32, C30 to C33, C31 to C34, C32 to C35, C33 to C36, C34 to C37, C35 to C38, C36 to C39, C37 to C40, C38 to C41, C39 to C42, C40 to C43, C41 to C44, C42 to C45, C43 to C46, C44 to C47, C45 to C48, C46 to C49, C47 to C50, C48 to C51, C49 to C52, C50 to C53, C51 to C54, C52 to C55, C53 to C56, C54 to C57, C55 to C58, C56 to C59, C57 to C60, C58 to C61, C59 to C62, C60 to C63, C61 to C64, C62 to C65, C63 to C66, C64 to C67, C65 to C68, C66 to C69, C67 to C70, C68 to C71, C69 to C72, C70 to C73, C71 to C74, C72 to C75, C73 to C76, C74 to C77, D9 to D10, D5 to D6, D6 to D7, D7 to D8, D8 to D9, L6 to L1, L3 to L2, L1 to L3, L2 to L5, R32 to R35, R33 to R36, R34 to R37, R35 to R38, R36 to R39, R37 to R40, R38 to R41, R39 to R42, R40 to R43, R41 to R44, R42 to R45, R43 to R46, R45 to R47, R44 to R48, R46 to R49, R47 to R50, R48 to R51, R49 to R52, R50 to R53, R51 to R54, R52 to R55, R53 to R56, R54 to R57, R55 to R58, R56 to R59, R57 to R60, R58 to R61, R59 to R62, R60 to R63, R61 to R64, R62 to R65, R63 to R66, U22 to U21, U26 to U22, U24 to U23, U25 to U24, U23 to U25

Commit message: kicad psu pcb finish psu
Parts:
- added C81, C82, C83, C84: 4,7uf, Capacitor_SMD:C_0805_2012Metric, symbol Device:C
Connections:
- net +3.3V: now also C81.1, C82.1, C83.1, C84.1
- net GND: now also C81.2, C82.2, C83.2, C84.2

Commit message: kicad FINISH PSU PCB
Parts:
- U21, U23, U24: footprint Package_SO:SOIC-8-1EP_3.9x4.9mm_P1.27mm_EP2.95x4.9mm_Mask2.71x3.4mm_ThermalVias -> psu:SOIC-8-1EP_3.9x4.9mm_P1.27mm_EP2.95x4.9mm_Mask2.71x3.4mm_ThermalVias_BigVias
Changed lines of the file:
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@@
 			)
 		)
-		(property "Footprint" "Package_SO:SOIC-8-1EP_3.9x4.9mm_P1.27mm_EP2.95x4.9mm_Mask2.71x3.4mm_ThermalVias"
+		(property "Footprint" "psu:SOIC-8-1EP_3.9x4.9mm_P1.27mm_EP2.95x4.9mm_Mask2.71x3.4mm_ThermalVias_BigVias"
 			(at 62.23 39.37 0)
 			(effects
@@
 			)
 		)
-		(property "Footprint" "Package_SO:SOIC-8-1EP_3.9x4.9mm_P1.27mm_EP2.95x4.9mm_Mask2.71x3.4mm_ThermalVias"
+		(property "Footprint" "psu:SOIC-8-1EP_3.9x4.9mm_P1.27mm_EP2.95x4.9mm_Mask2.71x3.4mm_ThermalVias_BigVias"
 			(at 60.96 95.25 0)
 			(effects
@@
 			)
 		)
-		(property "Footprint" "Package_SO:SOIC-8-1EP_3.9x4.9mm_P1.27mm_EP2.95x4.9mm_Mask2.71x3.4mm_ThermalVias"
+		(property "Footprint" "psu:SOIC-8-1EP_3.9x4.9mm_P1.27mm_EP2.95x4.9mm_Mask2.71x3.4mm_ThermalVias_BigVias"
 			(at 62.23 146.05 0)
 			(effects

Commit message: PSU bugfixes
Parts:
- added TP6, TP7: TestPoint, TestPoint:TestPoint_Pad_D2.0mm, symbol Connector:TestPoint
Connections:
- net GND: now also TP6.1, TP7.1

Commit message: updated bom, updated compon
Parts:
- C32, C33, C34, C40, C49, C58, C61, C62, C63, C73: Cikkszám (none) -> 100.011.22; Field4 Farnell -> (none); Field5 2611911 -> (none); Field6 RM EMK105 B7104KV-F -> (none); Field7 TAIYO YUDEN EUROPE GMBH -> (none); Field8 110091611 -> (none); Link (none) -> https://www.hestore.hu/prod_10001122.html; Part Description 0.1uF 10% 16V Ceramic Capacitor X7R 0402 (1005 Metric) -> (none)
- C35, C36, C38, C39, C43, C44, C45, C46, C48, C50, C51, C52, C54, C55, C56, C57, C64, C65, C67, C68, C69, C70, C71, C72, C77, C81, C82, C83, C84: Cikkszám (none) -> 100.427.11; Link (none) -> https://www.hestore.hu/prod_10042711.html
- C37, C53, C66: Cikkszám (none) -> 100.380.72; Field4 Digikey -> (none); Field5 490-17672-2-ND -> (none); Field6 GJM1555C1H270JB01D -> (none); Field7 Murata -> (none); Link (none) -> https://www.hestore.hu/prod_10038072.html; Part Description 27pF 5% 50V Ceramic Capacitor C0G, NP0 0402 (1005 Metric) -> (none)
- C41, C59, C74: Cikkszám (none) -> 100.380.72; Link (none) -> https://www.hestore.hu/prod_10038072.html
- C42, C60, C75: Cikkszám (none) -> 100.491.13; Field4 Digikey -> (none); Field5 490-16429-1-ND -> (none); Field6 GCM155R71H122KA37D -> (none); Field7 Murata -> (none); Link (none) -> https://www.hestore.hu/prod_10049113.html; Part Description 1200pF 10% 10V Ceramic Capacitor X5R 0402 (1005 Metric) -> (none)
- C47, C76: Cikkszám (none) -> 100.200.77; Field4 Digikey -> (none); Field5 490-17672-2-ND -> (none); Field6 GJM1555C1H270JB01D -> (none); Field7 Murata -> (none); Link (none) -> https://www.hestore.hu/prod_10020077.html; Part Description 27pF 5% 50V Ceramic Capacitor C0G, NP0 0402 (1005 Metric) -> (none)
- D10, D6, D7, D8, D9: Cikkszám (none) -> 100.365.90; Link (none) -> https://www.hestore.hu/prod_10036590.html
- L1, L2, L3, L4, L5: Cikkszám (none) -> 100.490.90; Link (none) -> https://www.hestore.hu/prod_10049090.html
- R35, R48, R54: Cikkszám (none) -> 100.011.44; Field4 Farnell -> (none); Field5 9238999 -> (none); Field6 RC0402FR-0710RL -> (none); Field7 Yageo -> (none); Field8 URES00256 -> (none); Link (none) -> https://www.hestore.hu/prod_10001144.html; Part Description Resistor 10R M1005 1% 63mW -> (none)
- R36: value 100 -> 100R; Cikkszám (none) -> 100.011.42; Link (none) -> https://www.hestore.hu/prod_10001142.html
- R37: Cikkszám (none) -> 100.491.09; Field4 Farnell -> (none); Field5 9239430 -> (none); Field6 RK73G1ETQTP4702D -> (none); Field7 KOA EUROPE GMBH -> (none); Field8 120892781 -> (none); Link (none) -> https://www.hestore.hu/prod_10049109.html; Part Description Resistor 47K M1005 1% 63mW -> (none)
- R38, R51, R58: Cikkszám (none) -> 100.011.48; Field4 Farnell -> (none); Field5 9239367 -> (none); Field6 MCR01MZPF1202 -> (none); Field7 Rohm -> (none); Link (none) -> https://www.hestore.hu/prod_10001148.html; Part Description Resistor 12K M1005 1% 63mW -> (none)
- R39, R52, R62: Cikkszám (none) -> 100.011.72; Field4 Farnell -> (none); Field5 9239375 -> (none); Field6 MCR01MZPF1502 -> (none); Field7 Rohm -> (none); Field8 120891581 -> (none); Link (none) -> https://www.hestore.hu/prod_10001172.html; Part Description Resistor 15K M1005 1% 63mW -> (none)
- R40, R57: Cikkszám (none) -> 100.011.45; Link (none) -> https://www.hestore.hu/prod_10001145.html
- R41, R43, R53, R60, R64: Cikkszám (none) -> 100.011.81; Field4 Farnell -> (none); Field5 9239375 -> (none); Field6 MCR01MZPF1502 -> (none); Field7 Rohm -> (none); Field8 120891581 -> (none); Link (none) -> https://www.hestore.hu/prod_10001181.html; Part Description Resistor 15K M1005 1% 63mW -> (none)
- R42, R59: Cikkszám (none) -> 100.201.73; Field4 Farnell -> (none); Field5 9239375 -> (none); Field6 MCR01MZPF1502 -> (none); Field7 Rohm -> (none); Field8 120891581 -> (none); Link (none) -> https://www.hestore.hu/prod_10020173.html; Part Description Resistor 15K M1005 1% 63mW -> (none)
- R44, R61: Cikkszám (none) -> 100.406.77; Link (none) -> https://www.hestore.hu/prod_10040677.html
- R45, R63: Cikkszám (none) -> 100.491.04; Field4 Farnell -> (none); Field5 9239375 -> (none); Field6 MCR01MZPF1502 -> (none); Field7 Rohm -> (none); Field8 120891581 -> (none); Link (none) -> https://www.hestore.hu/prod_10049104.html; Part Description Resistor 15K M1005 1% 63mW -> (none)
- R46, R65: Cikkszám (none) -> 100.491.11; Field4 Farnell -> (none); Field5 9239375 -> (none); Field6 MCR01MZPF1502 -> (none); Field7 Rohm -> (none); Field8 120891581 -> (none); Link (none) -> https://www.hestore.hu/prod_10049111.html; Part Description Resistor 15K M1005 1% 63mW -> (none)
- R47, R66: Cikkszám (none) -> 100.491.12; Link (none) -> https://www.hestore.hu/prod_10049112.html
- R49: Cikkszám (none) -> 100.011.57; Link (none) -> https://www.hestore.hu/prod_10001157.html
- R50: Cikkszám (none) -> 100.491.10; Field4 Farnell -> (none); Field5 9239430 -> (none); Field6 RK73G1ETQTP4702D -> (none); Field7 KOA EUROPE GMBH -> (none); Field8 120892781 -> (none); Link (none) -> https://www.hestore.hu/prod_10049110.html; Part Description Resistor 47K M1005 1% 63mW -> (none)
- R55: Cikkszám (none) -> 100.011.70; Link (none) -> https://www.hestore.hu/prod_10001170.html
- R56: Cikkszám (none) -> RC1206FR-07178KL; Field4 Farnell -> (none); Field5 9239430 -> (none); Field6 RK73G1ETQTP4702D -> (none); Field7 KOA EUROPE GMBH -> (none); Field8 120892781 -> (none); Link (none) -> https://www.tme.eu/hu/details/rc1206fr-07178kl/smd-ellenall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; Part Description Resistor 47K M1005 1% 63mW -> (none)
- TP1, TP2, TP3, TP4, TP5, TP6, TP7: now left out of the parts list
- U21, U23, U24: value ~ -> AP64501SP-13; Cikkszám (none) -> 100.491.27; Link (none) -> https://www.hestore.hu/prod_10049127.html
- U22, U25: Availability In Stock -> (none); Check_prices https://www.snapeda.com/parts/LTC3119EFE%23PBF/Analog+Devic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 -> (none); Cikkszám (none) -> LTC3119HFE#PBF; Description_1 Buck-Boost Switching Regulator IC Positive Adjustable 0.8V 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 -> (none); Link (none) -> https://eu.mouser.com/ProductDetail/Analog-Devices/LTC3119H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; MANUFACTURER Analog Devices -> (none); MAXIMUM_PACKAGE_HEIGHT 1.2mm -> (none); MF Analog Devices -> (none); MP LTC3119EFE#PBF -> (none); PARTREV B -> (none); Package TSSOP-28 Linear Technology -> (none); Price None -> (none); STANDARD IPC-7351B -> (none); SnapEDA_Link https://www.snapeda.com/parts/LTC3119EFE%23PBF/Analog+Devic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 -> (none)

Commit message: FINISH PSU V1.4.9 to production 1
Parts:
- L1, L2, L3, L4, L5: footprint Inductor_SMD:L_KOHERelec_MDA7030 -> panel:HCM1A0805
- U21, U23, U24: footprint psu:SOIC-8-1EP_3.9x4.9mm_P1.27mm_EP2.95x4.9mm_Mask2.71x3.4mm_ThermalVias_BigVias -> panel:SOIC-8-1EP_3.9x4.9mm_P1.27mm_EP2.95x4.9mm_Mask2.71x3.4mm_ThermalVias_BigVias
- U22, U25: footprint psu:SOP65P640X120-29N -> panel:SOP65P640X120-29N
Other:
- note added: "lehet sok a 10 ohm a bst re az apknél ha nem megy 2-5 ohmmal próbálni"
Changed lines of the file:
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@@
 		)
 	)
+	(text "lehet sok a 10 ohm a bst re az apknél ha nem megy 2-5 ohmmal próbálni "
+		(exclude_from_sim no)
+		(at 96.266 210.82 0)
+		(effects
+			(font
+				(size 2.54 2.54)
+			)
+		)
+	)
 	(junction
 		(at 152.4 25.4)
@@
 			)
 		)
-		(property "Footprint" "Inductor_SMD:L_KOHERelec_MDA7030"
+		(property "Footprint" "panel:HCM1A0805"
 			(at 88.9 132.08 0)
 			(effects
@@
 			)
 		)
-		(property "Footprint" "psu:SOP65P640X120-29N"
+		(property "Footprint" "panel:SOP65P640X120-29N"
 			(at 307.34 118.618 0)
 			(effects
@@
 			)
 		)
-		(property "Footprint" "Inductor_SMD:L_KOHERelec_MDA7030"
+		(property "Footprint" "panel:HCM1A0805"
 			(at 88.9 81.28 0)
 			(effects
@@
 			)
 		)
-		(property "Footprint" "psu:SOP65P640X120-29N"
+		(property "Footprint" "panel:SOP65P640X120-29N"
 			(at 307.34 25.908 0)
 			(effects
@@
 			)
 		)
-		(property "Footprint" "psu:SOIC-8-1EP_3.9x4.9mm_P1.27mm_EP2.95x4.9mm_Mask2.71x3.4mm_ThermalVias_BigVias"
+		(property "Footprint" "panel:SOIC-8-1EP_3.9x4.9mm_P1.27mm_EP2.95x4.9mm_Mask2.71x3.4mm_ThermalVias_BigVias"
 			(at 62.23 39.37 0)
 			(effects
@@
 			)
 		)
-		(property "Footprint" "Inductor_SMD:L_KOHERelec_MDA7030"
+		(property "Footprint" "panel:HCM1A0805"
 			(at 260.35 27.94 0)
 			(effects
@@
 			)
 		)
-		(property "Footprint" "Inductor_SMD:L_KOHERelec_MDA7030"
+		(property "Footprint" "panel:HCM1A0805"
 			(at 90.17 25.4 0)
 			(effects
@@
 			)
 		)
-		(property "Footprint" "psu:SOIC-8-1EP_3.9x4.9mm_P1.27mm_EP2.95x4.9mm_Mask2.71x3.4mm_ThermalVias_BigVias"
+		(property "Footprint" "panel:SOIC-8-1EP_3.9x4.9mm_P1.27mm_EP2.95x4.9mm_Mask2.71x3.4mm_ThermalVias_BigVias"
 			(at 60.96 95.25 0)
 			(effects
@@
 			)
 		)
-		(property "Footprint" "psu:SOIC-8-1EP_3.9x4.9mm_P1.27mm_EP2.95x4.9mm_Mask2.71x3.4mm_ThermalVias_BigVias"
+		(property "Footprint" "panel:SOIC-8-1EP_3.9x4.9mm_P1.27mm_EP2.95x4.9mm_Mask2.71x3.4mm_ThermalVias_BigVias"
 			(at 62.23 146.05 0)
 			(effects
@@
 			)
 		)
-		(property "Footprint" "Inductor_SMD:L_KOHERelec_MDA7030"
+		(property "Footprint" "panel:HCM1A0805"
 			(at 260.35 120.65 0)
 			(effects

Commit message: kicad: high speed V2.2 Circuit finish psu bom update
Parts:
- R56: Cikkszám RC1206FR-07178KL -> 100.491.25; Link https://www.tme.eu/hu/details/rc1206fr-07178kl/smd-ellenall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 -> https://www.hestore.hu/prod_10049125.html
Changed lines of the file:
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@@
 			)
 		)
-		(property "Cikkszám" "RC1206FR-07178KL"
+		(property "Cikkszám" "100.491.25"
 			(at 99.06 143.51 0)
 			(effects
@@
 			)
 		)
-		(property "Link" "https://www.tme.eu/hu/details/rc1206fr-07178kl/smd-ellenallasok/yageo/"
+		(property "Link" "https://www.hestore.hu/prod_10049125.html"
 			(at 99.06 143.51 0)
 			(effects
