File: Circuit/kicad/V4/high-speed/Shift_registers.kicad_sch (KiCad schematic)
At the start: 6 parts, among them U53 MCP23S17_SO, U54 MCP23S17_SO

Commit message: high speed first step
Parts:
- removed C103, C104, C105: 1uf, Capacitor_SMD:C_0805_2012Metric, symbol Device:C
- removed CT6: 10uf, Capacitor_Tantalum_SMD:CP_EIA-3528-21_Kemet-B, symbol Device:C_Polarized_Small
- removed U53, U54: MCP23S17_SO, Package_SO:SSOP-28_3.9x9.9mm_P0.635mm, symbol Interface_Expansion:MCP23S17_SO
Connections:
- no-connect marks 4 -> 0
