File: Circuit/kicad/V4/high-speed/high-speed.kicad_pcb (KiCad board)
At the start: 6 copper layers, 140 x 70 mm, 304 parts, among them J1 Conn_01x60_MountingPin, J10 USB_C_Receptacle_USB2.0_16P, J11 USB_C_Receptacle_USB2.0_16P, J12 690-008-221-904, J16 Conn_01x02_Pin, J17 Conn_01x02_Pin, J18 Conn_01x02_Pin, J19 Conn_01x02_Pin, J2 690-019-298-412, J20 Conn_01x02_Pin, J21 Conn_01x02_Pin, J3 USB3_A, J4 THD-02-R, J5 690-019-298-412, J6 THD-02-R, J7 MagJack-A70-112-331N126, J8 Conn_01x04_Socket, J9 Bus_M.2_Socket_M, Q1 bc akármi, Q2 bc akármi, SW1 Right angle Tact button, SW2 SW_Push, SW3 SW_Push, SW4 SW_Push, U1 RT9742SNGV, U10 FSUSB42MUX, U11 USB2514B-I/M2, U12 TPD4EUSB30, U13 AP22653W6, U14 TS5A23157DGSR, U15 LSF0108PWR, U16 TCA9548APWR, U17 CH343P, U18 ESP32-S3-WROOM-1, U19 MCP23S17_SO, U2 AP22653W6, U20 CD74HC154M, U21 BME280, U22 BNO080, U23 ICM-45686, U24 MCP3208, U25 PCM2704CDBR, U26 TPA6203A1DGN, U27 LSF0108PWR, U28 TCA9548APWR, U3 TPD4EUSB30, U4 TPD4EUSB30, U5 74LVC1G07SE-7, U6 ASEK-32.768KHZ-L-R-T, U7 AP22815AWU, U8 FSUSB42MUX, U9 TPD4EUSB30, Y1 24MHz, Y2 32.768MHz, Y3 5MHz

Commit message: high speed update
Parts:
- removed the U15 at (97.2, 108.6)
- added U27: LSF0108PWR, psu:SOP65P640X120-20N, B.Cu at (113.2, 100.2)
- JP1: renamed from JP2; moved to B.Cu
- JP2: renamed from JP1; moved to B.Cu
- moved C44 281.1 mm to (-3.79, -201.6)
- moved C51 281.1 mm to (2.66, -197.5)
- moved C52 281.1 mm to (-14.2, -209.8)
- moved C53 281.1 mm to (-14.2, -206.8)
- moved J16 281.1 mm to (-25.7, -220.7)
- moved J17 281.1 mm to (-25.7, -216.1)
- moved J18 281.1 mm to (-25.7, -211.5)
- moved J19 281.1 mm to (-25.7, -206.9)
- moved J20 281.1 mm to (-25.7, -202.3)
- moved J21 281.1 mm to (-25.7, -197.7)
- moved R70 281.1 mm to (-18.7, -221.5)
- moved R71 281.1 mm to (-18.7, -218.5)
- moved R72 281.1 mm to (-18.7, -215.6)
- moved R73 281.1 mm to (-18.7, -212.6)
- moved R74 281.1 mm to (-18.7, -209.7)
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- renumbered U27 to U15
Connections:
- JP1 pad 2: /I2C_devices/I2C_LSF_Vsel_2 -> /I2C_devices/I2C_LSF_Vsel_1
- JP2 pad 2: /I2C_devices/I2C_LSF_Vsel_1 -> /I2C_devices/I2C_LSF_Vsel_2
- U15 pad 10: /I2C_devices/AF_SDA5 -> /I2C_devices/AF_SDA1
- U15 pad 11: /I2C_devices/SDA5 -> /I2C_devices/SDA1
- U15 pad 12: /I2C_devices/SCL5 -> /I2C_devices/SCL1
- U15 pad 13: /I2C_devices/SDA6 -> /I2C_devices/SDA2
- U15 pad 14: /I2C_devices/SCL6 -> /I2C_devices/SCL2
- U15 pad 15: /I2C_devices/SDA7 -> /I2C_devices/SDA3
- U15 pad 16: /I2C_devices/SCL7 -> /I2C_devices/SCL3
- U15 pad 17: /I2C_devices/SDA8 -> /I2C_devices/SDA4
- U15 pad 18: /I2C_devices/SCL8 -> /I2C_devices/SCL4
- U15 pad 3: /I2C_devices/AF_SCL8 -> /I2C_devices/AF_SCL4
- U15 pad 4: /I2C_devices/AF_SDA8 -> /I2C_devices/AF_SDA4
- U15 pad 5: /I2C_devices/AF_SCL7 -> /I2C_devices/AF_SCL3
- U15 pad 6: /I2C_devices/AF_SDA7 -> /I2C_devices/AF_SDA3
- U15 pad 7: /I2C_devices/AF_SCL6 -> /I2C_devices/AF_SCL2
- U15 pad 8: /I2C_devices/AF_SDA6 -> /I2C_devices/AF_SDA2
- U15 pad 9: /I2C_devices/AF_SCL5 -> /I2C_devices/AF_SCL1
Routing:
- net /CM5_HighSpeed/DPHY0_D2_N: track 0.00 -> 51.7 mm
- net /CM5_HighSpeed/DPHY0_D2_P: track 0.00 -> 51.7 mm
- net /CM5_HighSpeed/DPHY0_D3_N: track 0.00 -> 51.7 mm
- net /CM5_HighSpeed/DPHY0_D3_P: track 0.00 -> 51.6 mm
- net /CM5_HighSpeed/DPHY0_D1_N: track 0.00 -> 51.5 mm
- net /CM5_HighSpeed/DPHY0_D1_P: track 0.00 -> 51.4 mm
- net /CM5_HighSpeed/DPHY0_C_N: track 0.00 -> 51.0 mm
- net /CM5_HighSpeed/DPHY0_C_P: track 0.00 -> 51.0 mm
- net /CM5_HighSpeed/DPHY0_D0_N: track 0.00 -> 51.0 mm
- net /CM5_HighSpeed/DPHY0_D0_P: track 0.00 -> 50.9 mm
- net /I2C_devices/AF_SDA1: track 0.00 -> 36.7 mm
- net /I2C_devices/AF_SCL1: track 0.00 -> 32.8 mm
- net ESP_3v3: track 22.6 -> 55.4 mm
- net /I2C_devices/AF_SDA2: track 0.00 -> 28.9 mm
- net /CM5_HighSpeed/DPHY1_D0_N: track 0.00 -> 28.8 mm
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- added copper zone on B.Cu, net /I2C_devices/I2C_LSF_Vsel_1
- added copper zone on B.Cu, net /I2C_devices/I2C_LSF_Vsel_2

Commit message: added psu start delay rc tag, high speed first inner and outboard impedance calculations
Parts:
- removed I2C_1, I2C_2: Conn_01x04_Pin, Connector_JST:JST_PH_B4B-PH-K_1x04_P2.00mm_Vertical
- removed U15, U27: LSF0108PWR, psu:SOP65P640X120-20N
- added C29: 10uf, Capacitor_SMD:C_0805_2012Metric, F.Cu at (34.0, 1.40)
- added I2C_0: Conn_01x04_Pin, Connector_JST:JST_SH_BM04B-SRSS-TB_1x04-1MP_P1.00mm_Vertical, F.Cu at (62.8, 96.9)
- JP1, JP2, R100, R102, R103, R104, R105, R31, R32, R33, R34, R35, R36, R37, R38, R39, R40, R41, R42, R43, R44, R45, R46, R47, R48, R49, R50, R51, R52, R53, R54, R55, R56, R57, R58, R59, R60, R61, R62, R63, R90, R91, R92, R93, R94, R95, R96, R97, R98, R99, U16, U28: moved to F.Cu
- TP10, TP11, TP12, TP13, TP14, TP15, TP16, TP17, TP18, TP19, TP2, TP20, TP21, TP23, TP24, TP25, TP26, TP27, TP28, TP29, TP3, TP30, TP4, TP5, TP6, TP7, TP8, TP9: moved to B.Cu
- moved C54 237.1 mm to (-162.0, 211.8)
- moved C55 237.1 mm to (-162.0, 214.8)
- moved C56 237.1 mm to (-162.0, 217.8)
- moved C57 237.1 mm to (-162.0, 220.8)
- moved C58 237.1 mm to (-162.0, 223.8)
- moved C59 237.1 mm to (-162.0, 226.8)
- moved C60 237.1 mm to (-147.9, 224.1)
- moved C61 237.1 mm to (-157.6, 211.8)
- moved C62 237.1 mm to (-157.6, 214.8)
- moved C63 237.1 mm to (-157.6, 217.8)
- moved C65 237.1 mm to (-157.6, 220.8)
- moved C66 237.1 mm to (-157.6, 223.8)
- moved C67 237.1 mm to (-157.6, 226.8)
- moved C68 237.1 mm to (-153.1, 211.8)
- moved C69 237.1 mm to (-145.9, 219.0)
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Connections:
- net /USB2-HUB/USB_AUDIO/BYPASS renamed /USB2-HUB/USB-AUDIO/BYPASS
- net /USB2-HUB/USB_AUDIO/Vdd renamed /USB2-HUB/USB-AUDIO/Vdd
- DSI1 pad 20: /CM5_HighSpeed/SCL0 -> /CM5_HighSpeed/CAM_SCL0
- DSI1 pad 21: /CM5_HighSpeed/SDA0 -> /CM5_HighSpeed/CAM_SDA0
- DSI2 pad 20: /CM5_HighSpeed/SCL1 -> /CM5_HighSpeed/CAM_SCL1
- DSI2 pad 21: /CM5_HighSpeed/SDA1 -> /CM5_HighSpeed/CAM_SDA1
- Module1 pad 57: /CM5_GPIO ( Ethernet, GPIO, SDCARD)/SD_CLK -> unconnected-(Module1A-SD_CLK-Pad57)
- Module1 pad 61: /CM5_GPIO ( Ethernet, GPIO, SDCARD)/SD_DAT3 -> unconnected-(Module1A-SD_DAT3-Pad61)
- Module1 pad 62: /CM5_GPIO ( Ethernet, GPIO, SDCARD)/SD_CMD -> unconnected-(Module1A-SD_CMD-Pad62)
- Module1 pad 63: /CM5_GPIO ( Ethernet, GPIO, SDCARD)/SD_DAT0 -> unconnected-(Module1A-SD_DAT0-Pad63)
- Module1 pad 67: /CM5_GPIO ( Ethernet, GPIO, SDCARD)/SD_DAT1 -> unconnected-(Module1A-SD_DAT1-Pad67)
- Module1 pad 69: /CM5_GPIO ( Ethernet, GPIO, SDCARD)/SD_DAT2 -> unconnected-(Module1A-SD_DAT2-Pad69)
- Module1 pad 75: /CM5_GPIO ( Ethernet, GPIO, SDCARD)/SD_PWR_ON -> unconnected-(Module1A-SD_PWR_ON-Pad75)
- Module1 pad 80: /CM5_HighSpeed/SCL0 -> /CM5_GPIO ( Ethernet, GPIO, SDCARD)/SCL0
- Module1 pad 82: /CM5_HighSpeed/SDA0 -> /CM5_GPIO ( Ethernet, GPIO, SDCARD)/SDA0
Routing:
- net /CM5_GPIO ( Ethernet, GPIO, SDCARD)/TRD3_N: track 0.00 -> 97.2 mm, vias 0 -> 2
- net /CM5_GPIO ( Ethernet, GPIO, SDCARD)/TRD3_P: track 0.00 -> 96.8 mm, vias 0 -> 2
- net /CM5_GPIO ( Ethernet, GPIO, SDCARD)/TRD2_N: track 0.00 -> 80.5 mm, vias 0 -> 2
- net /CM5_GPIO ( Ethernet, GPIO, SDCARD)/TRD0_N: track 0.00 -> 80.2 mm, vias 0 -> 2
- net /CM5_GPIO ( Ethernet, GPIO, SDCARD)/TRD1_N: track 0.00 -> 80.2 mm, vias 0 -> 2
- net /CM5_GPIO ( Ethernet, GPIO, SDCARD)/TRD0_P: track 0.00 -> 80.2 mm, vias 0 -> 2
- net /CM5_GPIO ( Ethernet, GPIO, SDCARD)/TRD1_P: track 0.00 -> 80.1 mm, vias 0 -> 2
- net /CM5_GPIO ( Ethernet, GPIO, SDCARD)/TRD2_P: track 0.00 -> 79.9 mm, vias 0 -> 2
- net /I2C_devices/SDA2_1: track 56.5 -> 0.00 mm, vias 1 -> 0
- net /I2C_devices/SCL2_1: track 54.5 -> 0.00 mm, vias 1 -> 0
- net ESP_3v3: track 55.4 -> 2.95 mm, vias 8 -> 0
- net /CM5_HighSpeed/PCIE_RX_N: track 4.02 -> 53.5 mm
- net /CM5_HighSpeed/PCIE_RX_P: track 4.02 -> 52.0 mm
- net /CM5_HighSpeed/PCIE_TX_P: track 3.30 -> 50.9 mm
- net /I2C_devices/SDA2_2: track 46.5 -> 0.00 mm, vias 1 -> 0
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- removed copper zone on B.Cu, net /I2C_devices/I2C_LSF_Vsel_2
- removed copper zone on B.Cu, net ESP_3v3

Commit message: kicad: high speed V2.2 Circuit finish psu bom update
Parts:
- removed C38: 100uf, Capacitor_Tantalum_SMD:CP_EIA-7343-31_Kemet-D
- removed C39: 100nf, Capacitor_SMD:C_0805_2012Metric
- removed J16, J17, J18, J19, J20, J21: Conn_01x02_Pin, Connector_PinHeader_2.54mm:PinHeader_2x01_P2.54mm_Vertical
- removed Q1, Q2: bc akármi, Package_TO_SOT_SMD:SOT-23
- removed R10, R11: 4.7k, Resistor_SMD:R_0805_2012Metric
- removed TP10, TP11, TP12, TP13, TP14, TP15, TP16, TP17, TP18, TP19, TP20, TP21, TP23, TP24, TP25, TP26, TP27, TP28, TP29, TP30, TP7, TP8: TestPoint_Small, TestPoint:TestPoint_Pad_D1.5mm
- removed TP22, TP31: TestPoint, TestPoint:TestPoint_Pad_D2.0mm
- removed Y2: 32.768MHz, Crystal:Crystal_SMD_HC49-SD
- added C30: 100nf, Capacitor_SMD:C_0805_2012Metric, F.Cu at (79.2, 55.7)
- added C31: 100nf, Capacitor_SMD:C_0805_2012Metric, F.Cu at (79.2, 58.7)
- added C32: 330pf, Capacitor_SMD:C_0805_2012Metric, F.Cu at (114.7, 67.7)
- added C33: 330pf, Capacitor_SMD:C_0805_2012Metric, F.Cu at (114.7, 70.8)
- added C34: 100nf, Capacitor_SMD:C_0805_2012Metric, F.Cu at (46.0, 53.1)
- added C35: 22nf c0g, Capacitor_SMD:C_0805_2012Metric, F.Cu at (46.0, 56.1)
- added C36: 1uf, Capacitor_SMD:C_0805_2012Metric, F.Cu at (79.2, 61.7)
- added C72: 22nf c0g, Capacitor_SMD:C_0805_2012Metric, F.Cu at (97.1, 11.3)
- added C73: 22nf c0g, Capacitor_SMD:C_0805_2012Metric, F.Cu at (90.1, -14.1)
- added C74: 100nf, Capacitor_SMD:C_0805_2012Metric, F.Cu at (85.6, 41.2)
- added C75: 22nf c0g, Capacitor_SMD:C_0805_2012Metric, F.Cu at (85.6, 44.2)
- added CT8: 100uF, Capacitor_Tantalum_SMD:CP_EIA-7343-31_Kemet-D, F.Cu at (76.1, 30.7)
- added CT9: 100uF, Capacitor_Tantalum_SMD:CP_EIA-7343-31_Kemet-D, F.Cu at (30.7, 60.3)
- added J13: Conn_02x04_Counter_Clockwise, Connector_Molex:Molex_Micro-Fit_3.0_43045-0812_2x04_P3.00mm_Vertical, F.Cu at (98.8, 57.7)
- added J5: HDMI, Connector_FFC-FPC:Amphenol_F32Q-1A7x1-11040_1x40-1MP_P0.5mm_Horizontal, F.Cu at (176.0, 122.7)
- added R106: 0R, Resistor_SMD:R_0805_2012Metric, F.Cu at (119.1, 58.6)
- added R107: 0R, Resistor_SMD:R_0805_2012Metric, F.Cu at (119.1, 61.6)
- added R108: 0R, Resistor_SMD:R_0805_2012Metric, F.Cu at (119.1, 64.5)
- added R109: 10K, Resistor_SMD:R_0805_2012Metric, F.Cu at (105.9, -17.2)
- added R110: 10K ntc, Resistor_SMD:R_0805_2012Metric, F.Cu at (105.9, -14.3)
- added R111: 10K ntc, Resistor_SMD:R_0805_2012Metric, F.Cu at (105.9, -11.3)
- added R112: 10K ntc, Resistor_SMD:R_0805_2012Metric, F.Cu at (110.3, -23.1)
- added R113: 1K, Resistor_SMD:R_0805_2012Metric, F.Cu at (110.3, -20.2)
- added R114: 1K, Resistor_SMD:R_0805_2012Metric, F.Cu at (110.3, -17.2)
- added R115: 1K, Resistor_SMD:R_0805_2012Metric, F.Cu at (110.3, -14.3)
- added R116: 1K, Resistor_SMD:R_0805_2012Metric, F.Cu at (110.3, -11.3)
- added R117: 1K, Resistor_SMD:R_0805_2012Metric, F.Cu at (114.7, -23.1)
- added R118: 1K, Resistor_SMD:R_0805_2012Metric, F.Cu at (114.7, -20.2)
- added R119: 1K, Resistor_SMD:R_0805_2012Metric, F.Cu at (114.7, -17.2)
- added R120: 1K, Resistor_SMD:R_0805_2012Metric, F.Cu at (114.7, -14.3)
- added R121: 22R, Resistor_SMD:R_0805_2012Metric, F.Cu at (61.1, 30.7)
- added R122: 22R, Resistor_SMD:R_0805_2012Metric, F.Cu at (65.1, 23.2)
- added R123: 22R, Resistor_SMD:R_0805_2012Metric, F.Cu at (65.1, 25.7)
- added R124: 22R, Resistor_SMD:R_0805_2012Metric, F.Cu at (65.1, 28.2)
- added R125: 22R, Resistor_SMD:R_0805_2012Metric, F.Cu at (65.1, 30.7)
- added R126: 22R, Resistor_SMD:R_0805_2012Metric, F.Cu at (69.1, 23.2)
- added R127: 22R, Resistor_SMD:R_0805_2012Metric, F.Cu at (69.1, 25.7)
- added R128: 22R, Resistor_SMD:R_0805_2012Metric, F.Cu at (69.1, 28.2)
- added R129: 1K, Resistor_SMD:R_0805_2012Metric, F.Cu at (69.1, 30.7)
- added R130: 10R, Resistor_SMD:R_0805_2012Metric, F.Cu at (114.7, -11.3)
- added R131: 0R, Resistor_SMD:R_0805_2012Metric, F.Cu at (32.3, 38.7)
- added R132: 2.2K, Capacitor_SMD:C_0603_1608Metric, F.Cu at (45.5, -11.3)
- added R133: 2.2K, Capacitor_SMD:C_0603_1608Metric, F.Cu at (45.2, -8.60)
- added R134: 10k, Resistor_SMD:R_0805_2012Metric, F.Cu at (87.2, 61.4)
- added TP36: TestPoint_Small, TestPoint:TestPoint_Pad_D1.5mm, F.Cu at (70.9, 3.35)
- added TP37: TestPoint_Small, TestPoint:TestPoint_Pad_D1.5mm, F.Cu at (70.9, 6.90)
- added TP38: TestPoint_Small, TestPoint:TestPoint_Pad_D1.5mm, F.Cu at (70.9, 10.5)
- added U15: LSF0108PWR, panel:SOP65P640X120-20N, F.Cu at (52.6, -20.5)
- added U27: LSF0108PWR, panel:SOP65P640X120-20N, F.Cu at (52.6, -12.4)
- C10, C11, C4, C5: value 100n -> 100nf
- C13, C42, C50, C57: value 1uf -> 100nf
- C14, C49, C56: value 1uf -> 22nf c0g
- C23, C6, C8, C9: value 10u -> 10uF
- C29, C60, CT4, CT7: value 10uf -> 10uF
- C37: value 100nf -> 1uf
- C45: value 0.1uF -> 100nf
- C46: value 0.1uF -> 22nf c0g
- C47: value 22pF -> 1uf
- C48: value 22pF -> 100nf
- C64, C69, CT2, CT3, CT5: value 100uf -> 100uF
- C66, C67, C71: value 0.022-μF -> 22nf c0g
- CT1, CT6: value 10uf -> 100uF; footprint Capacitor_Tantalum_SMD:CP_EIA-3528-21_Kemet-B -> Capacitor_Tantalum_SMD:CP_EIA-7343-31_Kemet-D
- D1, D3: value LED Green -> LED
- D2: value LED Red -> LED
- J1: value Conn_01x60_MountingPin -> Conn_01x10_Socket; footprint Connector_FFC-FPC:Amphenol_F32Q-1A7x1-11060_1x60-1MP_P0.5mm_Horizontal -> Connector_JST:JST_PH_B10B-PH-K_1x10_P2.00mm_Vertical
- J2, J5: value 690-019-298-412 -> HDMI
- J4: value THD-02-R -> Conn_01x40_MountingPin; footprint Connector_PinHeader_2.54mm:PinHeader_2x02_P2.54mm_Vertical -> Connector_FFC-FPC:Amphenol_F32Q-1A7x1-11040_1x40-1MP_P0.5mm_Horizontal
- J6: value THD-02-R -> Conn_02x04_Counter_Clockwise; footprint Connector_PinHeader_2.54mm:PinHeader_2x02_P2.54mm_Vertical -> Connector_Molex:Molex_Micro-Fit_3.0_43045-0812_2x04_P3.00mm_Vertical
- R1: value 2.2K 1% -> 10K
- R100, R102, R103, R104, R105, R31, R32, R33, R34, R35, R36, R37, R38, R39, R40, R41, R42, R43, R44, R45, R46, R47, R48, R49, R50, R51, R52, R53, R54, R55, R56, R57, R58, R59, R60, R61, R62, R63, R90, R91, R92, R93, R94, R95, R96, R97, R98, R99: value 2.2K 1% -> 2.2K; footprint Resistor_SMD:R_0805_2012Metric -> Capacitor_SMD:C_0603_1608Metric
- R101, R13, R23, R67, R70, R71, R72, R73, R74, R75: value 10k -> 10K
- R12, R5, R64, R65, R66: value 1k -> 1K
- R14: value 100 -> 100R
- R15, R16, R17, R18: value 5.1K 1% -> 5.1K
- R19, R20, R21, R22, R3: value 2.2K 1% -> 2.2K
- R2: value 2.2K 1% -> 0R
- R24: value 12K 1% -> 12K
- R25, R26, R27, R28: value 36K 1% -> 36K
- R29, R4: value 15K 1% -> 15K
- R30: value 47k -> 47K
- R68, R69: value 10k -> 220R
- R77: value 22 -> 22R
- R78: value 22Ω -> 22R
- R79, R80: value 1.5-kΩ -> 1.5K
- R8: value 1k -> 1K; footprint Resistor_SMD:R_0603_1608Metric -> Resistor_SMD:R_0805_2012Metric
- R83, R89: value 330 -> 330R
- R84, R88: value 16 -> 16R
- R9: value 4.7k -> 10K
- SW1: value Right angle Tact button -> SW_Push
- TP2: value TestPoint_Small -> bno_sda; moved to F.Cu
- TP3: value TestPoint_Small -> bno_scl; moved to F.Cu
- TP4, TP5: value TestPoint_Small -> TestPoint; footprint TestPoint:TestPoint_Pad_D1.5mm -> TestPoint:TestPoint_Pad_D2.0mm; moved to F.Cu
- TP6: value TestPoint_Small -> BNO_BOOT; moved to F.Cu
- TP9: moved to F.Cu
- U14: footprint psu:SOP50P490X110-10N -> panel:SOP50P490X110-10N
- U17: value CH343P -> TC1015-xCT; footprint Package_DFN_QFN:QFN-16-1EP_3x3mm_P0.5mm_EP1.7x1.7mm_ThermalVias -> Package_TO_SOT_SMD:SOT-23-5
- U22: value BNO080 -> BNO085
- U23: footprint psu:IC_ICM-45686 -> panel:IC_ICM-45686
- U25: footprint psu:SSOP28 -> panel:SSOP28
- U5: value 74LVC1G07SE-7 -> XC6206P332MR; footprint Package_TO_SOT_SMD:SOT-353_SC-70-5 -> Package_TO_SOT_SMD:SOT-23-3
- Y3: value 5MHz -> 12MHz
- moved U25 290.3 mm to (40.9, 32.5)
- moved U26 284.5 mm to (52.0, 22.4)
- moved SPEAKER1 283.6 mm to (50.1, 29.9)
- moved C45 283.2 mm to (79.2, 64.8)
- moved C46 283.2 mm to (79.2, 67.8)
- moved Y3 280.7 mm to (41.9, 16.7)
- moved R88 274.9 mm to (32.3, 32.8)
- moved R89 274.9 mm to (32.3, 35.8)
- moved R82 272.7 mm to (27.9, 32.8)
- moved R83 272.7 mm to (27.9, 35.8)
- moved R84 272.7 mm to (27.9, 38.7)
- moved R85 272.7 mm to (27.9, 41.7)
- moved C68 270.6 mm to (32.4, 14.8)
- moved C70 270.6 mm to (32.4, 17.8)
- moved C71 270.6 mm to (32.4, 20.8)
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Connections:
- net /CM5_GPIO ( Ethernet, GPIO, SDCARD)/VBAT renamed Net-(BT1-+)
- C37 pad 1: Net-(U17-V3) -> GND
- C37 pad 2: GND -> Net-(U24-Vref)
- C40 pad 1: /YD-ESP32-S3/esp32_chip_pu -> ESP_RST
- C41 pad 1: ESP_3v3 -> GND
- C41 pad 2: GND -> ESP_3v3
- C42 pad 1: ESP_3v3 -> GND
- C42 pad 2: GND -> ESP_3v3
- C43 pad 1: ESP_3v3 -> RPI_5V
- C45 pad 1: GND -> /YD-ESP32-S3/BMO085/3V3
- C45 pad 2: /YD-ESP32-S3/BMO085/CAP -> GND
- C47 pad 1: /YD-ESP32-S3/BMO085/XIN -> ESP_3v3
- C47 pad 2: unconnected-(C47-Pad2) -> GND
- C48 pad 1: /YD-ESP32-S3/BMO085/XOUT -> ESP_3v3
- C52 pad 1: ESP_3v3 -> Net-(U24-Vref)
- C53 pad 2: ESP_3v3 -> Net-(U24-Vref)
- C68 pad 1: GND -> GNDA
- CT6 pad 1: ESP_3v3 -> RPI_5V
- DSI2 pad 20: /CM5_HighSpeed/CAM_SCL1 -> /CM5_GPIO ( Ethernet, GPIO, SDCARD)/ID_SC
- DSI2 pad 21: /CM5_HighSpeed/CAM_SDA1 -> /CM5_GPIO ( Ethernet, GPIO, SDCARD)/ID_SD
- DSW1 pad 10: Net-(DSW1-Pad10) -> unconnected-(DSW1-Pad10)
- DSW1 pad 9: Net-(DSW1-Pad9) -> unconnected-(DSW1-Pad9)
- I2C_0 pad 2: /I2C_SCL_sensors -> /I2C_SDA_sensors
- I2C_0 pad 3: /I2C_SDA_sensors -> /I2C_SCL_sensors
- J1 pad 1: GND -> /CM5_GPIO ( Ethernet, GPIO, SDCARD)/GPIO8
- J1 pad 10: INA226_SDA -> GND
- J1 pad 2: MISO -> /CM5_GPIO ( Ethernet, GPIO, SDCARD)/GPIO7
- J1 pad 3: GND -> /CM5_GPIO ( Ethernet, GPIO, SDCARD)/GPIO11
- J1 pad 4: MOSI -> /CM5_GPIO ( Ethernet, GPIO, SDCARD)/GPIO9
- J1 pad 5: GND -> /CM5_GPIO ( Ethernet, GPIO, SDCARD)/GPIO10
- J1 pad 6: SPI_CLK -> /CM5_GPIO ( Ethernet, GPIO, SDCARD)/GPIO17
- J1 pad 7: GND -> /CM5_GPIO ( Ethernet, GPIO, SDCARD)/GPIO24
- J1 pad 8: /I2C_SCL_sensors -> /CM5_GPIO ( Ethernet, GPIO, SDCARD)/GPIO25
- J1 pad 9: /I2C_SDA_sensors -> /CM5_GPIO ( Ethernet, GPIO, SDCARD)/+3.3v
- J4 pad 1: /CM5_GPIO ( Ethernet, GPIO, SDCARD)/ID_SC -> GND
- J4 pad 2: /CM5_HighSpeed/SCL1 -> MISO
- J4 pad 3: /CM5_GPIO ( Ethernet, GPIO, SDCARD)/ID_SD -> GND
- J4 pad 4: /CM5_HighSpeed/SDA1 -> MOSI
- J6 pad 1: /CM5_GPIO ( Ethernet, GPIO, SDCARD)/TR1_TAP -> GND
- J6 pad 2: /CM5_GPIO ( Ethernet, GPIO, SDCARD)/TR2_TAP -> GND
- J6 pad 3: /CM5_GPIO ( Ethernet, GPIO, SDCARD)/TR0_TAP -> GND
- J6 pad 4: /CM5_GPIO ( Ethernet, GPIO, SDCARD)/TR3_TAP -> 3V3_M.2
- J9 pad 68: Net-(J9-SUSCLK) -> 32.768KHZ
- JP1 pad 3: 1.8V -> /I2C_devices/SEN_1.8V
- JP2 pad 3: 1.8V -> /I2C_devices/SEN_1.8V
- Module1 pad 30: /CM5_GPIO ( Ethernet, GPIO, SDCARD)/GPIO6 -> INA226_ALERT
- Module1 pad 46: /CM5_GPIO ( Ethernet, GPIO, SDCARD)/GPIO22 -> INA226_SCL
- Module1 pad 47: /CM5_GPIO ( Ethernet, GPIO, SDCARD)/GPIO23 -> INA226_SDA
- Module1 pad 48: /CM5_GPIO ( Ethernet, GPIO, SDCARD)/GPIO27 -> ESP_RST
- Module1 pad 56: /CM5_GPIO ( Ethernet, GPIO, SDCARD)/GPIO3 -> RPI_SEN_I2C_SCL
- Module1 pad 58: /CM5_GPIO ( Ethernet, GPIO, SDCARD)/GPIO2 -> RPI_SEN_I2C_SDA
- Module1 pad 95: /CM5_GPIO ( Ethernet, GPIO, SDCARD)/nPWR_LED -> Net-(Module1A-LED_nPWR)
- R1 pad 1: /CM5_HighSpeed/GPIO_VREF -> ESP_3v3
- R1 pad 2: /CM5_HighSpeed/SDA1 -> Net-(R1-Pad2)
- R2 pad 1: /CM5_HighSpeed/GPIO_VREF -> Net-(J4-Pin_37)
- R2 pad 2: /CM5_HighSpeed/SCL1 -> 1NTC
- R66 pad 2: ESP_3v3 -> ESP_RST
- R67 pad 1: /YD-ESP32-S3/esp32_chip_pu -> ESP_RST
- R68 pad 1: Net-(Q2-E) -> /CM5_GPIO ( Ethernet, GPIO, SDCARD)/GPIO4
- R68 pad 2: Net-(Q1-B) -> ESP_UART_RX
- R69 pad 1: Net-(Q2-B) -> /CM5_GPIO ( Ethernet, GPIO, SDCARD)/GPIO5
- R69 pad 2: Net-(Q1-E) -> ESP_UART_TX
- R70 pad 2: Net-(J16-Pin_1) -> PSU-NTC
- R71 pad 2: Net-(J17-Pin_1) -> 0NTC
- R72 pad 2: Net-(J18-Pin_1) -> 1NTC
- R73 pad 2: Net-(J19-Pin_1) -> 2NTC
- R74 pad 2: Net-(J20-Pin_1) -> 3NTC
- R8 pad 2: Net-(R8-Pad2) -> Net-(Module1A-LED_nPWR)
- R83 pad 1: GND -> GNDA
- R84 pad 1: GND -> GNDA
- R87 pad 2: GND -> GNDA
- R88 pad 1: GND -> GNDA
- R89 pad 1: GND -> GNDA
- TP2 pad 1: /CM5_GPIO ( Ethernet, GPIO, SDCARD)/GPIO2 -> Net-(U22-S_SDA)
- TP3 pad 1: /CM5_GPIO ( Ethernet, GPIO, SDCARD)/GPIO3 -> Net-(U22-S_SCL)
- TP4 pad 1: /CM5_GPIO ( Ethernet, GPIO, SDCARD)/GPIO4 -> /CM5_GPIO ( Ethernet, GPIO, SDCARD)/SYNC_OUT
- TP5 pad 1: /CM5_GPIO ( Ethernet, GPIO, SDCARD)/GPIO14 -> GND
- TP6 pad 1: /CM5_GPIO ( Ethernet, GPIO, SDCARD)/GPIO15 -> Net-(U22-BOOTN)
- TP9 pad 1: /CM5_GPIO ( Ethernet, GPIO, SDCARD)/GPIO27 -> /CM5_GPIO ( Ethernet, GPIO, SDCARD)/GPIO16
- U16 pad 22: /I2C_SDA_sensors -> /I2C_SCL_sensors
- U16 pad 23: /I2C_SCL_sensors -> /I2C_SDA_sensors
- U17 pad 3: USB_5V -> ESP_3v3
- U17 pad 4: /YD-ESP32-S3/esp_txd0 -> Net-(U17-Bypass)
- U17 pad 5: /YD-ESP32-S3/esp_txd0 -> /I2C_devices/SEN_1.8V
- U18 pad 27: /YD-ESP32-S3/esp32_gpio0 -> RPI-ESP_INT
- U18 pad 3: /YD-ESP32-S3/esp32_chip_pu -> ESP_RST
- U18 pad 35: RPI-ESP_INT -> unconnected-(U18-IO42-Pad35)
- U19 pad 11: /YD-ESP32-S3/CS -> MCP_CS
- U19 pad 12: /YD-ESP32-S3/SPI_CLK -> SENSOR_SPI_CLK
- U19 pad 13: /YD-ESP32-S3/MOSI -> SENSOR_MISO
- U19 pad 14: /YD-ESP32-S3/MISO -> SENSOR_MOSI
- U19 pad 21: /YD-ESP32-S3/M1_CS -> M1_CS
- U19 pad 22: /YD-ESP32-S3/M2_CS -> M2_CS
- U19 pad 23: /YD-ESP32-S3/M3_CS -> M3_CS
- U19 pad 24: /YD-ESP32-S3/M4_CS -> M4_CS
- U19 pad 5: unconnected-(U19-GPB4-Pad5) -> BNO_RST
- U20 pad 10: /YD-ESP32-S3/M2_CS -> M2_CS
- U20 pad 11: /YD-ESP32-S3/M3_CS -> M3_CS
- U20 pad 13: /YD-ESP32-S3/M4_CS -> M4_CS
- U20 pad 18: ESP_3v3 -> GND
- U20 pad 19: ESP_3v3 -> GND
- U20 pad 9: /YD-ESP32-S3/M1_CS -> M1_CS
- U22 pad 15: unconnected-(U22-S_SCL-Pad15) -> Net-(U22-S_SCL)
- U22 pad 16: unconnected-(U22-S_SDA-Pad16) -> Net-(U22-S_SDA)
- U22 pad 26: /YD-ESP32-S3/BMO085/XOUT -> unconnected-(U22-CLKSEL1/XOUT32-Pad26)
- U22 pad 27: /YD-ESP32-S3/BMO085/XIN -> 32.768KHZ
- U22 pad 4: unconnected-(U22-BOOTN-Pad4) -> Net-(U22-BOOTN)
- U22 pad 9: /YD-ESP32-S3/BMO085/CAP -> Net-(U22-CAP)
- U24 pad 15: ESP_3v3 -> Net-(U24-Vref)
- U24 pad 7: unconnected-(U24-CH6-Pad7) -> Net-(U24-CH6)
- U24 pad 8: unconnected-(U24-CH7-Pad8) -> Net-(U24-CH7)
- U25 pad 12: GND -> GNDA
- U25 pad 17: GND -> GNDA
- U26 pad 7: GND -> GNDA
- U26 pad 9: GND -> GNDA
- U28 pad 22: /I2C_SDA_sensors -> /I2C_SCL_sensors
- U28 pad 23: /I2C_SCL_sensors -> /I2C_SDA_sensors
- U5 pad 1: unconnected-(U5-nc-Pad1) -> GND
- U5 pad 2: /CM5_GPIO ( Ethernet, GPIO, SDCARD)/nPWR_LED -> Net-(U5-VO)
- U5 pad 3: GND -> USB_5V
- U6 pad 3: Net-(J9-SUSCLK) -> 32.768KHZ
Routing:
- net Net-(Module1A-LED_nPWR): track 0.00 -> 4.53 mm, vias 0 -> 1
- net /CM5_GPIO ( Ethernet, GPIO, SDCARD)/nPWR_LED: track 4.53 -> 0.00 mm, vias 1 -> 0
- net /USB2-HUB/HD3_N: track 0.00 -> 3.01 mm, vias 0 -> 1
- net /USB2-HUB/HD2_P: track 0.00 -> 2.97 mm, vias 0 -> 1
- net ESP_3v3: track 2.95 -> 0.00 mm
- net /USB2-HUB/HD1_P: track 0.00 -> 2.84 mm, vias 0 -> 1
- net /USB2-HUB/HD4_N: track 0.00 -> 2.83 mm, vias 0 -> 1
- net /USB2-HUB/HD3_P: track 0.00 -> 2.75 mm, vias 0 -> 1
- net /USB2-HUB/HD2_N: track 0.00 -> 2.71 mm, vias 0 -> 1
- net /USB2-HUB/HD1_N: track 0.00 -> 2.59 mm, vias 0 -> 1
- net /USB2-HUB/HD4_P: track 0.00 -> 2.58 mm, vias 0 -> 1
- net /CM5_HighSpeed/USB3-0-TX_N: track 31.6 -> 33.4 mm
- net /CM5_HighSpeed/USB3-0-TX_P: track 32.2 -> 34.0 mm
- net INA226_ALERT: track 0.00 -> 1.04 mm, vias 0 -> 1
- net /CM5_GPIO ( Ethernet, GPIO, SDCARD)/GPIO6: track 1.04 -> 0.00 mm, vias 1 -> 0
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